Commit message: Working mock and real hw interfaces

File: ada_description/urdf/kinova_common.xacro (robot description, xacro)
@@ -145,5 +145,5 @@
 		    </transmission>
         <xacro:kinova_armlink link_name="${prefix}link_finger_tip_${finger_number}" link_mesh="finger_distal" mesh_no="58"/>
-        <joint name="${prefix}joint_finger_tip_${finger_number}" type="revolute">
+        <joint name="${prefix}joint_finger_tip_${finger_number}" type="fixed">
             <parent link="${prefix}link_finger_${finger_number}"/>
             <child link="${prefix}link_finger_tip_${finger_number}"/>
