Commit message: fixed pre-commit issues

File: ada_description/urdf/ada_standalone.xacro (robot description, xacro)
@@ -1,4 +1,5 @@
 <?xml version="1.0"?>
-<robot xmlns:xi="http://www.w3.org/2001/XInclude"
+<robot
+  xmlns:xi="http://www.w3.org/2001/XInclude"
   xmlns:gazebo="http://playerstage.sourceforge.net/gazebo/xmlschema/#gz"
   xmlns:model="http://playerstage.sourceforge.net/gazebo/xmlschema/#model"
@@ -13,9 +14,19 @@
   xmlns:physics="http://playerstage.sourceforge.net/gazebo/xmlschema/#physics"
   xmlns:xacro="http://www.ros.org/wiki/xacro"
-  name="ada">
-  <xacro:arg name="use_forque" default="true" />
-  <xacro:include filename="$(find ada_description)/urdf/ada.xacro" />
-  <xacro:property name="root" value="root" />
-  <xacro:property name="use_forque" value="$(arg use_forque)" />
-  <xacro:ada use_forque="${use_forque}" />
+  name="ada"
+>
+  <xacro:arg
+    name="use_forque"
+    default="true"
+  />
+  <xacro:include filename="$(find ada_description)/urdf/ada.xacro"/>
+  <xacro:property
+    name="root"
+    value="root"
+  />
+  <xacro:property
+    name="use_forque"
+    value="$(arg use_forque)"
+  />
+  <xacro:ada use_forque="${use_forque}"/>
 </robot>

File: ada_moveit/config/ada.urdf.xacro (robot description, xacro)
@@ -32,5 +32,11 @@
   />
   <xacro:ada use_forque="$(arg use_forque)"/>
-  <xacro:articutool base_parent="j2n6s200_end_effector" end_effector_tool="${end_effector_tool}" joint_origin_rpy="0 0 ${J_PI/2}" joint_origin_xyz="0 -2.25 -1" lock_joints="$(arg lock_joints)"/>
+  <xacro:articutool
+    base_parent="j2n6s200_end_effector"
+    end_effector_tool="${end_effector_tool}"
+    joint_origin_rpy="0 0 ${J_PI/2}"
+    joint_origin_xyz="0 -2.25 -1"
+    lock_joints="$(arg lock_joints)"
+  />
   <!-- Import control_xacro -->
   <xacro:include filename="ada.ros2_control.xacro"/>
