Commit message: Finished unified ada.xacro

File: ada_description/urdf/ada.xacro (robot description, xacro)
@@ -13,7 +13,8 @@
     xmlns:physics="http://playerstage.sourceforge.net/gazebo/xmlschema/#physics"
   xmlns:xacro="http://www.ros.org/wiki/xacro" name="camera">
- <xacro:include filename="$(find ada_description)/urdf/forque/forque.xacro"/>
- <xacro:include filename="$(find ada_description)/urdf/camera/camera.xacro"/>
+  <xacro:include filename="$(find ada_description)/urdf/forque/forque.xacro"/>
+  <xacro:include filename="$(find ada_description)/urdf/camera/camera.xacro"/>
   <xacro:include filename="$(find ada_description)/urdf/j2n6s200.xacro"/>
+  <xacro:arg name="use_forque" default="false"/>
   <link name="root"/>
   <!-- for gazebo -->
@@ -26,6 +27,9 @@
   <xacro:property name="robot_root" value="root" />
   <xacro:j2n6s200 base_parent="${robot_root}"/>
-  <xacro:camera_assembly base_parent="j2n6s200_link_6" base_xyz="0.0165 0 0" base_rpy="${3*J_PI/2} 0 ${3*J_PI/2}"/>
+  <xacro:camera_assembly base_parent="j2n6s200_link_6" base_xyz="0.0165 0 0.0011" base_rpy="${3*J_PI/2} 0 ${3*J_PI/2}"/>
   <xacro:forque_assembly_link link_name="FTArmMount" link_mesh="2023_03_09_FTArmMount"/>
-  <xacro:forque_assembly_joint joint_name="FTArmMount_to_arm" parent="j2n6s200_link_6" child="FTArmMount" joint_origin_xyz="0 -0.01 0" joint_origin_rpy="${J_PI/2} 0 ${J_PI/2}"/>
+  <xacro:forque_assembly_joint joint_name="FTArmMount_to_arm" parent="j2n6s200_link_6" child="FTArmMount" joint_origin_xyz="0.0065 -0.011 -0.0075" joint_origin_rpy="${J_PI/2} 0 ${J_PI/2}"/>
+  <xacro:if value="$(arg use_forque)">
+    <xacro:forque_assembly base_parent="FTArmMount"/>
+  </xacro:if>
 </robot>

File: ada_description/urdf/camera/camera.xacro (robot description, xacro)
@@ -14,5 +14,5 @@
 	xmlns:xacro="http://www.ros.org/wiki/xacro">
 	<xacro:include filename="$(find ada_description)/urdf/camera/d415urdf.xacro"/>
-	<xacro:property name="camColor" value="1 0 0 1" />
+	<xacro:property name="camColor" value="0.4 0.4 0.4 1" />
 	<xacro:property name="J_PI" value="3.1415926535897931" />
 	<xacro:macro name="camera_assembly_link" params="link_name link_mesh">

File: ada_description/urdf/camera/d415urdf.xacro (robot description, xacro)
@@ -21,5 +21,5 @@
 <robot name="sensor_d415" xmlns:xacro="http://ros.org/wiki/xacro">
   <material name="aluminum">
-    <color rgba="0.5 0.5 0.5 1"/>
+    <color rgba="0.4 0.4 0.4 1"/>
   </material>
   <material name="plastic">

File: ada_description/urdf/forque/forque.xacro (robot description, xacro)
@@ -13,5 +13,5 @@
     xmlns:physics="http://playerstage.sourceforge.net/gazebo/xmlschema/#physics"
 	xmlns:xacro="http://www.ros.org/wiki/xacro">
-	<xacro:property name="forque_color" value="1 0 0 1" />
+	<xacro:property name="forque_color" value="0.4 0.4 0.4 1" />
 	<xacro:property name="J_PI" value="3.1415926535897931" />
 	<xacro:macro name="forque_assembly_link" params="link_name link_mesh">
@@ -52,4 +52,8 @@
 	  	<xacro:forque_assembly_link link_name="forkHandle" link_mesh="2023_03_09_forkHandle"/>
 	  	<xacro:forque_assembly_joint joint_name="forkHandle_to_FTMount" parent="FTMount" child="forkHandle" joint_origin_xyz="0 0 0" joint_origin_rpy="0 0 0"/>
+	  	<xacro:forque_assembly_link link_name="forque" link_mesh="ATI-9105-TW-NANO25-E"/>
+	  	<xacro:forque_assembly_joint joint_name="forque_to_forkHandle" parent="forkHandle" child="forque" joint_origin_xyz="-0.00634 -0.222553 -0.004286" joint_origin_rpy="${J_PI/2} ${J_PI/3} 0"/>
+	  	<xacro:forque_assembly_link link_name="forkTine" link_mesh="fork_tine"/>
+	  	<xacro:forque_assembly_joint joint_name="forkTine_to_forque" parent="forque" child="forkTine" joint_origin_xyz="-0.0054 0.008 0.093" joint_origin_rpy="0 ${J_PI} ${240*J_PI/180}"/>
 	</xacro:macro>
 </root>

Commit message: Added empirical extrinsics

File: ada_description/urdf/ada.xacro (robot description, xacro)
@@ -16,5 +16,5 @@
   <xacro:include filename="$(find ada_description)/urdf/camera/camera.xacro"/>
   <xacro:include filename="$(find ada_description)/urdf/j2n6s200.xacro"/>
-  <xacro:arg name="use_forque" default="false"/>
+  <xacro:arg name="use_forque" default="true"/>
   <link name="root"/>
   <!-- for gazebo -->
@@ -28,8 +28,28 @@
   <xacro:j2n6s200 base_parent="${robot_root}"/>
   <xacro:camera_assembly base_parent="j2n6s200_link_6" base_xyz="0.0165 0 0.0011" base_rpy="${3*J_PI/2} 0 ${3*J_PI/2}"/>
+  <!-- Extrinsics -->
+  <link name="camera_link" />
+  <joint name="extrinsics" type="fixed">
+    <origin xyz="0.023 0.055 0.005" rpy="-0.039 0.100 -0.007" />
+    <parent link="stabilizer" />
+    <child link="camera_link" />
+  </joint>
+  <!-- Copy Realsense in case of simulation -->
+  <link name="camera_color_optical_frame" />
+  <joint name="optical_republish" type="fixed">
+    <origin xyz="0.000 -0.015 0.000" rpy="-1.564 0.000 -1.573" />
+    <parent link="camera_link" />
+    <child link="camera_color_optical_frame" />
+  </joint>
   <xacro:forque_assembly_link link_name="FTArmMount" link_mesh="2023_03_09_FTArmMount"/>
   <xacro:forque_assembly_joint joint_name="FTArmMount_to_arm" parent="j2n6s200_link_6" child="FTArmMount" joint_origin_xyz="0.0065 -0.011 -0.0075" joint_origin_rpy="${J_PI/2} 0 ${J_PI/2}"/>
   <xacro:if value="$(arg use_forque)">
     <xacro:forque_assembly base_parent="FTArmMount"/>
+    <link name="FTSensor" />
+      <joint name="EE_to_FTSensor" type="fixed">
+        <child link="FTSensor"/>
+        <parent link="j2n6s200_end_effector"/>
+        <origin rpy="0 0 0" xyz="0.0 0.0 0.092"/>
+    </joint>
   </xacro:if>
 </robot>

File: ada_description/urdf/camera/camera.xacro (robot description, xacro)
@@ -57,5 +57,5 @@
 		<xacro:camera_assembly_link link_name="stabilizer" link_mesh="2023_03_09_cameraStabilizer"/>
 		<xacro:camera_assembly_joint joint_name="stabilizer_to_enclosureTop" parent="enclosureTop" child="stabilizer" joint_origin_xyz="0.0842 0.041 0.0343" joint_origin_rpy="0 ${14.621 * J_PI / 180} 0"/>
-		<xacro:sensor_d415 parent="stabilizer" use_mesh="true">
+		<xacro:sensor_d415 parent="stabilizer" use_mesh="true" name="uncalibrated_camera">
 			<origin xyz="0.0165 0 0.0005" rpy="0 0 0" />
 		</xacro:sensor_d415>

File: ada_description/urdf/camera/d415urdf.xacro (robot description, xacro)
@@ -26,5 +26,5 @@
     <color rgba="0.1 0.1 0.1 1"/>
   </material>
-  <xacro:macro name="sensor_d415" params="parent *origin  name:=camera  use_nominal_extrinsics:=false add_plug:=false use_mesh:=true">
+  <xacro:macro name="sensor_d415" params="parent *origin  name:=camera  use_nominal_extrinsics:=true add_plug:=false use_mesh:=true">
     <xacro:property name="M_PI" value="3.1415926535897931" />
     <!-- The following values are approximate, and the camera node

File: ada_hardware/urdf/ada_hardware.xacro (robot description, xacro)
@@ -4,16 +4,6 @@
 	xmlns:xacro="http://www.ros.org/wiki/xacro" name="ada_hardware">
   <xacro:arg name="use_mock_hardware" default="false" />
-  <xacro:include filename="$(find ada_description)/urdf/j2n6s200.xacro"/>
+  <xacro:include filename="$(find ada_description)/urdf/ada.xacro"/>
   <xacro:include filename="$(find ada_hardware)/urdf/ada_hardware.ros2_control.xacro"/>
-  <link name="root"/>
-  <!-- for gazebo -->
-  <link name="world"/>
-  <joint name="connect_root_and_world" type="fixed">
-    <child link="root" />
-    <parent link="world" />
-    <origin xyz="0 0 0" rpy="0 0 0" />
-  </joint>
-  <xacro:property name="robot_root" value="root" />
-  <xacro:j2n6s200  base_parent="${robot_root}"/>
   <xacro:ada_hardware_interface
     name="Jaco2"

Commit message: [WIP] adding masses and inertia to urdf

File: ada_description/urdf/ada.xacro (robot description, xacro)
@@ -42,5 +42,9 @@
     <child link="camera_color_optical_frame" />
   </joint>
-  <xacro:forque_assembly_link link_name="FTArmMount" link_mesh="2023_03_09_FTArmMount"/>
+  <xacro:forque_assembly_link link_name="FTArmMount" link_mesh="2023_03_09_FTArmMount" mass="0.0025" cog="0.011184837 -0.024537498 -0.035437509">
+    <inertia    ixx="0.00000016943"
+                iyy="0.00000010161" iyz="-0.000095997"
+                izz="0.00000025711" ixy="-0.050568" ixz="-0.019075" />
+  </xacro:forque_assembly_link>
   <xacro:forque_assembly_joint joint_name="FTArmMount_to_arm" parent="j2n6s200_link_6" child="FTArmMount" joint_origin_xyz="0.0065 -0.011 -0.0075" joint_origin_rpy="${J_PI/2} 0 ${J_PI/2}"/>
   <xacro:if value="$(arg use_forque)">

File: ada_description/urdf/camera/camera.xacro (robot description, xacro)
@@ -16,5 +16,5 @@
 	<xacro:property name="camColor" value="0.4 0.4 0.4 1" />
 	<xacro:property name="J_PI" value="3.1415926535897931" />
-	<xacro:macro name="camera_assembly_link" params="link_name link_mesh">
+	<xacro:macro name="camera_assembly_link" params="link_name link_mesh mass:=0">
 		<link name="${link_name}">
 			<visual>
@@ -35,4 +35,7 @@
                 </geometry>
             </collision>
+            <inertial>
+            	<mass value="${mass}"/>
+            </inertial>
 		</link>
 	</xacro:macro>

File: ada_description/urdf/forque/forque.xacro (robot description, xacro)
@@ -15,5 +15,9 @@
 	<xacro:property name="forque_color" value="0.4 0.4 0.4 1" />
 	<xacro:property name="J_PI" value="3.1415926535897931" />
-	<xacro:macro name="forque_assembly_link" params="link_name link_mesh">
+	<xacro:property name="default_origin" value="0 0 0"/>
+	<xacro:property name="default_inertial">
+		<inertia ixx="0.001" iyy="0.001" iyz="0.001" izz="0.001" ixy="0.001" ixz="0.001"/>
+	</xacro:property>
+	<xacro:macro name="forque_assembly_link" params="link_name link_mesh mass:=0 cog:='0 0 0' *inertia">
 		<link name="${link_name}">
 			<visual>
@@ -34,4 +38,9 @@
                 </geometry>
             </collision>
+            <inertial>
+            	<origin xyz="${cog}" rpy="0 0 0"/>
+            	<mass value="${mass}"/>
+            	<xacro:insert_block name="inertia"/>
+            </inertial>
 		</link>
 	</xacro:macro>
@@ -45,15 +54,27 @@
 	</xacro:macro>
 	<xacro:macro name="forque_assembly" params="base_parent">
-		<xacro:forque_assembly_link link_name="FTMount" link_mesh="2023_03_09_FTMount"/>
+		<xacro:forque_assembly_link link_name="FTMount" link_mesh="2023_03_09_FTMount" mass="0.022" cog="0.0111797 -0.110193 -0.0384312">
+			<inertia ixx="0.00000047293" iyy="7871700" iyz="0.001" izz="0.001" ixy="0.001" ixz="0.001"/>
+        </xacro:forque_assembly_link>
 	  	<xacro:forque_assembly_joint joint_name="FTMount_to_world" parent="${base_parent}" child="FTMount" joint_origin_xyz="0 0 0" joint_origin_rpy="0 0 0"/>
-	  	<xacro:forque_assembly_link link_name="FT" link_mesh="2023_03_09_wirelessFT"/>
+	  	<xacro:forque_assembly_link link_name="FT" link_mesh="2023_03_09_wirelessFT" mass="0.278">
+	  		<xacro:insert_block name="default_inertial"/>
+	  	</xacro:forque_assembly_link>
 	  	<xacro:forque_assembly_joint joint_name="FT_to_FTMount" parent="FTMount" child="FT" joint_origin_xyz="0 0 0" joint_origin_rpy="0 0 0"/>
-	  	<xacro:forque_assembly_link link_name="FTAntenna" link_mesh="2023_03_09_wirelessFTAntenna"/>
+	  	<xacro:forque_assembly_link link_name="FTAntenna" link_mesh="2023_03_09_wirelessFTAntenna">
+	  		<xacro:insert_block name="default_inertial"/>
+	  	</xacro:forque_assembly_link>
 	  	<xacro:forque_assembly_joint joint_name="FTAntenna_to_FT" parent="FT" child="FTAntenna" joint_origin_xyz="0 0 0" joint_origin_rpy="0 0 0"/>
-	  	<xacro:forque_assembly_link link_name="forkHandle" link_mesh="2023_03_09_forkHandle"/>
+	  	<xacro:forque_assembly_link link_name="forkHandle" link_mesh="2023_03_09_forkHandle">
+	  		<xacro:insert_block name="default_inertial"/>
+	  	</xacro:forque_assembly_link>
 	  	<xacro:forque_assembly_joint joint_name="forkHandle_to_FTMount" parent="FTMount" child="forkHandle" joint_origin_xyz="0 0 0" joint_origin_rpy="0 0 0"/>
-	  	<xacro:forque_assembly_link link_name="forque" link_mesh="ATI-9105-TW-NANO25-E"/>
+	  	<xacro:forque_assembly_link link_name="forque" link_mesh="ATI-9105-TW-NANO25-E">
+	  		<xacro:insert_block name="default_inertial"/>
+	  	</xacro:forque_assembly_link>
 	  	<xacro:forque_assembly_joint joint_name="forque_to_forkHandle" parent="forkHandle" child="forque" joint_origin_xyz="-0.00634 -0.222553 -0.004286" joint_origin_rpy="${J_PI/2} ${J_PI/3} 0"/>
-	  	<xacro:forque_assembly_link link_name="forkTine" link_mesh="fork_tine"/>
+	  	<xacro:forque_assembly_link link_name="forkTine" link_mesh="fork_tine">
+	  		<xacro:insert_block name="default_inertial"/>
+	  	</xacro:forque_assembly_link>
 	  	<xacro:forque_assembly_joint joint_name="forkTine_to_forque" parent="forque" child="forkTine" joint_origin_xyz="-0.0054 0.008 0.093" joint_origin_rpy="0 ${J_PI} ${240*J_PI/180}"/>
 	  	<link name="forkTip" />

Commit message: Added starter MoveIt 2 Config

File: ada_description/urdf/ada.xacro (robot description, xacro)
@@ -12,5 +12,5 @@
     xmlns:renderable="http://playerstage.sourceforge.net/gazebo/xmlschema/#renderable"
     xmlns:physics="http://playerstage.sourceforge.net/gazebo/xmlschema/#physics"
-  xmlns:xacro="http://www.ros.org/wiki/xacro" name="camera">
+  xmlns:xacro="http://www.ros.org/wiki/xacro" name="ada">
   <xacro:include filename="$(find ada_description)/urdf/forque/forque.xacro"/>
   <xacro:include filename="$(find ada_description)/urdf/camera/camera.xacro"/>
@@ -18,11 +18,4 @@
   <xacro:arg name="use_forque" default="true"/>
   <link name="root"/>
-  <!-- for gazebo -->
-  <link name="world"/>
-  <joint name="connect_root_and_world" type="fixed">
-    <child link="root" />
-    <parent link="world" />
-    <origin xyz="0 0 0" rpy="0 0 0" />
-  </joint>
   <xacro:property name="robot_root" value="root" />
   <xacro:j2n6s200 base_parent="${robot_root}"/>

File: ada_description/urdf/camera/d415urdf.xacro (robot description, xacro)
@@ -26,5 +26,5 @@
     <color rgba="0.1 0.1 0.1 1"/>
   </material>
-  <xacro:macro name="sensor_d415" params="parent *origin  name:=camera  use_nominal_extrinsics:=true add_plug:=false use_mesh:=true">
+  <xacro:macro name="sensor_d415" params="parent *origin  name:=camera  use_nominal_extrinsics:=false add_plug:=false use_mesh:=true">
     <xacro:property name="M_PI" value="3.1415926535897931" />
     <!-- The following values are approximate, and the camera node

File: ada_description/urdf/forque/forque.xacro (robot description, xacro)
@@ -44,11 +44,13 @@
 		</joint>
 	</xacro:macro>
-	<xacro:macro name="forque_assembly" params="base_parent">
+	<xacro:macro name="forque_assembly" params="base_parent use_antenna:=false">
 		<xacro:forque_assembly_link link_name="FTMount" link_mesh="2023_03_09_FTMount"/>
 	  	<xacro:forque_assembly_joint joint_name="FTMount_to_world" parent="${base_parent}" child="FTMount" joint_origin_xyz="0 0 0" joint_origin_rpy="0 0 0"/>
 	  	<xacro:forque_assembly_link link_name="FT" link_mesh="2023_03_09_wirelessFT"/>
 	  	<xacro:forque_assembly_joint joint_name="FT_to_FTMount" parent="FTMount" child="FT" joint_origin_xyz="0 0 0" joint_origin_rpy="0 0 0"/>
-	  	<xacro:forque_assembly_link link_name="FTAntenna" link_mesh="2023_03_09_wirelessFTAntenna"/>
-	  	<xacro:forque_assembly_joint joint_name="FTAntenna_to_FT" parent="FT" child="FTAntenna" joint_origin_xyz="0 0 0" joint_origin_rpy="0 0 0"/>
+	  	<xacro:if value="${use_antenna}">
+		  	<xacro:forque_assembly_link link_name="FTAntenna" link_mesh="2023_03_09_wirelessFTAntenna"/>
+		  	<xacro:forque_assembly_joint joint_name="FTAntenna_to_FT" parent="FT" child="FTAntenna" joint_origin_xyz="0 0 0" joint_origin_rpy="0 0 0"/>
+		</xacro:if>
 	  	<xacro:forque_assembly_link link_name="forkHandle" link_mesh="2023_03_09_forkHandle"/>
 	  	<xacro:forque_assembly_joint joint_name="forkHandle_to_FTMount" parent="FTMount" child="forkHandle" joint_origin_xyz="0 0 0" joint_origin_rpy="0 0 0"/>

Commit message: changed forque mount to have default inertia

File: ada_description/urdf/ada.xacro (robot description, xacro)
@@ -36,7 +36,5 @@
   </joint>
   <xacro:forque_assembly_link link_name="FTArmMount" link_mesh="2023_03_09_FTArmMount" mass="0.0025" cog="0.011184837 -0.024537498 -0.035437509">
-    <inertia    ixx="0.00000016943"
-                iyy="0.00000010161" iyz="-0.000095997"
-                izz="0.00000025711" ixy="-0.050568" ixz="-0.019075" />
+    <xacro:insert_block name="default_inertial"/>
   </xacro:forque_assembly_link>
   <xacro:forque_assembly_joint joint_name="FTArmMount_to_arm" parent="j2n6s200_link_6" child="FTArmMount" joint_origin_xyz="0.0065 -0.011 -0.0075" joint_origin_rpy="${J_PI/2} 0 ${J_PI/2}"/>

Commit message: Modified ADA urdf with updated camera-back position

File: ada_description/urdf/ada.xacro (robot description, xacro)
@@ -25,5 +25,5 @@
   <joint name="extrinsics" type="fixed">
     <origin xyz="0.023 0.055 0.005" rpy="-0.039 0.100 -0.007" />
-    <parent link="stabilizer" />
+    <parent link="cameraMount" />
     <child link="camera_link" />
   </joint>

File: ada_description/urdf/camera/camera.xacro (robot description, xacro)
@@ -67,14 +67,14 @@
 	  	</xacro:camera_assembly_link>
 		<xacro:camera_assembly_joint joint_name="nano_to_enclosureBottom" parent="enclosureBottom" child="nano" joint_origin_xyz="0.0105 0.014 -0.0015" joint_origin_rpy="0 0 0"/>
-		<xacro:camera_assembly_link link_name="enclosureTop" link_mesh="2023_03_09_nanoEnclosureTop" mass="0.046" cog="0.04817211 0.03496864 0.02671124">
+		<xacro:camera_assembly_link link_name="enclosureTop" link_mesh="2023_06_06_nanoEnclosureTopCameraBack" mass="0.046" cog="0.04817211 0.03496864 0.02671124">
 	  		<xacro:insert_block name="default_inertial"/>
 	  	</xacro:camera_assembly_link>
-		<xacro:camera_assembly_joint joint_name="enclosureTop_to_enclosureBottom" parent="enclosureBottom" child="enclosureTop" joint_origin_xyz="0 0 0" joint_origin_rpy="0 0 0"/>
-		<xacro:camera_assembly_link link_name="stabilizer" link_mesh="2023_03_09_cameraStabilizer" mass="0.004" cog="0.00272454 0.00000231884 0.00514249">
+		<xacro:camera_assembly_joint joint_name="enclosureTop_to_enclosureBottom" parent="enclosureBottom" child="enclosureTop" joint_origin_xyz="0.009925 0.04099 0.05442" joint_origin_rpy="0 ${165.4 * J_PI / 180} ${J_PI}"/>
+		<xacro:camera_assembly_link link_name="cameraMount" link_mesh="2023_06_06_cameraBackMount" mass="0.004" cog="0.00272454 0.00000231884 0.00514249">
 	  		<xacro:insert_block name="default_inertial"/>
 	  	</xacro:camera_assembly_link>
-		<xacro:camera_assembly_joint joint_name="stabilizer_to_enclosureTop" parent="enclosureTop" child="stabilizer" joint_origin_xyz="0.0842 0.041 0.0343" joint_origin_rpy="0 ${14.621 * J_PI / 180} 0"/>
-		<xacro:sensor_d415 parent="stabilizer" use_mesh="true" name="uncalibrated_camera">
-			<origin xyz="0.0165 0 0.0005" rpy="0 0 0" />
+		<xacro:camera_assembly_joint joint_name="cameraMount_to_enclosureTop" parent="enclosureTop" child="cameraMount" joint_origin_xyz="-0.0132 0 -0.022" joint_origin_rpy="0 ${J_PI / 2} 0"/>
+		<xacro:sensor_d415 parent="cameraMount" use_mesh="true" name="uncalibrated_camera">
+			<origin xyz="0.006 0 0.013" rpy="0 ${-J_PI / 2} ${J_PI}" />
 		</xacro:sensor_d415>
 	</xacro:macro>

Commit message: Updated default camera calibration

File: ada_description/urdf/ada.xacro (robot description, xacro)
@@ -24,5 +24,5 @@
   <link name="camera_link" />
   <joint name="extrinsics" type="fixed">
-    <origin xyz="0.023 0.055 0.005" rpy="-0.039 0.100 -0.007" />
+    <origin xyz="0.0194 -0.01606 0.029014" rpy="0.17234 -1.56127 2.96967" />
     <parent link="cameraMount" />
     <child link="camera_link" />

Commit message: [WIP] Started adding robot_tilt joint to urdf

File: ada_description/urdf/ada.xacro (robot description, xacro)
@@ -17,5 +17,15 @@
   <xacro:include filename="$(find ada_description)/urdf/j2n6s200.xacro"/>
   <xacro:arg name="use_forque" default="true"/>
+  <xacro:arg name="world_link" default="world"/>
   <link name="root"/>
+  <link name="$(arg world_link)"/>
+  <joint name="robot_tilt" type="revolute">
+    <origin xyz="0 0 0" rpy="0 0 0" />
+    <child link="root" />
+    <parent link="$(arg world_link)" />
+    <axis xyz="0 1 0"/>
+    <limit effort="80" velocity="${36*J_PI/180}" lower="${-J_PI}" upper="${J_PI}"/>
+    <dynamics damping="0.0" friction="0.0"/>
+  </joint>
   <xacro:property name="robot_root" value="root" />
   <xacro:j2n6s200 base_parent="${robot_root}"/>
@@ -44,5 +54,5 @@
     <xacro:forque_assembly base_parent="FTArmMount"/>
     <link name="FTSensor" />
-      <joint name="EE_to_FTSensor" type="fixed">
+    <joint name="EE_to_FTSensor" type="fixed">
         <child link="FTSensor"/>
         <parent link="j2n6s200_end_effector"/>

Commit message: Added tilt joint to urdf

File: ada_description/urdf/ada.xacro (robot description, xacro)
@@ -17,16 +17,15 @@
   <xacro:include filename="$(find ada_description)/urdf/j2n6s200.xacro"/>
   <xacro:arg name="use_forque" default="true"/>
-  <xacro:arg name="world_link" default="world"/>
   <link name="root"/>
-  <link name="$(arg world_link)"/>
+  <link name="root_tilt"/>
   <joint name="robot_tilt" type="revolute">
     <origin xyz="0 0 0" rpy="0 0 0" />
-    <child link="root" />
-    <parent link="$(arg world_link)" />
+    <child link="root_tilt" />
+    <parent link="root" />
     <axis xyz="0 1 0"/>
     <limit effort="80" velocity="${36*J_PI/180}" lower="${-J_PI}" upper="${J_PI}"/>
     <dynamics damping="0.0" friction="0.0"/>
   </joint>
-  <xacro:property name="robot_root" value="root" />
+  <xacro:property name="robot_root" value="root_tilt" />
   <xacro:j2n6s200 base_parent="${robot_root}"/>
   <xacro:camera_assembly base_parent="j2n6s200_link_6" base_xyz="0.0165 0 0.0011" base_rpy="${3*J_PI/2} 0 ${3*J_PI/2}"/>

Commit message: [WIP] Cleaning up code and adding documentation

File: ada_description/urdf/ada.xacro (robot description, xacro)
@@ -24,5 +24,7 @@
     <parent link="root" />
     <axis xyz="0 1 0"/>
-    <limit effort="80" velocity="${36*J_PI/180}" lower="${-J_PI}" upper="${J_PI}"/>
+    <!-- effort copied from j2n6s200 joint 2, velocity is max velocity the wheelchair can tilt,
+    lower and upper limits generously encompass the range of the wheelchair's tilt-->
+    <limit effort="80" velocity="0.15" lower="${-J_PI}" upper="${J_PI}"/>
     <dynamics damping="0.0" friction="0.0"/>
   </joint>
