Commit message: IMU Tilt Publisher (#11)
* Modified ADA urdf with updated camera-back position

* Created package for IMU data

* Added IMU data reader for calibration

* [WIP] worked on IMU jointstate publisher node

* [WIP] creating IMU jointstate publisher node

* [WIP] Added IMU position and velocity to message

* [WIP] Added IMU position and velocity to message

* [WIP] Added calibration parameters and launch file

* Connected launch file to yaml config file

* [WIP] Started adding robot_tilt joint to urdf

* Added tilt joint to urdf

* [WIP] Cleaning up code and adding documentation

* Addressed all comments, ran black and pylint

* [WIP] Update README.md

* Switch stabilizer frame to cameraMount frame

* Update README.md

* Remove flake8, add license, fix maintainer/author

---------

Co-authored-by: Ethan K. Gordon <ekgordon@cs.washington.edu>

File: ada_description/urdf/ada.xacro (robot description, xacro)
@@ -18,5 +18,16 @@
   <xacro:arg name="use_forque" default="true"/>
   <link name="root"/>
-  <xacro:property name="robot_root" value="root" />
+  <link name="root_tilt"/>
+  <joint name="robot_tilt" type="revolute">
+    <origin xyz="0 0 0" rpy="0 0 0" />
+    <child link="root_tilt" />
+    <parent link="root" />
+    <axis xyz="0 1 0"/>
+    <!-- effort copied from j2n6s200 joint 2, velocity is max velocity the wheelchair can tilt,
+    lower and upper limits generously encompass the range of the wheelchair's tilt-->
+    <limit effort="80" velocity="0.15" lower="${-J_PI}" upper="${J_PI}"/>
+    <dynamics damping="0.0" friction="0.0"/>
+  </joint>
+  <xacro:property name="robot_root" value="root_tilt" />
   <xacro:j2n6s200 base_parent="${robot_root}"/>
   <xacro:camera_assembly base_parent="j2n6s200_link_6" base_xyz="0.0165 0 0.0011" base_rpy="${3*J_PI/2} 0 ${3*J_PI/2}"/>
@@ -44,5 +55,5 @@
     <xacro:forque_assembly base_parent="FTArmMount"/>
     <link name="FTSensor" />
-      <joint name="EE_to_FTSensor" type="fixed">
+    <joint name="EE_to_FTSensor" type="fixed">
         <child link="FTSensor"/>
         <parent link="j2n6s200_end_effector"/>

Commit message: Changed axis of rotation for IMU joint

File: ada_description/urdf/ada.xacro (robot description, xacro)
@@ -23,5 +23,5 @@
     <child link="root_tilt" />
     <parent link="root" />
-    <axis xyz="0 1 0"/>
+    <axis xyz="1 0 0"/>
     <!-- effort copied from j2n6s200 joint 2, velocity is max velocity the wheelchair can tilt,
     lower and upper limits generously encompass the range of the wheelchair's tilt-->

Commit message: Changed axis of rotation for IMU joint

File: ada_description/urdf/ada.xacro (robot description, xacro)
@@ -23,5 +23,5 @@
     <child link="root_tilt" />
     <parent link="root" />
-    <axis xyz="1 0 0"/>
+    <axis xyz="-1 0 0"/>
     <!-- effort copied from j2n6s200 joint 2, velocity is max velocity the wheelchair can tilt,
     lower and upper limits generously encompass the range of the wheelchair's tilt-->

Commit message: Add sim to `ada_imu` (#16)
* Fix swapped parameter default value and parameter type

* Added sim param and launch arg

* Change logging severity

* Have MoveIt launch ada_imu by default, with the right sim mode

* Update README.md

* If reading from serial port fails, assume IMU angle of 0

* Changed axis of rotation for IMU joint

* Changed axis of rotation for IMU joint

* Update ada_imu/README.md

* Update ada_moveit/config/sensors_3d.yaml

* Update ada_watchdog_listener/ada_watchdog_listener/ada_watchdog_listener.py

---------

Co-authored-by: Haya Bolotski <hayabean@gmail.com>

File: ada_description/urdf/ada.xacro (robot description, xacro)
@@ -23,5 +23,5 @@
     <child link="root_tilt" />
     <parent link="root" />
-    <axis xyz="0 1 0"/>
+    <axis xyz="-1 0 0"/>
     <!-- effort copied from j2n6s200 joint 2, velocity is max velocity the wheelchair can tilt,
     lower and upper limits generously encompass the range of the wheelchair's tilt-->

Commit message: Added cartesian twist controller

File: ada_description/urdf/ada.xacro (robot description, xacro)
@@ -19,5 +19,5 @@
   <link name="root"/>
   <link name="root_tilt"/>
-  <joint name="robot_tilt" type="revolute">
+  <joint name="robot_tilt" type="fixed">
     <origin xyz="0 0 0" rpy="0 0 0" />
     <child link="root_tilt" />

Commit message: Return to revolute joint

File: ada_description/urdf/ada.xacro (robot description, xacro)
@@ -19,5 +19,5 @@
   <link name="root"/>
   <link name="root_tilt"/>
-  <joint name="robot_tilt" type="fixed">
+  <joint name="robot_tilt" type="revolute">
     <origin xyz="0 0 0" rpy="0 0 0" />
     <child link="root_tilt" />

Commit message: Added moment of inertia values for all remaining components and fixed top enclosure center of mass

File: ada_description/urdf/ada.xacro (robot description, xacro)
@@ -49,5 +49,5 @@
   -->
   <xacro:forque_assembly_link link_name="FTArmMount" link_mesh="2024_01_18_FTArmMount" mass="0.03783" cog="0.010957 -0.019223 -0.03777">
-    <xacro:insert_block name="default_inertial"/>
+    <inertia ixx="0.000018817" iyy="0.00001119989" iyz="-0.00000120296" izz="0.000026883" ixy="-0.0000003327" ixz="-0.000000092476"/>
   </xacro:forque_assembly_link>
   <xacro:forque_assembly_joint joint_name="FTArmMount_to_arm" parent="j2n6s200_link_6" child="FTArmMount" joint_origin_xyz="0.0065 -0.011 -0.0075" joint_origin_rpy="${J_PI/2} 0 ${J_PI/2}"/>

File: ada_description/urdf/camera/camera.xacro (robot description, xacro)
@@ -71,5 +71,5 @@
 	  	</xacro:camera_assembly_link>
 		<xacro:camera_assembly_joint joint_name="frontStabilizer_to_enclosureBottom" parent="enclosureBottom" child="frontStabilizer" joint_origin_xyz="0.1063 0.0493 -0.0363" joint_origin_rpy="0 0 ${J_PI/2}"/>
-		<xacro:camera_assembly_link link_name="enclosureTop" link_mesh="2023_06_06_nanoEnclosureTopCameraBack" mass="0.046" cog="0.04817211 0.03496864 0.02671124">
+		<xacro:camera_assembly_link link_name="enclosureTop" link_mesh="2023_06_06_nanoEnclosureTopCameraBack" mass="0.046" cog="0.041228 0.006275 0.016379">
 	  		<inertia ixx="0.00005942" iyy="0.000085611" iyz="0.0000012783" izz="0.000126390" ixy="-0.000000046193" ixz="0.0000091699"/>
 	  	</xacro:camera_assembly_link>
@@ -79,10 +79,10 @@
 	  	</xacro:camera_assembly_link>
 		<xacro:camera_assembly_joint joint_name="cameraMount_to_enclosureTop" parent="enclosureTop" child="cameraMount" joint_origin_xyz="-0.0132 0 -0.022" joint_origin_rpy="0 ${J_PI / 2} 0"/>
-		<xacro:camera_assembly_link link_name="screwHeadLeft" link_mesh="2023_11_07_screwHead" mass="0.0001" cog="0 0 0">
-     		<xacro:insert_block name="default_inertial"/>
+		<xacro:camera_assembly_link link_name="screwHeadLeft" link_mesh="2023_11_07_screwHead" mass="0.0001" cog="0 0 0.0015">
+     		<inertia ixx="0.000000000342785" iyy="0.000000000342785" iyz="0" izz="0.000000000543538" ixy="0" ixz="0"/>
      	</xacro:camera_assembly_link>
    	 	<xacro:camera_assembly_joint joint_name="screwHeadLeft_to_cameraMount" parent="cameraMount" child="screwHeadLeft" joint_origin_xyz="0.0165 -0.0225 0" joint_origin_rpy="${J_PI} 0 0"/>
-   	 	<xacro:camera_assembly_link link_name="screwHeadRight" link_mesh="2023_11_07_screwHead" mass="0.0001" cog="0 0 0">
-     		<xacro:insert_block name="default_inertial"/>
+   	 	<xacro:camera_assembly_link link_name="screwHeadRight" link_mesh="2023_11_07_screwHead" mass="0.0001" cog="0 0 0.0015">
+     		<inertia ixx="0.000000000342785" iyy="0.000000000342785" iyz="0" izz="0.000000000543538" ixy="0" ixz="0"/>
      	</xacro:camera_assembly_link>
    	 	<xacro:camera_assembly_joint joint_name="screwHeadRight_to_cameraMount" parent="cameraMount" child="screwHeadRight" joint_origin_xyz="0.0165 0.0225 0" joint_origin_rpy="${J_PI} 0 0"/>

File: ada_description/urdf/camera/d415urdf.xacro (robot description, xacro)
@@ -80,8 +80,7 @@
       </collision>
       <inertial>
-        <mass value="0.072" />
-        <!-- The following are not reliable values, and should not be used for modeling -->
-        <origin xyz="0 0 0" />
-        <inertia ixx="0.003881243" ixy="0.0" ixz="0.0" iyy="0.000498940" iyz="0.0" izz="0.003879257" />
+        <mass value="0.0589" /> <!-- manufacturer's value: 0.072 -->
+        <origin xyz="0 -0.02 0" />
+        <inertia ixx="0.00005491" ixy="-0.0000000249492" ixz="0.00000004862028" iyy="0.00000521068" iyz="0.00000000857625" izz="0.0000554597" />
       </inertial>
     </link>

File: ada_description/urdf/forque/forque.xacro (robot description, xacro)
@@ -52,11 +52,13 @@
 		</joint>
 	</xacro:macro>
+	<!-- <inertia ixx="" iyy="" iyz="" izz="" ixy="" ixz=""/>
+	-->
 	<xacro:macro name="forque_assembly" params="base_parent use_antenna:=false">
 		<xacro:forque_assembly_link link_name="FTMount" link_mesh="2024_01_18_FTMount" mass="0.103" cog="0.010934 -0.138522 -0.05066">
-			<xacro:insert_block name="default_inertial"/>
+			<inertia ixx="0.00017623" iyy="0.000068428" iyz="-0.00001757133" izz="0.00021455" ixy="0.00000095729" ixz="-0.0000000562908"/>
         </xacro:forque_assembly_link>
 	  	<xacro:forque_assembly_joint joint_name="FTMount_to_world" parent="${base_parent}" child="FTMount" joint_origin_xyz="0 0 -0.005" joint_origin_rpy="0 0 0"/>
 	  	<xacro:forque_assembly_link link_name="FT" link_mesh="2023_03_09_wirelessFT" mass="0.280" cog="0.0111446 -0.0882070 -0.0544936">
-	  		<xacro:insert_block name="default_inertial"/>
+	  		<inertia ixx="0.000543925" iyy="0.000165428" iyz="-0.00000001487288" izz="0.000691232" ixy="-0.00000128367" ixz="0"/>
 	  	</xacro:forque_assembly_link>
 	  	<xacro:forque_assembly_joint joint_name="FT_to_FTMount" parent="FTMount" child="FT" joint_origin_xyz="0 0 0" joint_origin_rpy="0 0 0"/>
@@ -68,14 +70,14 @@
 		  </xacro:if>
 	  	<xacro:forque_assembly_link link_name="forkHandle" link_mesh="2023_03_09_forkHandle" mass="0.0506" cog="0.0110024 -0.151715 -0.00934664">
-	  		<xacro:insert_block name="default_inertial"/>
+	  		<inertia ixx="0.0000418078" iyy="0.0000177249" iyz="-0.000000210639" izz="0.00005200336" ixy="-0.000000396292" ixz="0.00000002424697"/>
 	  	</xacro:forque_assembly_link>
 		<!-- The slight rotation was manually added due to empirical deformations in the robot gripped, such that the fingers and fork handle were slightly pitched up relative to the wrist. -->
 		<xacro:forque_assembly_joint joint_name="forkHandle_to_FTMount" parent="FTMount" child="forkHandle" joint_origin_xyz="0 0 0.005" joint_origin_rpy="-0.025 0 0"/>
 	  	<xacro:forque_assembly_link link_name="forque" link_mesh="ATI-9105-TW-NANO25-E" mass="0.0634" cog="0.0124692 0.0137169 0.010558">
-	  		<xacro:insert_block name="default_inertial"/>
+	  		<inertia ixx="0.000005235822" iyy="0.000006264852" iyz="-0.00000004033694" izz="0.00000640797" ixy="-0.0000003129932" ixz="0.000000013798"/>
 	  	</xacro:forque_assembly_link>
 	  	<xacro:forque_assembly_joint joint_name="forque_to_forkHandle" parent="forkHandle" child="forque" joint_origin_xyz="-0.00634 -0.222553 -0.004286" joint_origin_rpy="${J_PI/2} ${J_PI/3} 0"/>
 	  	<xacro:forque_assembly_link link_name="forkTine" link_mesh="fork_tine" mass="0.024" cog="0.013090 0.0180789 0.0445231">
-	  		<xacro:insert_block name="default_inertial"/>
+	  		<inertia ixx="0.0000098769" iyy="0.000009848103" iyz="0.00000057639" izz="0.0000015674" ixy="0.000000000806182" ixz="-0.00000000296036"/>
 	  	</xacro:forque_assembly_link>
 	  	<xacro:forque_assembly_joint joint_name="forkTine_to_forque" parent="forque" child="forkTine" joint_origin_xyz="-0.0054 0.008 0.093" joint_origin_rpy="0 ${J_PI} ${240*J_PI/180}"/>

Commit message: Changed FTSensor link to be a child of the forque

File: ada_description/urdf/ada.xacro (robot description, xacro)
@@ -57,6 +57,6 @@
     <joint name="EE_to_FTSensor" type="fixed">
         <child link="FTSensor"/>
-        <parent link="j2n6s200_end_effector"/>
-        <origin rpy="0 0 0" xyz="0.0 0.0 0.092"/>
+        <parent link="forque"/>
+        <origin rpy="${-4*J_PI/6} ${-J_PI/2} ${J_PI/2}" xyz="0.0125095 0.01291 0.02159"/>
     </joint>
   </xacro:if>
