Commit message: Update forque_assembly_joint macro to allow fixed, revolute, and continuous joints

File: ada_description/urdf/ada.xacro (robot description, xacro)
@@ -48,8 +48,26 @@
   </joint>
   -->
-  <xacro:forque_assembly_link link_name="FTArmMount" link_mesh="2024_01_18_FTArmMount" mass="0.03783" cog="0.010957 -0.019223 -0.03777">
-    <inertia ixx="0.000018817" iyy="0.00001119989" iyz="-0.00000120296" izz="0.000026883" ixy="-0.0000003327" ixz="-0.000000092476"/>
+  <xacro:forque_assembly_link
+      link_name="FTArmMount"
+      link_mesh="2024_01_18_FTArmMount"
+      mass="0.03783"
+      cog="0.010957 -0.019223 -0.03777">
+    <inertia
+        ixx="0.000018817"
+        iyy="0.00001119989"
+        iyz="-0.00000120296"
+        izz="0.000026883"
+        ixy="-0.0000003327"
+        ixz="-0.000000092476"/>
   </xacro:forque_assembly_link>
-  <xacro:forque_assembly_joint joint_name="FTArmMount_to_arm" parent="j2n6s200_link_6" child="FTArmMount" joint_origin_xyz="0.0065 -0.011 -0.0075" joint_origin_rpy="${J_PI/2} 0 ${J_PI/2}"/>
+  <xacro:forque_assembly_joint
+      joint_name="FTArmMount_to_arm"
+      type="fixed"
+      parent="j2n6s200_link_6"
+      child="FTArmMount"
+      joint_axis_xyz="0 0 1"
+      joint_origin_xyz="0.0065 -0.011 -0.0075"
+      joint_origin_rpy="${J_PI/2} 0 ${J_PI/2}"
+      fixed="true"/>
   <xacro:if value="$(arg use_forque)">
     <xacro:forque_assembly base_parent="FTArmMount"/>

File: ada_description/urdf/forque/forque.xacro (robot description, xacro)
@@ -44,39 +44,205 @@
 		</link>
 	</xacro:macro>
-	<xacro:macro name="forque_assembly_joint" params="joint_name parent child joint_origin_xyz joint_origin_rpy">
-		<joint name="${joint_name}" type="fixed">
-			<parent link="${parent}"/>
-			<child link="${child}"/>
-			<axis xyz="0 0 1"/>
-			<origin xyz="${joint_origin_xyz}" rpy="${joint_origin_rpy}"/>
-		</joint>
+	<xacro:macro name="forque_assembly_joint" params="joint_name
+                                                      type
+                                                      parent
+                                                      child
+                                                      joint_axis_xyz
+                                                      joint_origin_xyz
+                                                      joint_origin_rpy
+                                                      joint_lower_limit:=${dummy_default_value}
+                                                      joint_upper_limit:=${dummy_default_value}
+                                                      joint_velocity_limit:=${dummy_default_value}
+                                                      joint_torque_limit:=${dummy_default_value}
+                                                      fixed:=false">
+        <xacro:if value="${(type == 'fixed' and not fixed) or (type != 'fixed' and fixed)}">
+            <xacro:ERROR_inconsistent_joint_type_specification/>
+        </xacro:if>
+        <xacro:if value="${type == 'revolute'}">
+            <xacro:if value="${joint_lower_limit == dummy_default_value}">
+                <xacro:ERROR_joint_lower_limit_needs_to_be_set_for_a_revolute_joint/>
+            </xacro:if>
+            <xacro:if value="${joint_upper_limit == dummy_default_value}">
+                <xacro:ERROR_joint_upper_limit_needs_to_be_set_for_a_revolute_joint/>
+            </xacro:if>
+        </xacro:if>
+        <xacro:unless value="${type =='fixed'}">
+            <xacro:if value="${joint_velocity_limit == dummy_default_value}">
+                <xacro:ERROR_joint_velocity_limit_needs_to_be_set_for_a_non_fixed_joint/>
+            </xacro:if>
+            <xacro:if value="${joint_torque_limit == dummy_default_value}">
+                <xacro:ERROR_joint_torque_limit_needs_to_be_set_for_a_non_fixed_joint/>
+            </xacro:if>
+        </xacro:unless>
+        <joint name="${joint_name}" type="${type}">
+            <parent link="${parent}"/>
+            <child link="${child}"/>
+            <axis xyz="${joint_axis_xyz}"/>
+            <xacro:if value="${type == 'revolute'}">
+                <limit
+                    effort="${joint_torque_limit}"
+                    velocity="${joint_velocity_limit}"
+                    lower="${joint_lower_limit}"
+                    upper="${joint_upper_limit}"/>
+            </xacro:if>
+            <xacro:if value="${type == 'continuous'}">
+                <limit effort="${joint_torque_limit}" velocity="${joint_velocity_limit}"/>
+            </xacro:if>
+            <origin xyz="${joint_origin_xyz}" rpy="${joint_origin_rpy}"/>
+            <dynamics damping="0.0" friction="0.0"/>
+        </joint>
+        <xacro:unless value="${fixed}">
+            <transmission name="${joint_name}_trans">
+                <type>transmission_interface/SimpleTransmission</type>
+                <joint name="${joint_name}">
+                    <hardwareInterface>hardware_interface/EffortJointInterface</hardwareInterface>
+                </joint>
+                <actuator name="${joint_name}_actuator">
+                    <hardwareInterface>hardware_interface/EffortJointInterface</hardwareInterface>
+                    <mechanicalReduction>160</mechanicalReduction>
+                </actuator>
+            </transmission>
+            <!--For torque sensing in simulation-->
+            <gazebo reference="${joint_name}">
+                <provideFeedback>true</provideFeedback>
+            </gazebo>
+            <gazebo>
+                <plugin name="ft_sensor" filename="libgazebo_ros_ft_sensor.so">
+                    <updateRate>30.0</updateRate>
+                    <topicName>${joint_name}_ft_sensor_topic</topicName>
+                    <jointName>${joint_name}</jointName>
+                </plugin>
+            </gazebo>
+        </xacro:unless>
 	</xacro:macro>
 	<xacro:macro name="forque_assembly" params="base_parent use_antenna:=false">
-		<xacro:forque_assembly_link link_name="FTMount" link_mesh="2024_01_18_FTMount" mass="0.103" cog="0.010934 -0.138522 -0.05066">
-			<inertia ixx="0.00017623" iyy="0.000068428" iyz="-0.00001757133" izz="0.00021455" ixy="0.00000095729" ixz="-0.0000000562908"/>
+		<xacro:forque_assembly_link
+            link_name="FTMount"
+            link_mesh="2024_01_18_FTMount"
+            mass="0.103"
+            cog="0.010934 -0.138522 -0.05066">
+			<inertia
+                ixx="0.00017623"
+                iyy="0.000068428"
+                iyz="-0.00001757133"
+                izz="0.00021455"
+                ixy="0.00000095729"
+                ixz="-0.0000000562908"/>
         </xacro:forque_assembly_link>
-	  	<xacro:forque_assembly_joint joint_name="FTMount_to_world" parent="${base_parent}" child="FTMount" joint_origin_xyz="0 0 -0.005" joint_origin_rpy="0 0 0"/>
-	  	<xacro:forque_assembly_link link_name="FT" link_mesh="2023_03_09_wirelessFT" mass="0.280" cog="0.0111446 -0.0882070 -0.0544936">
-	  		<inertia ixx="0.000543925" iyy="0.000165428" iyz="-0.00000001487288" izz="0.000691232" ixy="-0.00000128367" ixz="0"/>
-	  	</xacro:forque_assembly_link>
-	  	<xacro:forque_assembly_joint joint_name="FT_to_FTMount" parent="FTMount" child="FT" joint_origin_xyz="0 0 0" joint_origin_rpy="0 0 0"/>
+	  	<xacro:forque_assembly_joint
+            joint_name="FTMount_to_world"
+            type="fixed"
+            parent="${base_parent}"
+            child="FTMount"
+            joint_axis_xyz="0 0 1"
+            joint_origin_xyz="0 0 -0.005"
+            joint_origin_rpy="0 0 0"
+            fixed="true"/>
+	  	<xacro:forque_assembly_link
+            link_name="FT"
+            link_mesh="2023_03_09_wirelessFT"
+            mass="0.280"
+            cog="0.0111446 -0.0882070 -0.0544936">
+	  		<inertia
+                ixx="0.000543925"
+                iyy="0.000165428"
+                iyz="-0.00000001487288"
+                izz="0.000691232"
+                ixy="-0.00000128367"
+                ixz="0"/>
+	  	</xacro:forque_assembly_link>
+	  	<xacro:forque_assembly_joint
+            joint_name="FT_to_FTMount"
+            type="fixed"
+            parent="FTMount"
+            child="FT"
+            joint_axis_xyz="0 0 1"
+            joint_origin_xyz="0 0 0"
+            joint_origin_rpy="0 0 0"
+            fixed="true"/>
 	  	<xacro:if value="${use_antenna}">
-		  	<xacro:forque_assembly_link link_name="FTAntenna" link_mesh="2023_03_09_wirelessFTAntenna" mass="0.018" cog="-0.0162965 0.0666626 -0.0545096">
-	  		  <xacro:insert_block name="default_inertial"/>
-	  	  </xacro:forque_assembly_link>
-	  	  <xacro:forque_assembly_joint joint_name="FTAntenna_to_FT" parent="FT" child="FTAntenna" joint_origin_xyz="0 0 0" joint_origin_rpy="0 0 0"/>
-		  </xacro:if>
-	  	<xacro:forque_assembly_link link_name="forkHandle" link_mesh="2023_03_09_forkHandle" mass="0.0506" cog="0.0110024 -0.151715 -0.00934664">
-	  		<inertia ixx="0.0000418078" iyy="0.0000177249" iyz="-0.000000210639" izz="0.00005200336" ixy="-0.000000396292" ixz="0.00000002424697"/>
-	  	</xacro:forque_assembly_link>
-		<xacro:forque_assembly_joint joint_name="forkHandle_to_FTMount" parent="FTMount" child="forkHandle" joint_origin_xyz="0 0 0" joint_origin_rpy="-0.025 0 0"/>
-	  	<xacro:forque_assembly_link link_name="forque" link_mesh="ATI-9105-TW-NANO25-E" mass="0.0634" cog="0.0124692 0.0137169 0.010558">
-	  		<inertia ixx="0.000005235822" iyy="0.000006264852" iyz="-0.00000004033694" izz="0.00000640797" ixy="-0.0000003129932" ixz="0.000000013798"/>
-	  	</xacro:forque_assembly_link>
-	  	<xacro:forque_assembly_joint joint_name="forque_to_forkHandle" parent="forkHandle" child="forque" joint_origin_xyz="-0.00634 -0.222553 -0.004286" joint_origin_rpy="${J_PI/2} ${J_PI/3} 0"/>
-	  	<xacro:forque_assembly_link link_name="forkTine" link_mesh="fork_tine" mass="0.024" cog="0.013090 0.0180789 0.0445231">
-	  		<inertia ixx="0.0000098769" iyy="0.000009848103" iyz="0.00000057639" izz="0.0000015674" ixy="0.000000000806182" ixz="-0.00000000296036"/>
-	  	</xacro:forque_assembly_link>
-	  	<xacro:forque_assembly_joint joint_name="forkTine_to_forque" parent="forque" child="forkTine" joint_origin_xyz="-0.0054 0.008 0.093" joint_origin_rpy="0 ${J_PI} ${240*J_PI/180}"/>
+            <xacro:forque_assembly_link
+                link_name="FTAntenna"
+                link_mesh="2023_03_09_wirelessFTAntenna"
+                mass="0.018"
+                cog="-0.0162965 0.0666626 -0.0545096">
+                <xacro:insert_block name="default_inertial"/>
+            </xacro:forque_assembly_link>
+    	  	<xacro:forque_assembly_joint
+                joint_name="FTAntenna_to_FT"
+                type="fixed"
+                parent="FT"
+                child="FTAntenna"
+                joint_axis_xyz="0 0 1"
+                joint_origin_xyz="0 0 0"
+                joint_origin_rpy="0 0 0"
+                fixed="true"/>
+		</xacro:if>
+	  	<xacro:forque_assembly_link
+            link_name="forkHandle"
+            link_mesh="2023_03_09_forkHandle"
+            mass="0.0506"
+            cog="0.0110024 -0.151715 -0.00934664">
+	  		<inertia
+                ixx="0.0000418078"
+                iyy="0.0000177249"
+                iyz="-0.000000210639"
+                izz="0.00005200336"
+                ixy="-0.000000396292"
+                ixz="0.00000002424697"/>
+	  	</xacro:forque_assembly_link>
+		<xacro:forque_assembly_joint
+            joint_name="forkHandle_to_FTMount"
+            type="fixed"
+            parent="FTMount"
+            child="forkHandle"
+            joint_axis_xyz="0 0 1"
+            joint_origin_xyz="0 0 0"
+            joint_origin_rpy="-0.025 0 0"
+            fixed="true"/>
+	  	<xacro:forque_assembly_link
+            link_name="forque"
+            link_mesh="ATI-9105-TW-NANO25-E"
+            mass="0.0634"
+            cog="0.0124692 0.0137169 0.010558">
+	  		<inertia
+                ixx="0.000005235822"
+                iyy="0.000006264852"
+                iyz="-0.00000004033694"
+                izz="0.00000640797"
+                ixy="-0.0000003129932"
+                ixz="0.000000013798"/>
+	  	</xacro:forque_assembly_link>
+	  	<xacro:forque_assembly_joint
+            joint_name="forque_to_forkHandle"
+            type="fixed"
+            parent="forkHandle"
+            child="forque"
+            joint_axis_xyz="0 0 1"
+            joint_origin_xyz="-0.00634 -0.222553 -0.004286"
+            joint_origin_rpy="${J_PI/2} ${J_PI/3} 0"
+            fixed="true"/>
+	  	<xacro:forque_assembly_link
+            link_name="forkTine"
+            link_mesh="fork_tine"
+            mass="0.024"
+            cog="0.013090 0.0180789 0.0445231">
+	  		<inertia
+                ixx="0.0000098769"
+                iyy="0.000009848103"
+                iyz="0.00000057639"
+                izz="0.0000015674"
+                ixy="0.000000000806182"
+                ixz="-0.00000000296036"/>
+	  	</xacro:forque_assembly_link>
+	  	<xacro:forque_assembly_joint
+            joint_name="forkTine_to_forque"
+            type="fixed"
+            parent="forque"
+            child="forkTine"
+            joint_axis_xyz="0 0 1"
+            joint_origin_xyz="-0.0054 0.008 0.093"
+            joint_origin_rpy="0 ${J_PI} ${240*J_PI/180}"
+            fixed="true"/>
 	  	<link name="forkTip" />
 	  	<joint name="forkTip_to_forkTine" type="fixed">

Commit message: Add end_effector_tool configuration, remove use_forque configuration

File: ada_description/urdf/ada.xacro (robot description, xacro)
@@ -16,5 +16,6 @@
   <xacro:include filename="$(find ada_description)/urdf/camera/camera.xacro"/>
   <xacro:include filename="$(find ada_description)/urdf/j2n6s200.xacro"/>
-  <xacro:arg name="use_forque" default="true"/>
+  <xacro:arg name="end_effector_tool" default="fork"/>
+  <xacro:property name="cmp_end_effector_tool" value="$(arg end_effector_tool)"/>
   <link name="root"/>
   <link name="root_tilt"/>
@@ -70,5 +71,5 @@
       joint_origin_rpy="${J_PI/2} 0 ${J_PI/2}"
       fixed="true"/>
-  <xacro:if value="$(arg use_forque)">
+  <xacro:unless value="${cmp_end_effector_tool == 'none'}">
     <xacro:forque_assembly base_parent="FTArmMount"/>
     <link name="FTSensor" />
@@ -78,4 +79,4 @@
         <origin rpy="0 0 0" xyz="0.0 0.0 0.092"/>
     </joint>
-  </xacro:if>
+  </xacro:unless>
 </robot>
