Commit message: Conditionally modify fork URDF based on end_effector_tool

File: ada_description/urdf/ada.xacro (robot description, xacro)
@@ -72,5 +72,5 @@
       fixed="true"/>
   <xacro:unless value="${cmp_end_effector_tool == 'none'}">
-    <xacro:forque_assembly base_parent="FTArmMount"/>
+    <xacro:forque_assembly base_parent="FTArmMount" end_effector_tool="${cmp_end_effector_tool}"/>
     <link name="FTSensor" />
     <joint name="EE_to_FTSensor" type="fixed">

File: ada_description/urdf/forque/forque.xacro (robot description, xacro)
@@ -120,5 +120,5 @@
         </xacro:unless>
 	</xacro:macro>
-	<xacro:macro name="forque_assembly" params="base_parent use_antenna:=false">
+	<xacro:macro name="forque_assembly" params="base_parent end_effector_tool use_antenna:=false">
 		<xacro:forque_assembly_link
             link_name="FTMount"
@@ -205,104 +205,106 @@
             joint_origin_rpy="-0.025 0 0"
             fixed="true"/>
-        <xacro:forque_assembly_link
-            link_name="af_link_base"
-            link_mesh="fr12-h103"
-            mass="0.0907185"
-            cog="0.0 0.0 0.0">
-            <xacro:insert_block name="default_inertial"/>
-        </xacro:forque_assembly_link>
-        <xacro:forque_assembly_joint
-            joint_name="af_joint_base"
-            type="fixed"
-            parent="forkHandle"
-            child="af_link_base"
-            joint_axis_xyz="0 0 1"
-            joint_origin_xyz="0.010929196 -0.278553 -0.011"
-            joint_origin_rpy="0 0 0"
-            fixed="true"/>
-        <xacro:forque_assembly_link
-            link_name="af_link_1"
-            link_mesh="XC-430_idle"
-            mass="0.065"
-            cog="0.21641853 -14.751192 -16.796092">
-            <inertia
-                ixx="18680.931"
-                iyy="9585.9138"
-                iyz="-845.46678"
-                izz="17346.641"
-                ixy="1.3348619"
-                ixz="-45.354028"/>
-        </xacro:forque_assembly_link>
-        <xacro:forque_assembly_joint
-            joint_name="af_joint_1"
-            type="revolute"
-            parent="af_link_base"
-            child="af_link_1"
-            joint_axis_xyz="0 0 1"
-            joint_origin_xyz="0 0 0"
-            joint_origin_rpy="${J_PI/2} 0 ${J_PI/2}"
-            joint_lower_limit="${-J_PI/2}"
-            joint_upper_limit="${J_PI/2}"
-            joint_velocity_limit="1"
-            joint_torque_limit="1.4"
-            fixed="false"/>
-        <xacro:forque_assembly_link
-            link_name="af_motor_fixture_link"
-            link_mesh="fr12-s101"
-            mass="0.0453592"
-            cog="0 0 0">
-            <xacro:insert_block name="default_inertial"/>
-        </xacro:forque_assembly_link>
-        <xacro:forque_assembly_joint
-            joint_name="af_motor_fixture_joint_1"
-            type="fixed"
-            parent="af_link_1"
-            child="af_motor_fixture_link"
-            joint_axis_xyz="0 0 1"
-            joint_origin_xyz="0 0 0"
-            joint_origin_rpy="0 ${-J_PI/2} 0"
-            fixed="true"/>
-        <xacro:forque_assembly_link
-            link_name="af_link_2"
-            link_mesh="XC-430_idle"
-            mass="0.065"
-            cog="0.21641853 -14.751192 -16.796092">
-            <inertia
-                ixx="18680.931"
-                iyy="9585.9138"
-                iyz="-845.46678"
-                izz="17346.641"
-                ixy="1.3348619"
-                ixz="-45.354028"/>
-        </xacro:forque_assembly_link>
-        <xacro:forque_assembly_joint
-            joint_name="af_motor_fixture_joint_2"
-            type="fixed"
-            parent="af_link_1"
-            child="af_link_2"
-            joint_axis_xyz="0 0 1"
-            joint_origin_xyz="-0.03825 0 0"
-            joint_origin_rpy="0 ${-J_PI/2} 0"
-            fixed="true"/>
-        <xacro:forque_assembly_link
-            link_name="af_ft_adapter_link"
-            link_mesh="roll_to_ft_adapter"
-            mass="0.001"
-            cog="0 0 0">
-            <xacro:insert_block name="default_inertial"/>
-        </xacro:forque_assembly_link>
-        <xacro:forque_assembly_joint
-            joint_name="af_joint_2"
-            type="revolute"
-            parent="af_link_2"
-            child="af_ft_adapter_link"
-            joint_axis_xyz="0 1 0"
-            joint_origin_xyz="0 0 0.019"
-            joint_origin_rpy="${-J_PI/2} 0 0"
-            joint_lower_limit="${-J_PI}"
-            joint_upper_limit="${J_PI}"
-            joint_velocity_limit="1"
-            joint_torque_limit="1.4"
-            fixed="false"/>
+      <xacro:if value="${end_effector_tool == 'articulable_fork'}">
+          <xacro:forque_assembly_link
+              link_name="af_link_base"
+              link_mesh="fr12-h103"
+              mass="0.0907185"
+              cog="0.0 0.0 0.0">
+              <xacro:insert_block name="default_inertial"/>
+          </xacro:forque_assembly_link>
+          <xacro:forque_assembly_joint
+              joint_name="af_joint_base"
+              type="fixed"
+              parent="forkHandle"
+              child="af_link_base"
+              joint_axis_xyz="0 0 1"
+              joint_origin_xyz="0.010929196 -0.278553 -0.011"
+              joint_origin_rpy="0 0 0"
+              fixed="true"/>
+          <xacro:forque_assembly_link
+              link_name="af_link_1"
+              link_mesh="XC-430_idle"
+              mass="0.065"
+              cog="0.21641853 -14.751192 -16.796092">
+              <inertia
+                  ixx="18680.931"
+                  iyy="9585.9138"
+                  iyz="-845.46678"
+                  izz="17346.641"
+                  ixy="1.3348619"
+                  ixz="-45.354028"/>
+          </xacro:forque_assembly_link>
+          <xacro:forque_assembly_joint
+              joint_name="af_joint_1"
+              type="revolute"
+              parent="af_link_base"
+              child="af_link_1"
+              joint_axis_xyz="0 0 1"
+              joint_origin_xyz="0 0 0"
+              joint_origin_rpy="${J_PI/2} 0 ${J_PI/2}"
+              joint_lower_limit="${-J_PI/2}"
+              joint_upper_limit="${J_PI/2}"
+              joint_velocity_limit="1"
+              joint_torque_limit="1.4"
+              fixed="false"/>
+          <xacro:forque_assembly_link
+              link_name="af_motor_fixture_link"
+              link_mesh="fr12-s101"
+              mass="0.0453592"
+              cog="0 0 0">
+              <xacro:insert_block name="default_inertial"/>
+          </xacro:forque_assembly_link>
+          <xacro:forque_assembly_joint
+              joint_name="af_motor_fixture_joint_1"
+              type="fixed"
+              parent="af_link_1"
+              child="af_motor_fixture_link"
+              joint_axis_xyz="0 0 1"
+              joint_origin_xyz="0 0 0"
+              joint_origin_rpy="0 ${-J_PI/2} 0"
+              fixed="true"/>
+          <xacro:forque_assembly_link
+              link_name="af_link_2"
+              link_mesh="XC-430_idle"
+              mass="0.065"
+              cog="0.21641853 -14.751192 -16.796092">
+              <inertia
+                  ixx="18680.931"
+                  iyy="9585.9138"
+                  iyz="-845.46678"
+                  izz="17346.641"
+                  ixy="1.3348619"
+                  ixz="-45.354028"/>
+          </xacro:forque_assembly_link>
+          <xacro:forque_assembly_joint
+              joint_name="af_motor_fixture_joint_2"
+              type="fixed"
+              parent="af_link_1"
+              child="af_link_2"
+              joint_axis_xyz="0 0 1"
+              joint_origin_xyz="-0.03825 0 0"
+              joint_origin_rpy="0 ${-J_PI/2} 0"
+              fixed="true"/>
+          <xacro:forque_assembly_link
+              link_name="af_ft_adapter_link"
+              link_mesh="roll_to_ft_adapter"
+              mass="0.001"
+              cog="0 0 0">
+              <xacro:insert_block name="default_inertial"/>
+          </xacro:forque_assembly_link>
+          <xacro:forque_assembly_joint
+              joint_name="af_joint_2"
+              type="revolute"
+              parent="af_link_2"
+              child="af_ft_adapter_link"
+              joint_axis_xyz="0 1 0"
+              joint_origin_xyz="0 0 0.019"
+              joint_origin_rpy="${-J_PI/2} 0 0"
+              joint_lower_limit="${-J_PI}"
+              joint_upper_limit="${J_PI}"
+              joint_velocity_limit="1"
+              joint_torque_limit="1.4"
+              fixed="false"/>
+      </xacro:if>
 	  	<xacro:forque_assembly_link
             link_name="forque"
@@ -318,13 +320,26 @@
                 ixz="0.000000013798"/>
 	  	</xacro:forque_assembly_link>
-	  	<xacro:forque_assembly_joint
-            joint_name="af_forque_joint"
-            type="fixed"
-            parent="af_ft_adapter_link"
-            child="forque"
-            joint_axis_xyz="0 0 1"
-            joint_origin_xyz="-0.0175 -0.011 0.004"
-            joint_origin_rpy="${J_PI/2} ${J_PI/3} 0"
-            fixed="true"/>
+      <xacro:if value="${end_effector_tool == 'articulable_fork'}">
+          <xacro:forque_assembly_joint
+                joint_name="af_forque_joint"
+                type="fixed"
+                parent="af_ft_adapter_link"
+                child="forque"
+                joint_axis_xyz="0 0 1"
+                joint_origin_xyz="-0.0175 -0.011 0.004"
+                joint_origin_rpy="${J_PI/2} ${J_PI/3} 0"
+                fixed="true"/>
+      </xacro:if>
+      <xacro:if value="${end_effector_tool == 'fork'}">
+          <xacro:forque_assembly_joint
+                joint_name="forque_to_forkHandle"
+                type="fixed"
+                parent="forkHandle"
+                child="forque"
+                joint_axis_xyz="0 0 1"
+                joint_origin_xyz="-0.00634 -0.222553 -0.004286"
+                joint_origin_rpy="${J_PI/2} ${J_PI/3} 0"
+                fixed="true"/>
+      </xacro:if>
 	  	<xacro:forque_assembly_link
             link_name="forkTine"

Commit message: More formatting

File: ada_description/urdf/ada.xacro (robot description, xacro)
@@ -49,26 +49,8 @@
   </joint>
   -->
-  <xacro:forque_assembly_link
-      link_name="FTArmMount"
-      link_mesh="2024_01_18_FTArmMount"
-      mass="0.03783"
-      cog="0.010957 -0.019223 -0.03777">
-    <inertia
-        ixx="0.000018817"
-        iyy="0.00001119989"
-        iyz="-0.00000120296"
-        izz="0.000026883"
-        ixy="-0.0000003327"
-        ixz="-0.000000092476"/>
+  <xacro:forque_assembly_link link_name="FTArmMount" link_mesh="2024_01_18_FTArmMount" mass="0.03783" cog="0.010957 -0.019223 -0.03777">
+    <inertia ixx="0.000018817" iyy="0.00001119989" iyz="-0.00000120296" izz="0.000026883" ixy="-0.0000003327" ixz="-0.000000092476"/>
   </xacro:forque_assembly_link>
-  <xacro:forque_assembly_joint
-      joint_name="FTArmMount_to_arm"
-      type="fixed"
-      parent="j2n6s200_link_6"
-      child="FTArmMount"
-      joint_axis_xyz="0 0 1"
-      joint_origin_xyz="0.0065 -0.011 -0.0075"
-      joint_origin_rpy="${J_PI/2} 0 ${J_PI/2}"
-      fixed="true"/>
+  <xacro:forque_assembly_joint joint_name="FTArmMount_to_arm" type="fixed" parent="j2n6s200_link_6" child="FTArmMount" joint_axis_xyz="0 0 1" joint_origin_xyz="0.0065 -0.011 -0.0075" joint_origin_rpy="${J_PI/2} 0 ${J_PI/2}" fixed="true"/>
   <xacro:unless value="${cmp_end_effector_tool == 'none'}">
     <xacro:forque_assembly base_parent="FTArmMount" end_effector_tool="${cmp_end_effector_tool}"/>

File: ada_description/urdf/forque/forque.xacro (robot description, xacro)
@@ -163,5 +163,5 @@
 	  	</xacro:forque_assembly_link>
 	  	<xacro:forque_assembly_joint joint_name="forkTine_to_forque" type="fixed" parent="forque" child="forkTine" joint_axis_xyz="0 0 1" joint_origin_xyz="-0.0054 0.008 0.093" joint_origin_rpy="0 ${J_PI} ${240*J_PI/180}" fixed="true"/>
-	  	<link name="forkTip"/>
+	  	<link name="forkTip" />
 	  	<joint name="forkTip_to_forkTine" type="fixed">
 		    <child link="forkTip"/>

Commit message: Decouple ADAs description into a macro that is explicitly instantiated in ada_standalone.xacro

File: ada_description/urdf/ada.xacro (robot description, xacro)
@@ -12,53 +12,52 @@
     xmlns:renderable="http://playerstage.sourceforge.net/gazebo/xmlschema/#renderable"
     xmlns:physics="http://playerstage.sourceforge.net/gazebo/xmlschema/#physics"
-  xmlns:xacro="http://www.ros.org/wiki/xacro" name="ada">
-  <xacro:include filename="$(find ada_description)/urdf/forque/forque.xacro"/>
-  <xacro:include filename="$(find ada_description)/urdf/camera/camera.xacro"/>
-  <xacro:include filename="$(find ada_description)/urdf/j2n6s200.xacro"/>
-  <xacro:arg name="end_effector_tool" default="fork"/>
-  <xacro:property name="cmp_end_effector_tool" value="$(arg end_effector_tool)"/>
-  <link name="root"/>
-  <link name="root_tilt"/>
-  <joint name="robot_tilt" type="revolute">
-    <origin xyz="0 0 0" rpy="0 0 0" />
-    <child link="root_tilt" />
-    <parent link="root" />
-    <axis xyz="-1 0 0"/>
-    <!-- effort copied from j2n6s200 joint 2, velocity is max velocity the wheelchair can tilt,
-    lower and upper limits generously encompass the range of the wheelchair's tilt-->
-    <limit effort="80" velocity="0.15" lower="${-J_PI}" upper="${J_PI}"/>
-    <dynamics damping="0.0" friction="0.0"/>
-  </joint>
-  <xacro:property name="robot_root" value="root_tilt" />
-  <xacro:j2n6s200 base_parent="${robot_root}"/>
-  <xacro:camera_assembly base_parent="j2n6s200_link_6" base_xyz="0.0165 0 0.0011" base_rpy="${3*J_PI/2} 0 ${3*J_PI/2}"/>
-  <!-- Hard-coded Extrinsics -->
-  <link name="camera_link" />
-  <joint name="extrinsics" type="fixed">
-    <origin xyz="0.0194 -0.01606 0.029014" rpy="0.17234 -1.56127 2.96967" />
-    <parent link="cameraMount" />
-    <child link="camera_link" />
-  </joint>
-  <!-- Copy Realsense in case of simulation -->
-  <!--
-  <link name="camera_color_optical_frame" />
-  <joint name="optical_republish" type="fixed">
-    <origin xyz="0.000 -0.015 0.000" rpy="-1.564 0.000 -1.573" />
-    <parent link="camera_link" />
-    <child link="camera_color_optical_frame" />
-  </joint>
-  -->
-  <xacro:forque_assembly_link link_name="FTArmMount" link_mesh="2024_01_18_FTArmMount" mass="0.03783" cog="0.010957 -0.019223 -0.03777">
-    <inertia ixx="0.000018817" iyy="0.00001119989" iyz="-0.00000120296" izz="0.000026883" ixy="-0.0000003327" ixz="-0.000000092476"/>
-  </xacro:forque_assembly_link>
-  <xacro:forque_assembly_joint joint_name="FTArmMount_to_arm" type="fixed" parent="j2n6s200_link_6" child="FTArmMount" joint_axis_xyz="0 0 1" joint_origin_xyz="0.0065 -0.011 -0.0075" joint_origin_rpy="${J_PI/2} 0 ${J_PI/2}" fixed="true"/>
-  <xacro:unless value="${cmp_end_effector_tool == 'none'}">
-    <xacro:forque_assembly base_parent="FTArmMount" end_effector_tool="${cmp_end_effector_tool}"/>
-    <link name="FTSensor" />
-    <joint name="EE_to_FTSensor" type="fixed">
-        <child link="FTSensor"/>
-        <parent link="j2n6s200_end_effector"/>
-        <origin rpy="0 0 0" xyz="0.0 0.0 0.092"/>
+  xmlns:xacro="http://www.ros.org/wiki/xacro">
+  <xacro:macro name="ada" params="base_parent end_effector_tool">
+    <xacro:include filename="$(find ada_description)/urdf/forque/forque.xacro"/>
+    <xacro:include filename="$(find ada_description)/urdf/camera/camera.xacro"/>
+    <xacro:include filename="$(find ada_description)/urdf/j2n6s200.xacro"/>
+    <link name="root_tilt"/>
+    <joint name="robot_tilt" type="revolute">
+      <origin xyz="0 0 0" rpy="0 0 0" />
+      <child link="root_tilt" />
+      <parent link="${base_parent}" />
+      <axis xyz="-1 0 0"/>
+      <!-- effort copied from j2n6s200 joint 2, velocity is max velocity the wheelchair can tilt,
+      lower and upper limits generously encompass the range of the wheelchair's tilt-->
+      <limit effort="80" velocity="0.15" lower="${-J_PI}" upper="${J_PI}"/>
+      <dynamics damping="0.0" friction="0.0"/>
     </joint>
-  </xacro:unless>
+    <xacro:property name="robot_root" value="root_tilt" />
+    <xacro:j2n6s200 base_parent="${robot_root}"/>
+    <xacro:camera_assembly base_parent="j2n6s200_link_6" base_xyz="0.0165 0 0.0011" base_rpy="${3*J_PI/2} 0 ${3*J_PI/2}"/>
+    <!-- Hard-coded Extrinsics -->
+    <link name="camera_link" />
+    <joint name="extrinsics" type="fixed">
+      <origin xyz="0.0194 -0.01606 0.029014" rpy="0.17234 -1.56127 2.96967" />
+      <parent link="cameraMount" />
+      <child link="camera_link" />
+    </joint>
+    <!-- Copy Realsense in case of simulation -->
+    <!--
+    <link name="camera_color_optical_frame" />
+    <joint name="optical_republish" type="fixed">
+      <origin xyz="0.000 -0.015 0.000" rpy="-1.564 0.000 -1.573" />
+      <parent link="camera_link" />
+      <child link="camera_color_optical_frame" />
+    </joint>
+    -->
+    <xacro:forque_assembly_link link_name="FTArmMount" link_mesh="2024_01_18_FTArmMount" mass="0.03783" cog="0.010957 -0.019223 -0.03777">
+      <inertia ixx="0.000018817" iyy="0.00001119989" iyz="-0.00000120296" izz="0.000026883" ixy="-0.0000003327" ixz="-0.000000092476"/>
+    </xacro:forque_assembly_link>
+    <xacro:forque_assembly_joint joint_name="FTArmMount_to_arm" type="fixed" parent="j2n6s200_link_6" child="FTArmMount" joint_axis_xyz="0 0 1" joint_origin_xyz="0.0065 -0.011 -0.0075" joint_origin_rpy="${J_PI/2} 0 ${J_PI/2}" fixed="true"/>
+    <xacro:unless value="${end_effector_tool == 'none'}">
+      <xacro:forque_assembly base_parent="FTArmMount" end_effector_tool="${end_effector_tool}"/>
+      <link name="FTSensor" />
+      <joint name="EE_to_FTSensor" type="fixed">
+          <child link="FTSensor"/>
+          <parent link="j2n6s200_end_effector"/>
+          <origin rpy="0 0 0" xyz="0.0 0.0 0.092"/>
+      </joint>
+    </xacro:unless>
+  </xacro:macro>
 </robot>

Commit message: Remove base_parent argument for ada macro, use root by default

File: ada_description/urdf/ada.xacro (robot description, xacro)
@@ -13,14 +13,15 @@
     xmlns:physics="http://playerstage.sourceforge.net/gazebo/xmlschema/#physics"
   xmlns:xacro="http://www.ros.org/wiki/xacro">
-  <xacro:macro name="ada" params="base_parent end_effector_tool">
+  <xacro:macro name="ada" params="end_effector_tool">
     <!-- Import macros associated with forque, robot, and camera. Macros are added to the tree below -->
     <xacro:include filename="$(find ada_description)/urdf/forque/forque.xacro"/>
     <xacro:include filename="$(find ada_description)/urdf/camera/camera.xacro"/>
     <xacro:include filename="$(find ada_description)/urdf/j2n6s200.xacro"/>
+    <link name="root"/>
     <link name="root_tilt"/>
     <joint name="robot_tilt" type="revolute">
       <origin xyz="0 0 0" rpy="0 0 0" />
       <child link="root_tilt" />
-      <parent link="${base_parent}" />
+      <parent link="root" />
       <axis xyz="-1 0 0"/>
       <!-- effort copied from j2n6s200 joint 2, velocity is max velocity the wheelchair can tilt,

File: ada_description/urdf/ada_standalone.xacro (robot description, xacro)
@@ -16,7 +16,6 @@
   <xacro:arg name="end_effector_tool" default="fork" />
   <xacro:include filename="$(find ada_description)/urdf/ada.xacro" />
-  <link name="root"/>
   <xacro:property name="root" value="root" />
   <xacro:property name="end_effector_tool" value="$(arg end_effector_tool)" />
-  <xacro:ada base_parent="${root}" end_effector_tool="${end_effector_tool}" />
+  <xacro:ada end_effector_tool="${end_effector_tool}" />
 </robot>
