Commit message: Remove broken error messages, remove fixed parameter for forque_assembly_joint

File: ada_description/urdf/ada.xacro (robot description, xacro)
@@ -52,5 +52,5 @@
       <inertia ixx="0.000018817" iyy="0.00001119989" iyz="-0.00000120296" izz="0.000026883" ixy="-0.0000003327" ixz="-0.000000092476"/>
     </xacro:forque_assembly_link>
-    <xacro:forque_assembly_joint joint_name="FTArmMount_to_arm" type="fixed" parent="j2n6s200_link_6" child="FTArmMount" joint_axis_xyz="0 0 1" joint_origin_xyz="0.0065 -0.011 -0.0075" joint_origin_rpy="${J_PI/2} 0 ${J_PI/2}" fixed="true"/>
+    <xacro:forque_assembly_joint joint_name="FTArmMount_to_arm" type="fixed" parent="j2n6s200_link_6" child="FTArmMount" joint_axis_xyz="0 0 1" joint_origin_xyz="0.0065 -0.011 -0.0075" joint_origin_rpy="${J_PI/2} 0 ${J_PI/2}"/>
     <xacro:unless value="${end_effector_tool == 'none'}">
       <xacro:forque_assembly base_parent="FTArmMount" end_effector_tool="${end_effector_tool}"/>

File: ada_description/urdf/forque/forque.xacro (robot description, xacro)
@@ -45,24 +45,5 @@
 		</link>
 	</xacro:macro>
-	<xacro:macro name="forque_assembly_joint" params="joint_name type parent child joint_axis_xyz joint_origin_xyz joint_origin_rpy joint_lower_limit:=${forque_assembly_dummy_default_value} joint_upper_limit:=${forque_assembly_dummy_default_value} joint_velocity_limit:=${forque_assembly_dummy_default_value} joint_torque_limit:=${forque_assembly_dummy_default_value} fixed:=false">
-    <xacro:if value="${(type == 'fixed' and not fixed) or (type != 'fixed' and fixed)}">
-      <xacro:ERROR_inconsistent_joint_type_specification/>
-    </xacro:if>
-    <xacro:if value="${type == 'revolute'}">
-      <xacro:if value="${joint_lower_limit == forque_assembly_dummy_default_value}">
-        <xacro:ERROR_joint_lower_limit_needs_to_be_set_for_a_revolute_joint/>
-      </xacro:if>
-      <xacro:if value="${joint_upper_limit == forque_assembly_dummy_default_value}">
-        <xacro:ERROR_joint_upper_limit_needs_to_be_set_for_a_revolute_joint/>
-      </xacro:if>
-    </xacro:if>
-    <xacro:unless value="${type =='fixed'}">
-      <xacro:if value="${joint_velocity_limit == forque_assembly_dummy_default_value}">
-        <xacro:ERROR_joint_velocity_limit_needs_to_be_set_for_a_non_fixed_joint/>
-      </xacro:if>
-      <xacro:if value="${joint_torque_limit == forque_assembly_dummy_default_value}">
-        <xacro:ERROR_joint_torque_limit_needs_to_be_set_for_a_non_fixed_joint/>
-      </xacro:if>
-    </xacro:unless>
+	<xacro:macro name="forque_assembly_joint" params="joint_name type parent child joint_axis_xyz joint_origin_xyz joint_origin_rpy joint_lower_limit:=${forque_assembly_dummy_default_value} joint_upper_limit:=${forque_assembly_dummy_default_value} joint_velocity_limit:=${forque_assembly_dummy_default_value} joint_torque_limit:=${forque_assembly_dummy_default_value}">
     <joint name="${joint_name}" type="${type}">
       <parent link="${parent}"/>
@@ -87,14 +68,14 @@
 			<inertia ixx="0.00017623" iyy="0.000068428" iyz="-0.00001757133" izz="0.00021455" ixy="0.00000095729" ixz="-0.0000000562908"/>
         </xacro:forque_assembly_link>
-	  	<xacro:forque_assembly_joint joint_name="FTMount_to_world" type="fixed" parent="${base_parent}" child="FTMount" joint_axis_xyz="0 0 1" joint_origin_xyz="0 0 -0.005" joint_origin_rpy="0 0 0" fixed="true"/>
+	  	<xacro:forque_assembly_joint joint_name="FTMount_to_world" type="fixed" parent="${base_parent}" child="FTMount" joint_axis_xyz="0 0 1" joint_origin_xyz="0 0 -0.005" joint_origin_rpy="0 0 0"/>
 	  	<xacro:forque_assembly_link link_name="FT" link_mesh="2023_03_09_wirelessFT" mass="0.280" cog="0.0111446 -0.0882070 -0.0544936">
 	  		<inertia ixx="0.000543925" iyy="0.000165428" iyz="-0.00000001487288" izz="0.000691232" ixy="-0.00000128367" ixz="0"/>
 	  	</xacro:forque_assembly_link>
-	  	<xacro:forque_assembly_joint joint_name="FT_to_FTMount" type="fixed" parent="FTMount" child="FT" joint_axis_xyz="0 0 1" joint_origin_xyz="0 0 0" joint_origin_rpy="0 0 0" fixed="true"/>
+	  	<xacro:forque_assembly_joint joint_name="FT_to_FTMount" type="fixed" parent="FTMount" child="FT" joint_axis_xyz="0 0 1" joint_origin_xyz="0 0 0" joint_origin_rpy="0 0 0"/>
 	  	<xacro:if value="${use_antenna}">
             <xacro:forque_assembly_link link_name="FTAntenna" link_mesh="2023_03_09_wirelessFTAntenna" mass="0.018" cog="-0.0162965 0.0666626 -0.0545096">
                 <xacro:insert_block name="default_inertial"/>
             </xacro:forque_assembly_link>
-    	  	<xacro:forque_assembly_joint joint_name="FTAntenna_to_FT" type="fixed" parent="FT" child="FTAntenna" joint_axis_xyz="0 0 1" joint_origin_xyz="0 0 0" joint_origin_rpy="0 0 0" fixed="true"/>
+    	  	<xacro:forque_assembly_joint joint_name="FTAntenna_to_FT" type="fixed" parent="FT" child="FTAntenna" joint_axis_xyz="0 0 1" joint_origin_xyz="0 0 0" joint_origin_rpy="0 0 0"/>
 		</xacro:if>
 	  	<xacro:forque_assembly_link link_name="forkHandle" link_mesh="2024_06_24_forkHandleHollow" mass="0.028" cog="0.011097 -0.162629 -0.011948">
@@ -102,30 +83,30 @@
 	  	</xacro:forque_assembly_link>
 		<!-- The slight rotation was manually added due to empirical deformations in the robot gripped, such that the fingers and fork handle were slightly pitched up relative to the wrist. -->
-		<xacro:forque_assembly_joint joint_name="forkHandle_to_FTMount" type="fixed" parent="FTMount" child="forkHandle" joint_axis_xyz="0 0 1" joint_origin_xyz="0 0.005 0.0013" joint_origin_rpy="-0.025 0 -0.0065" fixed="true"/>
+		<xacro:forque_assembly_joint joint_name="forkHandle_to_FTMount" type="fixed" parent="FTMount" child="forkHandle" joint_axis_xyz="0 0 1" joint_origin_xyz="0 0.005 0.0013" joint_origin_rpy="-0.025 0 -0.0065"/>
 		<xacro:forque_assembly_link link_name="forkHandleCover" link_mesh="2024_06_24_forkHandleCover" mass="0.004" cog="0.011157 -0.168451 0.006404">
 	  		<inertia ixx="0.0000027878" iyy="0.00000064518" iyz="0.00000016201" izz="0.000003363634" ixy="0.00000000012805" ixz="0.00000000006585"/>
 	  	</xacro:forque_assembly_link>
-		<xacro:forque_assembly_joint joint_name="forkHandleCover_to_forkHandle" type="fixed" parent="forkHandle" child="forkHandleCover" joint_axis_xyz="0 0 1" joint_origin_xyz="0 0 0" joint_origin_rpy="0 0 0" fixed="true"/>
+		<xacro:forque_assembly_joint joint_name="forkHandleCover_to_forkHandle" type="fixed" parent="forkHandle" child="forkHandleCover" joint_axis_xyz="0 0 1" joint_origin_xyz="0 0 0" joint_origin_rpy="0 0 0"/>
       <xacro:if value="${end_effector_tool == 'articulable_fork'}">
           <xacro:forque_assembly_link link_name="af_link_base" link_mesh="fr12-h103" mass="0.0907185" cog="0.0 0.0 0.0">
               <xacro:insert_block name="default_inertial"/>
           </xacro:forque_assembly_link>
-          <xacro:forque_assembly_joint joint_name="af_joint_base" type="fixed" parent="forkHandle" child="af_link_base" joint_axis_xyz="0 0 1" joint_origin_xyz="0.010929196 -0.278553 -0.011" joint_origin_rpy="0 0 0" fixed="true"/>
+          <xacro:forque_assembly_joint joint_name="af_joint_base" type="fixed" parent="forkHandle" child="af_link_base" joint_axis_xyz="0 0 1" joint_origin_xyz="0.010929196 -0.278553 -0.011" joint_origin_rpy="0 0 0"/>
           <xacro:forque_assembly_link link_name="af_link_1" link_mesh="XC-430_idle" mass="0.065" cog="0.21641853 -14.751192 -16.796092">
               <inertia ixx="18680.931" iyy="9585.9138" iyz="-845.46678" izz="17346.641" ixy="1.3348619" ixz="-45.354028"/>
           </xacro:forque_assembly_link>
-          <xacro:forque_assembly_joint joint_name="af_joint_1" type="revolute" parent="af_link_base" child="af_link_1" joint_axis_xyz="0 0 1" joint_origin_xyz="0 0 0" joint_origin_rpy="${J_PI/2} 0 ${J_PI/2}" joint_lower_limit="${-J_PI/2}" joint_upper_limit="${J_PI/2}" joint_velocity_limit="1" joint_torque_limit="1.4" fixed="false"/>
+          <xacro:forque_assembly_joint joint_name="af_joint_1" type="revolute" parent="af_link_base" child="af_link_1" joint_axis_xyz="0 0 1" joint_origin_xyz="0 0 0" joint_origin_rpy="${J_PI/2} 0 ${J_PI/2}" joint_lower_limit="${-J_PI/2}" joint_upper_limit="${J_PI/2}" joint_velocity_limit="1" joint_torque_limit="1.4"/>
           <xacro:forque_assembly_link link_name="af_motor_fixture_link" link_mesh="fr12-s101" mass="0.0453592" cog="0 0 0">
               <xacro:insert_block name="default_inertial"/>
           </xacro:forque_assembly_link>
-          <xacro:forque_assembly_joint joint_name="af_motor_fixture_joint_1" type="fixed" parent="af_link_1" child="af_motor_fixture_link" joint_axis_xyz="0 0 1" joint_origin_xyz="0 0 0" joint_origin_rpy="0 ${-J_PI/2} 0" fixed="true"/>
+          <xacro:forque_assembly_joint joint_name="af_motor_fixture_joint_1" type="fixed" parent="af_link_1" child="af_motor_fixture_link" joint_axis_xyz="0 0 1" joint_origin_xyz="0 0 0" joint_origin_rpy="0 ${-J_PI/2} 0"/>
           <xacro:forque_assembly_link link_name="af_link_2" link_mesh="XC-430_idle" mass="0.065" cog="0.21641853 -14.751192 -16.796092">
               <inertia ixx="18680.931" iyy="9585.9138" iyz="-845.46678" izz="17346.641" ixy="1.3348619" ixz="-45.354028"/>
           </xacro:forque_assembly_link>
-          <xacro:forque_assembly_joint joint_name="af_motor_fixture_joint_2" type="fixed" parent="af_link_1" child="af_link_2" joint_axis_xyz="0 0 1" joint_origin_xyz="-0.03825 0 0" joint_origin_rpy="0 ${-J_PI/2} 0" fixed="true"/>
+          <xacro:forque_assembly_joint joint_name="af_motor_fixture_joint_2" type="fixed" parent="af_link_1" child="af_link_2" joint_axis_xyz="0 0 1" joint_origin_xyz="-0.03825 0 0" joint_origin_rpy="0 ${-J_PI/2} 0"/>
           <xacro:forque_assembly_link link_name="af_ft_adapter_link" link_mesh="roll_to_ft_adapter" mass="0.001" cog="0 0 0">
               <xacro:insert_block name="default_inertial"/>
           </xacro:forque_assembly_link>
-          <xacro:forque_assembly_joint joint_name="af_joint_2" type="revolute" parent="af_link_2" child="af_ft_adapter_link" joint_axis_xyz="0 1 0" joint_origin_xyz="0 0 0.019" joint_origin_rpy="${-J_PI/2} 0 0" joint_lower_limit="${-J_PI}" joint_upper_limit="${J_PI}" joint_velocity_limit="1" joint_torque_limit="1.4" fixed="false"/>
+          <xacro:forque_assembly_joint joint_name="af_joint_2" type="revolute" parent="af_link_2" child="af_ft_adapter_link" joint_axis_xyz="0 1 0" joint_origin_xyz="0 0 0.019" joint_origin_rpy="${-J_PI/2} 0 0" joint_lower_limit="${-J_PI}" joint_upper_limit="${J_PI}" joint_velocity_limit="1" joint_torque_limit="1.4"/>
       </xacro:if>
 	  	<xacro:forque_assembly_link link_name="forque" link_mesh="ATI-9105-TW-NANO25-E" mass="0.0634" cog="0.0124692 0.0137169 0.010558">
@@ -133,13 +114,13 @@
 	  	</xacro:forque_assembly_link>
       <xacro:if value="${end_effector_tool == 'articulable_fork'}">
-          <xacro:forque_assembly_joint joint_name="af_forque_joint" type="fixed" parent="af_ft_adapter_link" child="forque" joint_axis_xyz="0 0 1" joint_origin_xyz="-0.0175 -0.011 0.004" joint_origin_rpy="${J_PI/2} ${J_PI/3} 0" fixed="true"/>
+          <xacro:forque_assembly_joint joint_name="af_forque_joint" type="fixed" parent="af_ft_adapter_link" child="forque" joint_axis_xyz="0 0 1" joint_origin_xyz="-0.0175 -0.011 0.004" joint_origin_rpy="${J_PI/2} ${J_PI/3} 0"/>
       </xacro:if>
       <xacro:if value="${end_effector_tool == 'fork'}">
-          <xacro:forque_assembly_joint joint_name="af_forque_joint" type="fixed" parent="forkHandle" child="forque" joint_axis_xyz="0 0 1" joint_origin_xyz="-0.00634 -0.222553 -0.004286" joint_origin_rpy="${J_PI/2} ${J_PI/3} 0" fixed="true"/>
+          <xacro:forque_assembly_joint joint_name="af_forque_joint" type="fixed" parent="forkHandle" child="forque" joint_axis_xyz="0 0 1" joint_origin_xyz="-0.00634 -0.222553 -0.004286" joint_origin_rpy="${J_PI/2} ${J_PI/3} 0"/>
       </xacro:if>
 	  	<xacro:forque_assembly_link link_name="forkTine" link_mesh="fork_tine" mass="0.024" cog="0.013090 0.0180789 0.0445231">
 	  		<inertia ixx="0.0000098769" iyy="0.000009848103" iyz="0.00000057639" izz="0.0000015674" ixy="0.000000000806182" ixz="-0.00000000296036"/>
 	  	</xacro:forque_assembly_link>
-	  	<xacro:forque_assembly_joint joint_name="forkTine_to_forque" type="fixed" parent="forque" child="forkTine" joint_axis_xyz="0 0 1" joint_origin_xyz="-0.0054 0.008 0.093" joint_origin_rpy="0 ${J_PI} ${240*J_PI/180}" fixed="true"/>
+	  	<xacro:forque_assembly_joint joint_name="forkTine_to_forque" type="fixed" parent="forque" child="forkTine" joint_axis_xyz="0 0 1" joint_origin_xyz="-0.0054 0.008 0.093" joint_origin_rpy="0 ${J_PI} ${240*J_PI/180}"/>
 	  	<link name="forkTip" />
 	  	<joint name="forkTip_to_forkTine" type="fixed">

Commit message: Implement ADA Xacro macro, and instantiate explicitly in ada_standalone.xacro

File: ada_description/urdf/ada.xacro (robot description, xacro)
@@ -14,107 +14,100 @@
   xmlns:physics="http://playerstage.sourceforge.net/gazebo/xmlschema/#physics"
   xmlns:xacro="http://www.ros.org/wiki/xacro"
-  name="ada"
 >
-  <xacro:include filename="$(find ada_description)/urdf/forque/forque.xacro"/>
-  <xacro:include filename="$(find ada_description)/urdf/camera/camera.xacro"/>
-  <xacro:include filename="$(find ada_description)/urdf/j2n6s200.xacro"/>
-  <xacro:arg
-    name="use_forque"
-    default="true"
-  />
-  <link name="root"/>
-  <link name="root_tilt"/>
-  <joint
-    name="robot_tilt"
-    type="revolute"
+  <!-- Robot name must be defined in the Xacro file that instantiates the ada macro -->
+  <xacro:macro
+    name="ada"
+    params="end_effector_tool"
   >
-    <origin
-      xyz="0 0 0"
-      rpy="0 0 0"
+    <!-- Import macros associated with forque, robot, and camera. Macros are added to the tree below -->
+    <xacro:include filename="$(find ada_description)/urdf/forque/forque.xacro"/>
+    <xacro:include filename="$(find ada_description)/urdf/camera/camera.xacro"/>
+    <xacro:include filename="$(find ada_description)/urdf/j2n6s200.xacro"/>
+    <xacro:include filename="$(find articutool_description)/urdf/articutool.xacro"/>
+    <link name="root"/>
+    <link name="root_tilt"/>
+    <joint
+      name="robot_tilt"
+      type="revolute"
+    >
+      <origin
+        xyz="0 0 0"
+        rpy="0 0 0"
+      />
+      <child link="root_tilt"/>
+      <parent link="root"/>
+      <axis xyz="-1 0 0"/>
+      <!-- effort copied from j2n6s200 joint 2, velocity is max velocity the wheelchair can tilt,
+      lower and upper limits generously encompass the range of the wheelchair's tilt-->
+      <limit
+        effort="80"
+        velocity="0.15"
+        lower="${-J_PI}"
+        upper="${J_PI}"
+      />
+      <dynamics
+        damping="0.0"
+        friction="0.0"
+      />
+    </joint>
+    <xacro:property
+      name="robot_root"
+      value="root_tilt"
     />
-    <child link="root_tilt"/>
-    <parent link="root"/>
-    <axis xyz="-1 0 0"/>
-    <!-- effort copied from j2n6s200 joint 2, velocity is max velocity the wheelchair can tilt,
-    lower and upper limits generously encompass the range of the wheelchair's tilt-->
-    <limit
-      effort="80"
-      velocity="0.15"
-      lower="${-J_PI}"
-      upper="${J_PI}"
+    <xacro:j2n6s200 base_parent="${robot_root}"/>
+    <xacro:camera_assembly
+      base_parent="j2n6s200_link_6"
+      base_xyz="0.0165 0 0.0011"
+      base_rpy="${3*J_PI/2} 0 ${3*J_PI/2}"
     />
-    <dynamics
-      damping="0.0"
-      friction="0.0"
-    />
-  </joint>
-  <xacro:property
-    name="robot_root"
-    value="root_tilt"
-  />
-  <xacro:j2n6s200 base_parent="${robot_root}"/>
-  <xacro:camera_assembly
-    base_parent="j2n6s200_link_6"
-    base_xyz="0.0165 0 0.0011"
-    base_rpy="${3*J_PI/2} 0 ${3*J_PI/2}"
-  />
-  <!-- Hard-coded Extrinsics -->
-  <link name="camera_link"/>
-  <joint
-    name="extrinsics"
-    type="fixed"
-  >
-    <origin
-      xyz="0.0194 -0.01606 0.029014"
-      rpy="0.17234 -1.56127 2.96967"
-    />
-    <parent link="cameraMount"/>
-    <child link="camera_link"/>
-  </joint>
-  <!-- Copy Realsense in case of simulation -->
-  <!--
-  <link name="camera_color_optical_frame" />
-  <joint name="optical_republish" type="fixed">
-    <origin xyz="0.000 -0.015 0.000" rpy="-1.564 0.000 -1.573" />
-    <parent link="camera_link" />
-    <child link="camera_color_optical_frame" />
-  </joint>
-  -->
-  <xacro:forque_assembly_link
-    link_name="FTArmMount"
-    link_mesh="2024_01_18_FTArmMount"
-    mass="0.03783"
-    cog="0.010957 -0.019223 -0.03777"
-  >
-    <inertia
-      ixx="0.000018817"
-      iyy="0.00001119989"
-      iyz="-0.00000120296"
-      izz="0.000026883"
-      ixy="-0.0000003327"
-      ixz="-0.000000092476"
-    />
-  </xacro:forque_assembly_link>
-  <xacro:forque_assembly_joint
-    joint_name="FTArmMount_to_arm"
-    parent="j2n6s200_link_6"
-    child="FTArmMount"
-    joint_origin_xyz="0.0065 -0.011 -0.0075"
-    joint_origin_rpy="${J_PI/2} 0 ${J_PI/2}"
-  />
-  <xacro:if value="$(arg use_forque)">
-    <xacro:forque_assembly base_parent="FTArmMount"/>
-    <link name="FTSensor"/>
+    <!-- Hard-coded Extrinsics -->
+    <link name="camera_link"/>
     <joint
-      name="EE_to_FTSensor"
+      name="extrinsics"
       type="fixed"
     >
-      <child link="FTSensor"/>
-      <parent link="j2n6s200_end_effector"/>
       <origin
-        rpy="0 0 0"
-        xyz="0.0 0.0 0.092"
+        xyz="0.0194 -0.01606 0.029014"
+        rpy="0.17234 -1.56127 2.96967"
       />
+      <parent link="cameraMount"/>
+      <child link="camera_link"/>
     </joint>
-  </xacro:if>
+    <!-- Copy Realsense in case of simulation -->
+    <!--
+    <link name="camera_color_optical_frame" />
+    <joint name="optical_republish" type="fixed">
+      <origin xyz="0.000 -0.015 0.000" rpy="-1.564 0.000 -1.573" />
+      <parent link="camera_link" />
+      <child link="camera_color_optical_frame" />
+    </joint>
+    -->
+    <xacro:forque_assembly_link
+      link_name="FTArmMount"
+      link_mesh="2024_01_18_FTArmMount"
+      mass="0.03783"
+      cog="0.010957 -0.019223 -0.03777"
+    >
+      <inertia
+        ixx="0.000018817"
+        iyy="0.00001119989"
+        iyz="-0.00000120296"
+        izz="0.000026883"
+        ixy="-0.0000003327"
+        ixz="-0.000000092476"
+      />
+    </xacro:forque_assembly_link>
+    <xacro:forque_assembly_joint
+      joint_name="FTArmMount_to_arm"
+      type="fixed"
+      parent="j2n6s200_link_6"
+      child="FTArmMount"
+      joint_axis_xyz="0 0 1"
+      joint_origin_xyz="0.0065 -0.011 -0.0075"
+      joint_origin_rpy="${J_PI/2} 0 ${J_PI/2}"
+    />
+    <xacro:unless value="${end_effector_tool == 'none'}">
+      <xacro:articutool base_parent="j2n6s200_end_effector" end_effector_tool="${end_effector_tool}" joint_origin_rpy="0 0 ${J_PI/2}" joint_origin_xyz="0 -2.25 -1"/>
+    </xacro:unless>
+  </xacro:macro>
 </robot>
