Commit message: Integration of Articutool Description and MoveIt Configuration (#60)
* Update forque Xacro macro

* Implement ADA Xacro macro, and instantiate explicitly in ada_standalone.xacro

* Revert "Implement ADA Xacro macro, and instantiate explicitly in ada_standalone.xacro"

This reverts commit b3785d5300abfb86a6d2d53091b5feffa7e7e9d6.

* Revert "Update forque Xacro macro"

This reverts commit 130922fe86c3708d6046c8b2f4715c25edc6f9d4.

* Implement ADA Xacro macro

* Instantiate ADA URDF using new macro, and add Articutool URDF

* Remove Articutool instance from ada.urdf.xacro

* Add ada namespace to controllers

* Add ada_moveit.launch.py (WIP)

* Update tip_link/end_effector_link to use j2n6s200_end_effector

* Remove disable_collisions for various links on the original forque

* Update ada_keyboard_teleop to use ada namespace for controllers

* Implement node to combine joint states from ADA and Articutool

* Launch combined_joint_states node and remap robot_state_publisher to read from it

* Add Articutool URDF/SRDF to existing ADA URDF/SRDF

* Add IMU joint state publisher

* Add ada namespace into moveit.rviz and moveit_controllers.yaml. Perform required remapping to namespaced topics

* Remove /ada namespaces

* Add jaco_arm_with_articutool move group, and define Articutool joints as passive so that they aren't actuated when planning a trajectory. Despite not being actuated, the planner still seems to incorporate the Articutool joints into the planned trajectory, so we need to find a way to also have the planner ignore the joints entirely, as if the Articutool were a rigid extension from the Jaco's hand

* Add IK and OMPL planner for jaco_arm_with_articutool group

* Use jaco_arm_with_articutool move group and tool_tip frame for mock servo

* Remove combined_joint_states.py

* Remove unused joint_map parameter

* Configure Articutool Xacro as dummy so that the jaco_arm_with_articutool planning group will consider the Articutool's joint as fixed, effectively circumventing an issue where planning with the group would use all joints in the kinematic chain when it was only desired to use the Jaco joints.

* Remove Articutool planning group and group_state

* Set Articutool to not use dummy mimic joints. This will allow the IK solver to use the passive joints from the Articutool, but we will try to use joint constraints during planning instead to prevent this in both the IK solution as well as the generated trajectory

* Add a node to publish a unified joint state from ADA and the Articutool. If either has no up to date data, we use the previous valid joint state message.

* Add Articutool planning group again

* Add SimulatedOrientationPublisherNode which publishes the orientation of a desired link relative to some base frame. We use this to simulated an ideal orientation estimate from the IMU on the Articutool

* Add IK solver and planner for Articutool

* Modify planning parameters for Articutool

* Adjust moveit RViz configuration to only show robot model, and disable query goal state

* Extend IK solver timeout and attempts for jaco_arm_with_articutool

* Add CHOMP planner and set to default for now so we can test

* Reformatting

* Remove simulated orientation node

* Add configurations for end_effector_tool argument

* Reduce frequency of unified joint state publishing

* Update F/T topics

* Add a bunch of launch arguments so that the end_effector_tool argument actually propagates through to the argument in the Xacro. We should really consider simplifying all these launch files, they are not modular at all

* Remove dummy parameter

* Disable collisions for new Xacro

* Remove dependency on CHOMP planner

* Remove CHOMP dependency from CMakeLists.txt

* Remove CHOMP from planning pipelines

* Remove CHOMP planning config file

* Increase timeout and attempts for all planning groups

* Update frame for tele-op

* Remove collisions for screw heads with arm

* Add lock_joints parameter

* Conditionally restrict Articutool joint states from being published by the unified joint state publisher if they are locked

* Increase Articutool roll joint limit on ADA-side

* Remove redundant launch file

* Remove commented out packages

* Revert moveit.rviz settings

* Remove comments for CHOMP

* Remove unused import

* Add license to simulated_orientation_publisher_node

* Adjust RRTstar range and goal_bias. This change seems to dramatically increase the performance of the Articutool's planning success rate with lower planning times

* Tune 8-DOF planning group's IK solve, and reduce the Articutool's roll joint limits back down to +/- pi

* Increase longest_valid_segment_fraction for RRT*

* Run pre-commit

* fixed pre-commit issues

---------

Co-authored-by: Eddie Ni <eddieni06@gmail.com>

File: ada_description/urdf/ada.xacro (robot description, xacro)
@@ -14,107 +14,108 @@
   xmlns:physics="http://playerstage.sourceforge.net/gazebo/xmlschema/#physics"
   xmlns:xacro="http://www.ros.org/wiki/xacro"
-  name="ada"
 >
-  <xacro:include filename="$(find ada_description)/urdf/forque/forque.xacro"/>
-  <xacro:include filename="$(find ada_description)/urdf/camera/camera.xacro"/>
-  <xacro:include filename="$(find ada_description)/urdf/j2n6s200.xacro"/>
-  <xacro:arg
-    name="use_forque"
-    default="true"
-  />
-  <link name="root"/>
-  <link name="root_tilt"/>
-  <joint
-    name="robot_tilt"
-    type="revolute"
+  <!-- Robot name must be defined in the Xacro file that instantiates the ada macro -->
+  <xacro:macro
+    name="ada"
+    params="use_forque"
   >
-    <origin
-      xyz="0 0 0"
-      rpy="0 0 0"
+    <xacro:include filename="$(find ada_description)/urdf/forque/forque.xacro"/>
+    <xacro:include filename="$(find ada_description)/urdf/camera/camera.xacro"/>
+    <xacro:include filename="$(find ada_description)/urdf/j2n6s200.xacro"/>
+    <link name="root"/>
+    <link name="root_tilt"/>
+    <joint
+      name="robot_tilt"
+      type="revolute"
+    >
+      <origin
+        xyz="0 0 0"
+        rpy="0 0 0"
+      />
+      <child link="root_tilt"/>
+      <parent link="root"/>
+      <axis xyz="-1 0 0"/>
+      <!-- effort copied from j2n6s200 joint 2, velocity is max velocity the wheelchair can tilt,
+      lower and upper limits generously encompass the range of the wheelchair's tilt-->
+      <limit
+        effort="80"
+        velocity="0.15"
+        lower="${-J_PI}"
+        upper="${J_PI}"
+      />
+      <dynamics
+        damping="0.0"
+        friction="0.0"
+      />
+    </joint>
+    <xacro:property
+      name="robot_root"
+      value="root_tilt"
     />
-    <child link="root_tilt"/>
-    <parent link="root"/>
-    <axis xyz="-1 0 0"/>
-    <!-- effort copied from j2n6s200 joint 2, velocity is max velocity the wheelchair can tilt,
-    lower and upper limits generously encompass the range of the wheelchair's tilt-->
-    <limit
-      effort="80"
-      velocity="0.15"
-      lower="${-J_PI}"
-      upper="${J_PI}"
+    <xacro:j2n6s200 base_parent="${robot_root}"/>
+    <xacro:camera_assembly
+      base_parent="j2n6s200_link_6"
+      base_xyz="0.0165 0 0.0011"
+      base_rpy="${3*J_PI/2} 0 ${3*J_PI/2}"
     />
-    <dynamics
-      damping="0.0"
-      friction="0.0"
-    />
-  </joint>
-  <xacro:property
-    name="robot_root"
-    value="root_tilt"
-  />
-  <xacro:j2n6s200 base_parent="${robot_root}"/>
-  <xacro:camera_assembly
-    base_parent="j2n6s200_link_6"
-    base_xyz="0.0165 0 0.0011"
-    base_rpy="${3*J_PI/2} 0 ${3*J_PI/2}"
-  />
-  <!-- Hard-coded Extrinsics -->
-  <link name="camera_link"/>
-  <joint
-    name="extrinsics"
-    type="fixed"
-  >
-    <origin
-      xyz="0.0194 -0.01606 0.029014"
-      rpy="0.17234 -1.56127 2.96967"
-    />
-    <parent link="cameraMount"/>
-    <child link="camera_link"/>
-  </joint>
-  <!-- Copy Realsense in case of simulation -->
-  <!--
-  <link name="camera_color_optical_frame" />
-  <joint name="optical_republish" type="fixed">
-    <origin xyz="0.000 -0.015 0.000" rpy="-1.564 0.000 -1.573" />
-    <parent link="camera_link" />
-    <child link="camera_color_optical_frame" />
-  </joint>
-  -->
-  <xacro:forque_assembly_link
-    link_name="FTArmMount"
-    link_mesh="2024_01_18_FTArmMount"
-    mass="0.03783"
-    cog="0.010957 -0.019223 -0.03777"
-  >
-    <inertia
-      ixx="0.000018817"
-      iyy="0.00001119989"
-      iyz="-0.00000120296"
-      izz="0.000026883"
-      ixy="-0.0000003327"
-      ixz="-0.000000092476"
-    />
-  </xacro:forque_assembly_link>
-  <xacro:forque_assembly_joint
-    joint_name="FTArmMount_to_arm"
-    parent="j2n6s200_link_6"
-    child="FTArmMount"
-    joint_origin_xyz="0.0065 -0.011 -0.0075"
-    joint_origin_rpy="${J_PI/2} 0 ${J_PI/2}"
-  />
-  <xacro:if value="$(arg use_forque)">
-    <xacro:forque_assembly base_parent="FTArmMount"/>
-    <link name="FTSensor"/>
+    <!-- Hard-coded Extrinsics -->
+    <link name="camera_link"/>
     <joint
-      name="EE_to_FTSensor"
+      name="extrinsics"
       type="fixed"
     >
-      <child link="FTSensor"/>
-      <parent link="j2n6s200_end_effector"/>
       <origin
-        rpy="0 0 0"
-        xyz="0.0 0.0 0.092"
+        xyz="0.0194 -0.01606 0.029014"
+        rpy="0.17234 -1.56127 2.96967"
       />
+      <parent link="cameraMount"/>
+      <child link="camera_link"/>
     </joint>
-  </xacro:if>
+    <!-- Copy Realsense in case of simulation -->
+    <!--
+    <link name="camera_color_optical_frame" />
+    <joint name="optical_republish" type="fixed">
+      <origin xyz="0.000 -0.015 0.000" rpy="-1.564 0.000 -1.573" />
+      <parent link="camera_link" />
+      <child link="camera_color_optical_frame" />
+    </joint>
+    -->
+    <xacro:forque_assembly_link
+      link_name="FTArmMount"
+      link_mesh="2024_01_18_FTArmMount"
+      mass="0.03783"
+      cog="0.010957 -0.019223 -0.03777"
+    >
+      <inertia
+        ixx="0.000018817"
+        iyy="0.00001119989"
+        iyz="-0.00000120296"
+        izz="0.000026883"
+        ixy="-0.0000003327"
+        ixz="-0.000000092476"
+      />
+    </xacro:forque_assembly_link>
+    <xacro:forque_assembly_joint
+      joint_name="FTArmMount_to_arm"
+      parent="j2n6s200_link_6"
+      child="FTArmMount"
+      joint_origin_xyz="0.0065 -0.011 -0.0075"
+      joint_origin_rpy="${J_PI/2} 0 ${J_PI/2}"
+    />
+    <xacro:if value="$(arg use_forque)">
+      <xacro:forque_assembly base_parent="FTArmMount"/>
+      <link name="FTSensor"/>
+      <joint
+        name="EE_to_FTSensor"
+        type="fixed"
+      >
+        <child link="FTSensor"/>
+        <parent link="j2n6s200_end_effector"/>
+        <origin
+          rpy="0 0 0"
+          xyz="0.0 0.0 0.092"
+        />
+      </joint>
+    </xacro:if>
+  </xacro:macro>
 </robot>

File: ada_moveit/config/ada.urdf.xacro (robot description, xacro)
@@ -12,6 +12,31 @@
     default="real"
   />
+  <xacro:arg
+    name="use_forque"
+    default="false"
+  />
+  <xacro:arg
+    name="end_effector_tool"
+    default="fork"
+  />
+  <xacro:arg
+    name="lock_joints"
+    default="false"
+  />
   <!-- Import ada urdf file -->
   <xacro:include filename="$(find ada_description)/urdf/ada.xacro"/>
+  <xacro:include filename="$(find articutool_description)/urdf/articutool.xacro"/>
+  <xacro:property
+    name="end_effector_tool"
+    value="$(arg end_effector_tool)"
+  />
+  <xacro:ada use_forque="$(arg use_forque)"/>
+  <xacro:articutool
+    base_parent="j2n6s200_end_effector"
+    end_effector_tool="${end_effector_tool}"
+    joint_origin_rpy="0 0 ${J_PI/2}"
+    joint_origin_xyz="0 -2.25 -1"
+    lock_joints="$(arg lock_joints)"
+  />
   <!-- Import control_xacro -->
   <xacro:include filename="ada.ros2_control.xacro"/>
