Commit message: [WIP] kept working on camera xacro

File: ada_description/urdf/camera/camera.xacro (robot description, xacro)
@@ -1,10 +1,36 @@
 <?xml version="1.0"?>
-<xacro:macro name="camera" params="base_parent" />
-	<link name="nano_arm_mount">
-		<visual>
-			<geometry>
-				<mesh
-					filename="package://ada_description/meshes/camera/2023_03_09_nanoArmMount.stl"/>
-			</geometry>
-			<material name=""
-</xacro:macro>
+<root xmlns:xi="http://www.w3.org/2001/XInclude"
+	xmlns:gazebo="http://playerstage.sourceforge.net/gazebo/xmlschema/#gz"
+    xmlns:model="http://playerstage.sourceforge.net/gazebo/xmlschema/#model"
+	xmlns:sensor="http://playerstage.sourceforge.net/gazebo/xmlschema/#sensor"
+	xmlns:body="http://playerstage.sourceforge.net/gazebo/xmlschema/#body"
+    xmlns:geom="http://playerstage.sourceforge.net/gazebo/xmlschema/#geom"
+    xmlns:joint="http://playerstage.sourceforge.net/gazebo/xmlschema/#joint"
+	xmlns:controller="http://playerstage.sourceforge.net/gazebo/xmlschema/#controller"
+	xmlns:interface="http://playerstage.sourceforge.net/gazebo/xmlschema/#interface"
+	xmlns:rendering="http://playerstage.sourceforge.net/gazebo/xmlschema/#rendering"
+    xmlns:renderable="http://playerstage.sourceforge.net/gazebo/xmlschema/#renderable"
+    xmlns:physics="http://playerstage.sourceforge.net/gazebo/xmlschema/#physics"
+	xmlns:xacro="http://www.ros.org/wiki/xacro">
+	<xacro:property name="camColor" value="255 0 0 1" />
+	<xacro:macro name="armMount_link" params="base_parent">
+		<link name="nano_arm_mount">
+			<visual>
+				<geometry>
+					<mesh
+						filename="package://ada_description/meshes/camera/2023_03_09_nanoArmMount.stl"/>
+				</geometry>
+				<material name="abs">
+					<color rgba="${camColor}" />
+				</material>
+			</visual>
+		</link>
+	</xacro:macro>
+	<xacro:macro name="armMount_joint">
+		<joint name="nano_arm_mount_to_world" type="continuous">
+			<parent link="base_parent"/>
+			<child link="nano_arm_mount"/>
+			<axis xyz="0 0 1"/>
+		</joint>
+	</xacro:macro>
+</root>

Commit message: [WIP] continued working on camera xacro

File: ada_description/urdf/camera/camera.xacro (robot description, xacro)
@@ -13,11 +13,13 @@
     xmlns:physics="http://playerstage.sourceforge.net/gazebo/xmlschema/#physics"
 	xmlns:xacro="http://www.ros.org/wiki/xacro">
-	<xacro:property name="camColor" value="255 0 0 1" />
-	<xacro:macro name="armMount_link" params="base_parent">
-		<link name="nano_arm_mount">
+	<xacro:property name="camColor" value="1 0 0 1" />
+	<xacro:property name="J_PI" value="3.1415926535897931" />
+	<xacro:macro name="camera_assembly_link" params="link_name link_mesh">
+		<link name="${link_name}">
 			<visual>
 				<geometry>
 					<mesh
-						filename="package://ada_description/meshes/camera/2023_03_09_nanoArmMount.stl"/>
+						filename="package://ada_description/meshes/camera/${link_mesh}.stl"
+						scale="0.001 0.001 0.001"/>
 				</geometry>
 				<material name="abs">
@@ -27,10 +29,23 @@
 		</link>
 	</xacro:macro>
-	<xacro:macro name="armMount_joint">
-		<joint name="nano_arm_mount_to_world" type="continuous">
-			<parent link="base_parent"/>
-			<child link="nano_arm_mount"/>
+	<xacro:macro name="camera_assembly_joint" params="joint_name parent child joint_origin_xyz joint_origin_rpy">
+		<joint name="${joint_name}" type="continuous">
+			<parent link="${parent}"/>
+			<child link="${child}"/>
 			<axis xyz="0 0 1"/>
+			<origin xyz="${joint_origin_xyz}" rpy="${joint_origin_rpy}"/>
 		</joint>
 	</xacro:macro>
+	<xacro:macro name="camera_assembly" params="base_parent">
+		<xacro:camera_assembly_link link_name="nanoMount" link_mesh="2023_03_09_nanoArmMount"/>
+	  	<xacro:camera_assembly_joint joint_name="nanoMount_to_world" parent="${base_parent}" child="nanoMount" joint_origin_xyz="0 0 0" joint_origin_rpy="0 0 0"/>
+		<xacro:camera_assembly_link link_name="enclosureBottom" link_mesh="2023_03_16_nanoEnclosureBottom"/>
+		<xacro:camera_assembly_joint joint_name="enclosureBottom_to_nanoMount" parent="nanoMount" child="enclosureBottom" joint_origin_xyz="0.0412 -0.0218 0.026" joint_origin_rpy="0 0 ${J_PI/2}"/>
+		<xacro:camera_assembly_link link_name="nano" link_mesh="2023_03_21_jetsonNano"/>
+		<xacro:camera_assembly_joint joint_name="nano_to_enclosureBottom" parent="enclosureBottom" child="nano" joint_origin_xyz="0 0 0" joint_origin_rpy="0 0 0"/>
+		<xacro:camera_assembly_link link_name="enclosureTop" link_mesh="2023_03_09_nanoEnclosureTop"/>
+		<xacro:camera_assembly_joint joint_name="enclosureTop_to_enclosureBottom" parent="enclosureBottom" child="enclosureTop" joint_origin_xyz="0 0 0" joint_origin_rpy="0 0 0"/>
+		<xacro:camera_assembly_link link_name="stabilizer" link_mesh="2023_03_09_cameraStabilizer"/>
+		<xacro:camera_assembly_joint joint_name="stabilizer_to_enclosureTop" parent="enclosureTop" child="stabilizer" joint_origin_xyz="0 0 0" joint_origin_rpy="0 0 0"/>
+	</xacro:macro>
 </root>

File: ada_description/urdf/camera/camera_standalone.xacro (robot description, xacro)
@@ -23,4 +23,4 @@
   </joint>
   <xacro:property name="robot_root" value="root" />
-  <xacro:armMount_link base_parent="${robot_root}"/>
+  <xacro:camera_assembly base_parent="${robot_root}"/>
 </robot>

Commit message: fixed camera stabilizer naming issue

File: ada_description/urdf/camera/camera.xacro (robot description, xacro)
@@ -30,5 +30,5 @@
 	</xacro:macro>
 	<xacro:macro name="camera_assembly_joint" params="joint_name parent child joint_origin_xyz joint_origin_rpy">
-		<joint name="${joint_name}" type="continuous">
+		<joint name="${joint_name}" type="fixed">
 			<parent link="${parent}"/>
 			<child link="${child}"/>
@@ -42,10 +42,12 @@
 		<xacro:camera_assembly_link link_name="enclosureBottom" link_mesh="2023_03_16_nanoEnclosureBottom"/>
 		<xacro:camera_assembly_joint joint_name="enclosureBottom_to_nanoMount" parent="nanoMount" child="enclosureBottom" joint_origin_xyz="0.0412 -0.0218 0.026" joint_origin_rpy="0 0 ${J_PI/2}"/>
+		<!--
 		<xacro:camera_assembly_link link_name="nano" link_mesh="2023_03_21_jetsonNano"/>
-		<xacro:camera_assembly_joint joint_name="nano_to_enclosureBottom" parent="enclosureBottom" child="nano" joint_origin_xyz="0 0 0" joint_origin_rpy="0 0 0"/>
+		<xacro:camera_assembly_joint joint_name="nano_to_enclosureBottom" parent="enclosureBottom" child="nano" joint_origin_xyz="0.0105 0.014 -0.0015" joint_origin_rpy="0 0 0"/>
+		-->
 		<xacro:camera_assembly_link link_name="enclosureTop" link_mesh="2023_03_09_nanoEnclosureTop"/>
 		<xacro:camera_assembly_joint joint_name="enclosureTop_to_enclosureBottom" parent="enclosureBottom" child="enclosureTop" joint_origin_xyz="0 0 0" joint_origin_rpy="0 0 0"/>
 		<xacro:camera_assembly_link link_name="stabilizer" link_mesh="2023_03_09_cameraStabilizer"/>
-		<xacro:camera_assembly_joint joint_name="stabilizer_to_enclosureTop" parent="enclosureTop" child="stabilizer" joint_origin_xyz="0 0 0" joint_origin_rpy="0 0 0"/>
+		<xacro:camera_assembly_joint joint_name="stabilizer_to_enclosureTop" parent="enclosureTop" child="stabilizer" joint_origin_xyz="-0.072824 -0.041 0.05442" joint_origin_rpy="0 0 0"/>
 	</xacro:macro>
 </root>

Commit message: [WIP] finished camera and forque xacro, started working on unified ada xacro

File: ada_description/urdf/camera/camera.xacro (robot description, xacro)
@@ -28,4 +28,10 @@
 				</material>
 			</visual>
+			<collision>
+                <geometry>
+                    <mesh
+                        filename="package://ada_description/meshes/camera/${link_mesh}.stl"/>
+                </geometry>
+            </collision>
 		</link>
 	</xacro:macro>
@@ -38,7 +44,8 @@
 		</joint>
 	</xacro:macro>
-	<xacro:macro name="camera_assembly" params="base_parent">
+	<xacro:property name="default_origin" value="0 0 0"/>
+	<xacro:macro name="camera_assembly" params="base_parent base_xyz:=${default_origin} base_rpy:=${default_origin}">
 		<xacro:camera_assembly_link link_name="nanoMount" link_mesh="2023_03_09_nanoArmMount"/>
-	  	<xacro:camera_assembly_joint joint_name="nanoMount_to_world" parent="${base_parent}" child="nanoMount" joint_origin_xyz="0 0 0" joint_origin_rpy="0 0 0"/>
+	  	<xacro:camera_assembly_joint joint_name="nanoMount_to_world" parent="${base_parent}" child="nanoMount" joint_origin_xyz="${base_xyz}" joint_origin_rpy="${base_rpy}"/>
 		<xacro:camera_assembly_link link_name="enclosureBottom" link_mesh="2023_03_16_nanoEnclosureBottom"/>
 		<xacro:camera_assembly_joint joint_name="enclosureBottom_to_nanoMount" parent="nanoMount" child="enclosureBottom" joint_origin_xyz="0.0412 -0.0218 0.026" joint_origin_rpy="0 0 ${J_PI/2}"/>
@@ -49,8 +56,7 @@
 		<xacro:camera_assembly_link link_name="stabilizer" link_mesh="2023_03_09_cameraStabilizer"/>
 		<xacro:camera_assembly_joint joint_name="stabilizer_to_enclosureTop" parent="enclosureTop" child="stabilizer" joint_origin_xyz="0.0842 0.041 0.0343" joint_origin_rpy="0 ${14.621 * J_PI / 180} 0"/>
-		<!--
-		<xacro:camera_assembly_link link_name="cameraLink" link_mesh="2023_03_30_realsenseD415"/>
-		<xacro:camera_assembly_joint joint_name="cameraLink_to_stabilizer" parent="stabilizer" child="cameraLink" joint_origin_xyz="0.03672 0 0.004" joint_origin_rpy="0 ${3*J_PI/2} ${J_PI}"/>
-		-->
+		<xacro:sensor_d415 parent="stabilizer" use_mesh="true">
+			<origin xyz="0.0165 0 0.0005" rpy="0 0 0" />
+		</xacro:sensor_d415>
 	</xacro:macro>
 </root>

File: ada_description/urdf/camera/d415urdf.xacro (robot description, xacro)
@@ -62,5 +62,5 @@
           <origin xyz="${d415_cam_mount_from_center_offset} ${-d415_cam_depth_py} 0" rpy="${M_PI/2} 0 ${M_PI/2}"/>
           <geometry>
-            <mesh filename="package://realsense2_description/meshes/d415.stl" />
+            <mesh filename="package://ada_description/meshes/camera/d415.stl" />
           </geometry>
           <material name="aluminum"/>

Commit message: Added masses and center of gravity to camera and forque links in urf

File: ada_description/urdf/camera/camera.xacro (robot description, xacro)
@@ -16,5 +16,8 @@
 	<xacro:property name="camColor" value="0.4 0.4 0.4 1" />
 	<xacro:property name="J_PI" value="3.1415926535897931" />
-	<xacro:macro name="camera_assembly_link" params="link_name link_mesh mass:=0">
+	<xacro:property name="default_inertial">
+		<inertia ixx="0.001" iyy="0.001" iyz="0.001" izz="0.001" ixy="0.001" ixz="0.001"/>
+	</xacro:property>
+	<xacro:macro name="camera_assembly_link" params="link_name link_mesh mass:=0 cog:='0 0 0' *inertia">
 		<link name="${link_name}">
 			<visual>
@@ -36,5 +39,7 @@
             </collision>
             <inertial>
+            	<origin xyz="${cog}" rpy="0 0 0"/>
             	<mass value="${mass}"/>
+            	<xacro:insert_block name="inertia"/>
             </inertial>
 		</link>
@@ -50,13 +55,23 @@
 	<xacro:property name="default_origin" value="0 0 0"/>
 	<xacro:macro name="camera_assembly" params="base_parent base_xyz:=${default_origin} base_rpy:=${default_origin}">
-		<xacro:camera_assembly_link link_name="nanoMount" link_mesh="2023_03_09_nanoArmMount"/>
+		<xacro:camera_assembly_link link_name="nanoMount" link_mesh="2023_03_09_nanoArmMount" mass="0.008" cog="-0.002400 0.0046958 0.0115245">
+			<xacro:insert_block name="default_inertial"/>
+        </xacro:camera_assembly_link>
 	  	<xacro:camera_assembly_joint joint_name="nanoMount_to_world" parent="${base_parent}" child="nanoMount" joint_origin_xyz="${base_xyz}" joint_origin_rpy="${base_rpy}"/>
-		<xacro:camera_assembly_link link_name="enclosureBottom" link_mesh="2023_03_16_nanoEnclosureBottom"/>
+		<xacro:camera_assembly_link link_name="enclosureBottom" link_mesh="2023_03_16_nanoEnclosureBottom" mass="0.040" cog="0.0546451 0.0472161 0.00043655">
+	  		<xacro:insert_block name="default_inertial"/>
+	  	</xacro:camera_assembly_link>
 		<xacro:camera_assembly_joint joint_name="enclosureBottom_to_nanoMount" parent="nanoMount" child="enclosureBottom" joint_origin_xyz="0.0412 -0.0218 0.026" joint_origin_rpy="0 0 ${J_PI/2}"/>
-		<xacro:camera_assembly_link link_name="nano" link_mesh="2023_03_21_jetsonNano"/>
+		<xacro:camera_assembly_link link_name="nano" link_mesh="2023_03_21_jetsonNano" mass="0.142" cog="0.0435615 0.02502709 0.0091247">
+	  		<xacro:insert_block name="default_inertial"/>
+	  	</xacro:camera_assembly_link>
 		<xacro:camera_assembly_joint joint_name="nano_to_enclosureBottom" parent="enclosureBottom" child="nano" joint_origin_xyz="0.0105 0.014 -0.0015" joint_origin_rpy="0 0 0"/>
-		<xacro:camera_assembly_link link_name="enclosureTop" link_mesh="2023_03_09_nanoEnclosureTop"/>
+		<xacro:camera_assembly_link link_name="enclosureTop" link_mesh="2023_03_09_nanoEnclosureTop" mass="0.046" cog="0.04817211 0.03496864 0.02671124">
+	  		<xacro:insert_block name="default_inertial"/>
+	  	</xacro:camera_assembly_link>
 		<xacro:camera_assembly_joint joint_name="enclosureTop_to_enclosureBottom" parent="enclosureBottom" child="enclosureTop" joint_origin_xyz="0 0 0" joint_origin_rpy="0 0 0"/>
-		<xacro:camera_assembly_link link_name="stabilizer" link_mesh="2023_03_09_cameraStabilizer"/>
+		<xacro:camera_assembly_link link_name="stabilizer" link_mesh="2023_03_09_cameraStabilizer" mass="0.004" cog="0.00272454 0.00000231884 0.00514249">
+	  		<xacro:insert_block name="default_inertial"/>
+	  	</xacro:camera_assembly_link>
 		<xacro:camera_assembly_joint joint_name="stabilizer_to_enclosureTop" parent="enclosureTop" child="stabilizer" joint_origin_xyz="0.0842 0.041 0.0343" joint_origin_rpy="0 ${14.621 * J_PI / 180} 0"/>
 		<xacro:sensor_d415 parent="stabilizer" use_mesh="true" name="uncalibrated_camera">

File: ada_description/urdf/forque/forque.xacro (robot description, xacro)
@@ -15,5 +15,4 @@
 	<xacro:property name="forque_color" value="0.4 0.4 0.4 1" />
 	<xacro:property name="J_PI" value="3.1415926535897931" />
-	<xacro:property name="default_origin" value="0 0 0"/>
 	<xacro:property name="default_inertial">
 		<inertia ixx="0.001" iyy="0.001" iyz="0.001" izz="0.001" ixy="0.001" ixz="0.001"/>
@@ -55,24 +54,24 @@
 	<xacro:macro name="forque_assembly" params="base_parent">
 		<xacro:forque_assembly_link link_name="FTMount" link_mesh="2023_03_09_FTMount" mass="0.022" cog="0.0111797 -0.110193 -0.0384312">
-			<inertia ixx="0.00000047293" iyy="7871700" iyz="0.001" izz="0.001" ixy="0.001" ixz="0.001"/>
+			<xacro:insert_block name="default_inertial"/>
         </xacro:forque_assembly_link>
 	  	<xacro:forque_assembly_joint joint_name="FTMount_to_world" parent="${base_parent}" child="FTMount" joint_origin_xyz="0 0 0" joint_origin_rpy="0 0 0"/>
-	  	<xacro:forque_assembly_link link_name="FT" link_mesh="2023_03_09_wirelessFT" mass="0.278">
+	  	<xacro:forque_assembly_link link_name="FT" link_mesh="2023_03_09_wirelessFT" mass="0.280" cog="0.0111446 -0.0882070 -0.0544936">
 	  		<xacro:insert_block name="default_inertial"/>
 	  	</xacro:forque_assembly_link>
 	  	<xacro:forque_assembly_joint joint_name="FT_to_FTMount" parent="FTMount" child="FT" joint_origin_xyz="0 0 0" joint_origin_rpy="0 0 0"/>
-	  	<xacro:forque_assembly_link link_name="FTAntenna" link_mesh="2023_03_09_wirelessFTAntenna">
+	  	<xacro:forque_assembly_link link_name="FTAntenna" link_mesh="2023_03_09_wirelessFTAntenna" mass="0.018" cog="-0.0162965 0.0666626 -0.0545096">
 	  		<xacro:insert_block name="default_inertial"/>
 	  	</xacro:forque_assembly_link>
 	  	<xacro:forque_assembly_joint joint_name="FTAntenna_to_FT" parent="FT" child="FTAntenna" joint_origin_xyz="0 0 0" joint_origin_rpy="0 0 0"/>
-	  	<xacro:forque_assembly_link link_name="forkHandle" link_mesh="2023_03_09_forkHandle">
+	  	<xacro:forque_assembly_link link_name="forkHandle" link_mesh="2023_03_09_forkHandle" mass="0.0506" cog="0.0110024 -0.151715 -0.00934664">
 	  		<xacro:insert_block name="default_inertial"/>
 	  	</xacro:forque_assembly_link>
 	  	<xacro:forque_assembly_joint joint_name="forkHandle_to_FTMount" parent="FTMount" child="forkHandle" joint_origin_xyz="0 0 0" joint_origin_rpy="0 0 0"/>
-	  	<xacro:forque_assembly_link link_name="forque" link_mesh="ATI-9105-TW-NANO25-E">
+	  	<xacro:forque_assembly_link link_name="forque" link_mesh="ATI-9105-TW-NANO25-E" mass="0.0634" cog="0.0124692 0.0137169 0.010558">
 	  		<xacro:insert_block name="default_inertial"/>
 	  	</xacro:forque_assembly_link>
 	  	<xacro:forque_assembly_joint joint_name="forque_to_forkHandle" parent="forkHandle" child="forque" joint_origin_xyz="-0.00634 -0.222553 -0.004286" joint_origin_rpy="${J_PI/2} ${J_PI/3} 0"/>
-	  	<xacro:forque_assembly_link link_name="forkTine" link_mesh="fork_tine">
+	  	<xacro:forque_assembly_link link_name="forkTine" link_mesh="fork_tine" mass="0.024" cog="0.013090 0.0180789 0.0445231">
 	  		<xacro:insert_block name="default_inertial"/>
 	  	</xacro:forque_assembly_link>

Commit message: Added screws on camera mount to urdf and disabled collisions between camera mount and arm links 3&4

File: ada_description/urdf/camera/camera.xacro (robot description, xacro)
@@ -79,7 +79,15 @@
 	  	</xacro:camera_assembly_link>
 		<xacro:camera_assembly_joint joint_name="cameraMount_to_enclosureTop" parent="enclosureTop" child="cameraMount" joint_origin_xyz="-0.0132 0 -0.022" joint_origin_rpy="0 ${J_PI / 2} 0"/>
-		<xacro:sensor_d415 parent="cameraMount" use_mesh="true" name="uncalibrated_camera">
-			<origin xyz="0.006 0 0.013" rpy="0 ${-J_PI / 2} ${J_PI}" />
-		</xacro:sensor_d415>
+		<xacro:camera_assembly_link link_name="screwHeadLeft" link_mesh="2023_11_07_screwHead" mass="0.0001" cog="0 0 0">
+     		<xacro:insert_block name="default_inertial"/>
+     	</xacro:camera_assembly_link>
+   	 	<xacro:camera_assembly_joint joint_name="screwHeadLeft_to_cameraMount" parent="cameraMount" child="screwHeadLeft" joint_origin_xyz="0.0165 -0.0225 0" joint_origin_rpy="${J_PI} 0 0"/>
+   	 	<xacro:camera_assembly_link link_name="screwHeadRight" link_mesh="2023_11_07_screwHead" mass="0.0001" cog="0 0 0">
+     		<xacro:insert_block name="default_inertial"/>
+     	</xacro:camera_assembly_link>
+   	 	<xacro:camera_assembly_joint joint_name="screwHeadRight_to_cameraMount" parent="cameraMount" child="screwHeadRight" joint_origin_xyz="0.0165 0.0225 0" joint_origin_rpy="${J_PI} 0 0"/>
+   	 	<xacro:sensor_d415 parent="cameraMount" use_mesh="true" name="uncalibrated_camera">
+   		 	<origin xyz="0.006 0 0.013" rpy="0 ${-J_PI / 2} ${J_PI}" />
+   	 	</xacro:sensor_d415>
 	</xacro:macro>
 </root>

Commit message: [WIP] Adding moment of inertia values to components

File: ada_description/urdf/camera/camera.xacro (robot description, xacro)
@@ -60,5 +60,5 @@
 	  	<xacro:camera_assembly_joint joint_name="nanoMount_to_world" parent="${base_parent}" child="nanoMount" joint_origin_xyz="${base_xyz}" joint_origin_rpy="${base_rpy}"/>
 		<xacro:camera_assembly_link link_name="enclosureBottom" link_mesh="2023_09_28_nanoEnclosureBottom" mass="0.040" cog="0.0546451 0.0472161 0.00043655">
-	  		<xacro:insert_block name="default_inertial"/>
+	  		<inertia ixx="0.000041028" iyy="0.000083168" iyz="0.0000026243" izz="0.000116424" ixy="-0.000000324" ixz="-0.00000045367"/>
 	  	</xacro:camera_assembly_link>
 		<xacro:camera_assembly_joint joint_name="enclosureBottom_to_nanoMount" parent="nanoMount" child="enclosureBottom" joint_origin_xyz="0.0412 -0.0218 0.026" joint_origin_rpy="0 0 ${J_PI/2}"/>

Commit message: [WIP] Adding moment of inertia values to components, enclosure top and bottom complete

File: ada_description/urdf/camera/camera.xacro (robot description, xacro)
@@ -56,5 +56,5 @@
 	<xacro:macro name="camera_assembly" params="base_parent base_xyz:=${default_origin} base_rpy:=${default_origin}">
 		<xacro:camera_assembly_link link_name="nanoMount" link_mesh="2023_03_09_nanoArmMount" mass="0.008" cog="-0.002400 0.0046958 0.0115245">
-			<xacro:insert_block name="default_inertial"/>
+			<inertia ixx="0.00000095025" iyy="0.0000067325" iyz="0.000000000470196" izz="0.0000069433" ixy="-0.000000297842" ixz="-0.00000000010444"/>
         </xacro:camera_assembly_link>
 	  	<xacro:camera_assembly_joint joint_name="nanoMount_to_world" parent="${base_parent}" child="nanoMount" joint_origin_xyz="${base_xyz}" joint_origin_rpy="${base_rpy}"/>
@@ -72,5 +72,5 @@
 		<xacro:camera_assembly_joint joint_name="frontStabilizer_to_enclosureBottom" parent="enclosureBottom" child="frontStabilizer" joint_origin_xyz="0.1063 0.0493 -0.0363" joint_origin_rpy="0 0 ${J_PI/2}"/>
 		<xacro:camera_assembly_link link_name="enclosureTop" link_mesh="2023_06_06_nanoEnclosureTopCameraBack" mass="0.046" cog="0.04817211 0.03496864 0.02671124">
-	  		<xacro:insert_block name="default_inertial"/>
+	  		<inertia ixx="0.00005942" iyy="0.000085611" iyz="0.0000012783" izz="0.000126390" ixy="-0.000000046193" ixz="0.0000091699"/>
 	  	</xacro:camera_assembly_link>
 		<xacro:camera_assembly_joint joint_name="enclosureTop_to_enclosureBottom" parent="enclosureBottom" child="enclosureTop" joint_origin_xyz="0.009925 0.04099 0.05442" joint_origin_rpy="0 ${165.4 * J_PI / 180} ${J_PI}"/>

Commit message: [WIP] Added inertia values for the front stabilizer

File: ada_description/urdf/camera/camera.xacro (robot description, xacro)
@@ -68,5 +68,5 @@
 		<xacro:camera_assembly_joint joint_name="nano_to_enclosureBottom" parent="enclosureBottom" child="nano" joint_origin_xyz="0.0105 0.014 -0.0015" joint_origin_rpy="0 0 0"/>
 		<xacro:camera_assembly_link link_name="frontStabilizer" link_mesh="2023_09_21_nanoEnclosureFrontStabilizer" mass="0.0198" cog="-0.008107 -0.000955 0.02045">
-	  		<xacro:insert_block name="default_inertial"/>
+	  		<inertia ixx="0.00000074776" iyy="0.0000118843" iyz="0.00001021778" izz="0.0000119096" ixy="0.000000000071856" ixz="0.0000000002764"/>
 	  	</xacro:camera_assembly_link>
 		<xacro:camera_assembly_joint joint_name="frontStabilizer_to_enclosureBottom" parent="enclosureBottom" child="frontStabilizer" joint_origin_xyz="0.1063 0.0493 -0.0363" joint_origin_rpy="0 0 ${J_PI/2}"/>
