Commit message: Added inertia tensors for the Jetson nano and improved the default inertial block

File: ada_description/urdf/camera/camera.xacro (robot description, xacro)
@@ -17,5 +17,5 @@
 	<xacro:property name="J_PI" value="3.1415926535897931" />
 	<xacro:property name="default_inertial">
-		<inertia ixx="0.001" iyy="0.001" iyz="0.001" izz="0.001" ixy="0.001" ixz="0.001"/>
+		<inertia ixx="0.000005" iyy="0.000005" iyz="0" izz="0.000005" ixy="0" ixz="0"/>
 	</xacro:property>
 	<xacro:macro name="camera_assembly_link" params="link_name link_mesh mass:=0 cog:='0 0 0' *inertia">
@@ -64,9 +64,9 @@
 		<xacro:camera_assembly_joint joint_name="enclosureBottom_to_nanoMount" parent="nanoMount" child="enclosureBottom" joint_origin_xyz="0.0412 -0.0218 0.026" joint_origin_rpy="0 0 ${J_PI/2}"/>
 		<xacro:camera_assembly_link link_name="nano" link_mesh="2023_03_21_jetsonNano" mass="0.142" cog="0.0435615 0.02502709 0.0091247">
-	  		<xacro:insert_block name="default_inertial"/>
+	  		<inertia ixx="0.000077456" iyy="0.0001013" iyz="0.0000036951" izz="0.0001727" ixy="-0.000004935" ixz="0.0000015461"/>
 	  	</xacro:camera_assembly_link>
 		<xacro:camera_assembly_joint joint_name="nano_to_enclosureBottom" parent="enclosureBottom" child="nano" joint_origin_xyz="0.0105 0.014 -0.0015" joint_origin_rpy="0 0 0"/>
 		<xacro:camera_assembly_link link_name="frontStabilizer" link_mesh="2023_09_21_nanoEnclosureFrontStabilizer" mass="0.0198" cog="-0.008107 -0.000955 0.02045">
-	  		<inertia ixx="0.00000074776" iyy="0.0000118843" iyz="0.00001021778" izz="0.0000119096" ixy="0.000000000071856" ixz="0.0000000002764"/>
+	  		<inertia ixx="0.00000074776" iyy="0.0000118843" iyz="0.00000001021778" izz="0.0000119096" ixy="0.000000000071856" ixz="0.0000000002764"/>
 	  	</xacro:camera_assembly_link>
 		<xacro:camera_assembly_joint joint_name="frontStabilizer_to_enclosureBottom" parent="enclosureBottom" child="frontStabilizer" joint_origin_xyz="0.1063 0.0493 -0.0363" joint_origin_rpy="0 0 ${J_PI/2}"/>
@@ -75,5 +75,5 @@
 	  	</xacro:camera_assembly_link>
 		<xacro:camera_assembly_joint joint_name="enclosureTop_to_enclosureBottom" parent="enclosureBottom" child="enclosureTop" joint_origin_xyz="0.009925 0.04099 0.05442" joint_origin_rpy="0 ${165.4 * J_PI / 180} ${J_PI}"/>
-		<xacro:camera_assembly_link link_name="cameraMount" link_mesh="2023_06_06_cameraBackMount" mass="0.004" cog="0.00272454 0.00000231884 0.00514249">
+		<xacro:camera_assembly_link link_name="cameraMount" link_mesh="2023_06_06_cameraBackMount" mass="0.004" cog="-0.007986 0 0.010064">
 	  		<xacro:insert_block name="default_inertial"/>
 	  	</xacro:camera_assembly_link>

File: ada_description/urdf/forque/forque.xacro (robot description, xacro)
@@ -16,5 +16,5 @@
 	<xacro:property name="J_PI" value="3.1415926535897931" />
 	<xacro:property name="default_inertial">
-		<inertia ixx="0.001" iyy="0.001" iyz="0.001" izz="0.001" ixy="0.001" ixz="0.001"/>
+		<inertia ixx="0.000005" iyy="0.000005" iyz="0" izz="0.000005" ixy="0" ixz="0"/>
 	</xacro:property>
 	<xacro:macro name="forque_assembly_link" params="link_name link_mesh mass:=0 cog:='0 0 0' *inertia">

Commit message: [WIP] added inertia values for the camera mount

File: ada_description/urdf/camera/camera.xacro (robot description, xacro)
@@ -76,5 +76,5 @@
 		<xacro:camera_assembly_joint joint_name="enclosureTop_to_enclosureBottom" parent="enclosureBottom" child="enclosureTop" joint_origin_xyz="0.009925 0.04099 0.05442" joint_origin_rpy="0 ${165.4 * J_PI / 180} ${J_PI}"/>
 		<xacro:camera_assembly_link link_name="cameraMount" link_mesh="2023_06_06_cameraBackMount" mass="0.004" cog="-0.007986 0 0.010064">
-	  		<xacro:insert_block name="default_inertial"/>
+	  		<inertia ixx="0.000002782" iyy="00.0000005528" iyz="-0.00000000000178" izz="0.000002964" ixy="-0.00000000002321" ixz="0.000000074385"/>
 	  	</xacro:camera_assembly_link>
 		<xacro:camera_assembly_joint joint_name="cameraMount_to_enclosureTop" parent="enclosureTop" child="cameraMount" joint_origin_xyz="-0.0132 0 -0.022" joint_origin_rpy="0 ${J_PI / 2} 0"/>

Commit message: Added Inertia Values To URDF (#44)
* [WIP] Adding moment of inertia values to components

* [WIP] Adding moment of inertia values to components, enclosure top and bottom complete

* [WIP] Added inertia values for the front stabilizer

* Added inertia tensors for the Jetson nano and improved the default inertial block

* [WIP] added inertia values for the camera mount

* Added moment of inertia values for all remaining components and fixed top enclosure center of mass

* Fixed formatting

File: ada_description/urdf/camera/camera.xacro (robot description, xacro)
@@ -17,5 +17,5 @@
 	<xacro:property name="J_PI" value="3.1415926535897931" />
 	<xacro:property name="default_inertial">
-		<inertia ixx="0.001" iyy="0.001" iyz="0.001" izz="0.001" ixy="0.001" ixz="0.001"/>
+		<inertia ixx="0.000005" iyy="0.000005" iyz="0" izz="0.000005" ixy="0" ixz="0"/>
 	</xacro:property>
 	<xacro:macro name="camera_assembly_link" params="link_name link_mesh mass:=0 cog:='0 0 0' *inertia">
@@ -56,33 +56,33 @@
 	<xacro:macro name="camera_assembly" params="base_parent base_xyz:=${default_origin} base_rpy:=${default_origin}">
 		<xacro:camera_assembly_link link_name="nanoMount" link_mesh="2023_03_09_nanoArmMount" mass="0.008" cog="-0.002400 0.0046958 0.0115245">
-			<xacro:insert_block name="default_inertial"/>
+			<inertia ixx="0.00000095025" iyy="0.0000067325" iyz="0.000000000470196" izz="0.0000069433" ixy="-0.000000297842" ixz="-0.00000000010444"/>
         </xacro:camera_assembly_link>
 	  	<xacro:camera_assembly_joint joint_name="nanoMount_to_world" parent="${base_parent}" child="nanoMount" joint_origin_xyz="${base_xyz}" joint_origin_rpy="${base_rpy}"/>
 		<xacro:camera_assembly_link link_name="enclosureBottom" link_mesh="2023_09_28_nanoEnclosureBottom" mass="0.040" cog="0.0546451 0.0472161 0.00043655">
-	  		<xacro:insert_block name="default_inertial"/>
+	  		<inertia ixx="0.000041028" iyy="0.000083168" iyz="0.0000026243" izz="0.000116424" ixy="-0.000000324" ixz="-0.00000045367"/>
 	  	</xacro:camera_assembly_link>
 		<xacro:camera_assembly_joint joint_name="enclosureBottom_to_nanoMount" parent="nanoMount" child="enclosureBottom" joint_origin_xyz="0.0412 -0.0218 0.026" joint_origin_rpy="0 0 ${J_PI/2}"/>
 		<xacro:camera_assembly_link link_name="nano" link_mesh="2023_03_21_jetsonNano" mass="0.142" cog="0.0435615 0.02502709 0.0091247">
-	  		<xacro:insert_block name="default_inertial"/>
+	  		<inertia ixx="0.000077456" iyy="0.0001013" iyz="0.0000036951" izz="0.0001727" ixy="-0.000004935" ixz="0.0000015461"/>
 	  	</xacro:camera_assembly_link>
 		<xacro:camera_assembly_joint joint_name="nano_to_enclosureBottom" parent="enclosureBottom" child="nano" joint_origin_xyz="0.0105 0.014 -0.0015" joint_origin_rpy="0 0 0"/>
 		<xacro:camera_assembly_link link_name="frontStabilizer" link_mesh="2023_09_21_nanoEnclosureFrontStabilizer" mass="0.0198" cog="-0.008107 -0.000955 0.02045">
-	  		<xacro:insert_block name="default_inertial"/>
+	  		<inertia ixx="0.00000074776" iyy="0.0000118843" iyz="0.00000001021778" izz="0.0000119096" ixy="0.000000000071856" ixz="0.0000000002764"/>
 	  	</xacro:camera_assembly_link>
 		<xacro:camera_assembly_joint joint_name="frontStabilizer_to_enclosureBottom" parent="enclosureBottom" child="frontStabilizer" joint_origin_xyz="0.1063 0.0493 -0.0363" joint_origin_rpy="0 0 ${J_PI/2}"/>
-		<xacro:camera_assembly_link link_name="enclosureTop" link_mesh="2023_06_06_nanoEnclosureTopCameraBack" mass="0.046" cog="0.04817211 0.03496864 0.02671124">
-	  		<xacro:insert_block name="default_inertial"/>
+		<xacro:camera_assembly_link link_name="enclosureTop" link_mesh="2023_06_06_nanoEnclosureTopCameraBack" mass="0.046" cog="0.041228 0.006275 0.016379">
+	  		<inertia ixx="0.00005942" iyy="0.000085611" iyz="0.0000012783" izz="0.000126390" ixy="-0.000000046193" ixz="0.0000091699"/>
 	  	</xacro:camera_assembly_link>
 		<xacro:camera_assembly_joint joint_name="enclosureTop_to_enclosureBottom" parent="enclosureBottom" child="enclosureTop" joint_origin_xyz="0.009925 0.04099 0.05442" joint_origin_rpy="0 ${165.4 * J_PI / 180} ${J_PI}"/>
-		<xacro:camera_assembly_link link_name="cameraMount" link_mesh="2023_06_06_cameraBackMount" mass="0.004" cog="0.00272454 0.00000231884 0.00514249">
-	  		<xacro:insert_block name="default_inertial"/>
+		<xacro:camera_assembly_link link_name="cameraMount" link_mesh="2023_06_06_cameraBackMount" mass="0.004" cog="-0.007986 0 0.010064">
+	  		<inertia ixx="0.000002782" iyy="00.0000005528" iyz="-0.00000000000178" izz="0.000002964" ixy="-0.00000000002321" ixz="0.000000074385"/>
 	  	</xacro:camera_assembly_link>
 		<xacro:camera_assembly_joint joint_name="cameraMount_to_enclosureTop" parent="enclosureTop" child="cameraMount" joint_origin_xyz="-0.0132 0 -0.022" joint_origin_rpy="0 ${J_PI / 2} 0"/>
-		<xacro:camera_assembly_link link_name="screwHeadLeft" link_mesh="2023_11_07_screwHead" mass="0.0001" cog="0 0 0">
-     		<xacro:insert_block name="default_inertial"/>
+		<xacro:camera_assembly_link link_name="screwHeadLeft" link_mesh="2023_11_07_screwHead" mass="0.0001" cog="0 0 0.0015">
+     		<inertia ixx="0.000000000342785" iyy="0.000000000342785" iyz="0" izz="0.000000000543538" ixy="0" ixz="0"/>
      	</xacro:camera_assembly_link>
    	 	<xacro:camera_assembly_joint joint_name="screwHeadLeft_to_cameraMount" parent="cameraMount" child="screwHeadLeft" joint_origin_xyz="0.0165 -0.0225 0" joint_origin_rpy="${J_PI} 0 0"/>
-   	 	<xacro:camera_assembly_link link_name="screwHeadRight" link_mesh="2023_11_07_screwHead" mass="0.0001" cog="0 0 0">
-     		<xacro:insert_block name="default_inertial"/>
+   	 	<xacro:camera_assembly_link link_name="screwHeadRight" link_mesh="2023_11_07_screwHead" mass="0.0001" cog="0 0 0.0015">
+     		<inertia ixx="0.000000000342785" iyy="0.000000000342785" iyz="0" izz="0.000000000543538" ixy="0" ixz="0"/>
      	</xacro:camera_assembly_link>
    	 	<xacro:camera_assembly_joint joint_name="screwHeadRight_to_cameraMount" parent="cameraMount" child="screwHeadRight" joint_origin_xyz="0.0165 0.0225 0" joint_origin_rpy="${J_PI} 0 0"/>

File: ada_description/urdf/forque/forque.xacro (robot description, xacro)
@@ -16,5 +16,5 @@
 	<xacro:property name="J_PI" value="3.1415926535897931" />
 	<xacro:property name="default_inertial">
-		<inertia ixx="0.001" iyy="0.001" iyz="0.001" izz="0.001" ixy="0.001" ixz="0.001"/>
+		<inertia ixx="0.000005" iyy="0.000005" iyz="0" izz="0.000005" ixy="0" ixz="0"/>
 	</xacro:property>
 	<xacro:macro name="forque_assembly_link" params="link_name link_mesh mass:=0 cog:='0 0 0' *inertia">
@@ -54,9 +54,9 @@
 	<xacro:macro name="forque_assembly" params="base_parent use_antenna:=false">
 		<xacro:forque_assembly_link link_name="FTMount" link_mesh="2024_01_18_FTMount" mass="0.103" cog="0.010934 -0.138522 -0.05066">
-			<xacro:insert_block name="default_inertial"/>
+			<inertia ixx="0.00017623" iyy="0.000068428" iyz="-0.00001757133" izz="0.00021455" ixy="0.00000095729" ixz="-0.0000000562908"/>
         </xacro:forque_assembly_link>
 	  	<xacro:forque_assembly_joint joint_name="FTMount_to_world" parent="${base_parent}" child="FTMount" joint_origin_xyz="0 0 -0.005" joint_origin_rpy="0 0 0"/>
 	  	<xacro:forque_assembly_link link_name="FT" link_mesh="2023_03_09_wirelessFT" mass="0.280" cog="0.0111446 -0.0882070 -0.0544936">
-	  		<xacro:insert_block name="default_inertial"/>
+	  		<inertia ixx="0.000543925" iyy="0.000165428" iyz="-0.00000001487288" izz="0.000691232" ixy="-0.00000128367" ixz="0"/>
 	  	</xacro:forque_assembly_link>
 	  	<xacro:forque_assembly_joint joint_name="FT_to_FTMount" parent="FTMount" child="FT" joint_origin_xyz="0 0 0" joint_origin_rpy="0 0 0"/>
@@ -68,14 +68,14 @@
 		  </xacro:if>
 	  	<xacro:forque_assembly_link link_name="forkHandle" link_mesh="2023_03_09_forkHandle" mass="0.0506" cog="0.0110024 -0.151715 -0.00934664">
-	  		<xacro:insert_block name="default_inertial"/>
+	  		<inertia ixx="0.0000418078" iyy="0.0000177249" iyz="-0.000000210639" izz="0.00005200336" ixy="-0.000000396292" ixz="0.00000002424697"/>
 	  	</xacro:forque_assembly_link>
 		<!-- The slight rotation was manually added due to empirical deformations in the robot gripped, such that the fingers and fork handle were slightly pitched up relative to the wrist. -->
 		<xacro:forque_assembly_joint joint_name="forkHandle_to_FTMount" parent="FTMount" child="forkHandle" joint_origin_xyz="0 0 0.005" joint_origin_rpy="-0.025 0 0"/>
 	  	<xacro:forque_assembly_link link_name="forque" link_mesh="ATI-9105-TW-NANO25-E" mass="0.0634" cog="0.0124692 0.0137169 0.010558">
-	  		<xacro:insert_block name="default_inertial"/>
+	  		<inertia ixx="0.000005235822" iyy="0.000006264852" iyz="-0.00000004033694" izz="0.00000640797" ixy="-0.0000003129932" ixz="0.000000013798"/>
 	  	</xacro:forque_assembly_link>
 	  	<xacro:forque_assembly_joint joint_name="forque_to_forkHandle" parent="forkHandle" child="forque" joint_origin_xyz="-0.00634 -0.222553 -0.004286" joint_origin_rpy="${J_PI/2} ${J_PI/3} 0"/>
 	  	<xacro:forque_assembly_link link_name="forkTine" link_mesh="fork_tine" mass="0.024" cog="0.013090 0.0180789 0.0445231">
-	  		<xacro:insert_block name="default_inertial"/>
+	  		<inertia ixx="0.0000098769" iyy="0.000009848103" iyz="0.00000057639" izz="0.0000015674" ixy="0.000000000806182" ixz="-0.00000000296036"/>
 	  	</xacro:forque_assembly_link>
 	  	<xacro:forque_assembly_joint joint_name="forkTine_to_forque" parent="forque" child="forkTine" joint_origin_xyz="-0.0054 0.008 0.093" joint_origin_rpy="0 ${J_PI} ${240*J_PI/180}"/>
