Commit message: Working IsaacSim Hardware Interface

File: ada_hardware/urdf/ada_hardware.ros2_control.xacro (robot description, xacro)
@@ -1,15 +1,19 @@
 <?xml version="1.0"?>
 <robot xmlns:xacro="http://www.ros.org/wiki/xacro">
-  <xacro:macro name="ada_hardware_interface" params="name prefix:=j2n6s200 use_mock_hardware:=^|true">
+  <xacro:macro name="ada_hardware_interface" params="name prefix:=j2n6s200 sim">
     <ros2_control name="${name}" type="system">
       <hardware>
-        <xacro:if value="${use_mock_hardware}">
+        <xacro:if value="${sim == 'mock'}">
           <plugin>mock_components/GenericSystem</plugin>
           <param name="mock_sensor_commands">false</param>
           <param name="state_following_offset">0.0</param>
         </xacro:if>
-        <xacro:unless value="${use_mock_hardware}">
+        <xacro:if value="${sim == 'isaac'}">
+          <plugin>ada_hardware/JacoIsaac</plugin>
+          <param name="namespace">/simulation</param>
+        </xacro:if>
+        <xacro:if value="${sim == 'none'}">
           <plugin>ada_hardware/Jaco2</plugin>
-        </xacro:unless>
+        </xacro:if>
       </hardware>
       <!-- Arm DOFs -->

File: ada_hardware/urdf/ada_hardware.xacro (robot description, xacro)
@@ -3,9 +3,9 @@
 <robot xmlns:xi="http://www.w3.org/2001/XInclude"
 	xmlns:xacro="http://www.ros.org/wiki/xacro" name="ada_hardware">
-  <xacro:arg name="use_mock_hardware" default="false" />
+  <xacro:arg name="use_mock_hardware" default="none" />
   <xacro:include filename="$(find ada_description)/urdf/ada.xacro"/>
   <xacro:include filename="$(find ada_hardware)/urdf/ada_hardware.ros2_control.xacro"/>
   <xacro:ada_hardware_interface
     name="Jaco2"
-    use_mock_hardware="$(arg use_mock_hardware)" />
+    sim="$(arg sim)" />
 </robot>

Commit message: Added readonly to Jaco2 HW interface

File: ada_hardware/urdf/ada_hardware.ros2_control.xacro (robot description, xacro)
@@ -1,5 +1,5 @@
 <?xml version="1.0"?>
 <robot xmlns:xacro="http://www.ros.org/wiki/xacro">
-  <xacro:macro name="ada_hardware_interface" params="name prefix:=j2n6s200 sim">
+  <xacro:macro name="ada_hardware_interface" params="name prefix:=j2n6s200 sim readonly:=false">
     <ros2_control name="${name}" type="system">
       <hardware>
@@ -19,7 +19,9 @@
       <!-- Arm DOFs -->
       <joint name="${prefix}_joint_1">
-        <command_interface name="position"/>
-        <command_interface name="velocity"/>
-        <command_interface name="effort"/>
+        <xacro:unless value="${readonly}">
+          <command_interface name="position"/>
+          <command_interface name="velocity"/>
+          <command_interface name="effort"/>
+        </xacro:unless>
         <state_interface name="position"/>
         <state_interface name="velocity"/>
@@ -27,7 +29,9 @@
       </joint>
       <joint name="${prefix}_joint_2">
-        <command_interface name="position"/>
-        <command_interface name="velocity"/>
-        <command_interface name="effort"/>
+        <xacro:unless value="${readonly}">
+          <command_interface name="position"/>
+          <command_interface name="velocity"/>
+          <command_interface name="effort"/>
+        </xacro:unless>
         <state_interface name="position"/>
         <state_interface name="velocity"/>
@@ -35,7 +39,9 @@
       </joint>
       <joint name="${prefix}_joint_3">
-        <command_interface name="position"/>
-        <command_interface name="velocity"/>
-        <command_interface name="effort"/>
+        <xacro:unless value="${readonly}">
+          <command_interface name="position"/>
+          <command_interface name="velocity"/>
+          <command_interface name="effort"/>
+        </xacro:unless>
         <state_interface name="position"/>
         <state_interface name="velocity"/>
@@ -43,7 +49,9 @@
       </joint>
       <joint name="${prefix}_joint_4">
-        <command_interface name="position"/>
-        <command_interface name="velocity"/>
-        <command_interface name="effort"/>
+        <xacro:unless value="${readonly}">
+          <command_interface name="position"/>
+          <command_interface name="velocity"/>
+          <command_interface name="effort"/>
+        </xacro:unless>
         <state_interface name="position"/>
         <state_interface name="velocity"/>
@@ -51,7 +59,9 @@
       </joint>
       <joint name="${prefix}_joint_5">
-        <command_interface name="position"/>
-        <command_interface name="velocity"/>
-        <command_interface name="effort"/>
+        <xacro:unless value="${readonly}">
+          <command_interface name="position"/>
+          <command_interface name="velocity"/>
+          <command_interface name="effort"/>
+        </xacro:unless>
         <state_interface name="position"/>
         <state_interface name="velocity"/>
@@ -59,7 +69,9 @@
       </joint>
       <joint name="${prefix}_joint_6">
-        <command_interface name="position"/>
-        <command_interface name="velocity"/>
-        <command_interface name="effort"/>
+        <xacro:unless value="${readonly}">
+          <command_interface name="position"/>
+          <command_interface name="velocity"/>
+          <command_interface name="effort"/>
+        </xacro:unless>
         <state_interface name="position"/>
         <state_interface name="velocity"/>
@@ -68,7 +80,9 @@
       <!-- Finger DOFs -->
       <joint name="${prefix}_joint_finger_1">
-        <command_interface name="position"/>
-        <command_interface name="velocity"/>
-        <command_interface name="effort"/>
+        <xacro:unless value="${readonly}">
+          <command_interface name="position"/>
+          <command_interface name="velocity"/>
+          <command_interface name="effort"/>
+        </xacro:unless>
         <state_interface name="position"/>
         <state_interface name="velocity"/>
@@ -76,7 +90,9 @@
       </joint>
       <joint name="${prefix}_joint_finger_2">
-        <command_interface name="position"/>
-        <command_interface name="velocity"/>
-        <command_interface name="effort"/>
+        <xacro:unless value="${readonly}">
+          <command_interface name="position"/>
+          <command_interface name="velocity"/>
+          <command_interface name="effort"/>
+        </xacro:unless>
         <state_interface name="position"/>
         <state_interface name="velocity"/>

File: ada_hardware/urdf/ada_hardware.xacro (robot description, xacro)
@@ -4,8 +4,10 @@
 	xmlns:xacro="http://www.ros.org/wiki/xacro" name="ada_hardware">
   <xacro:arg name="sim" default="none" />
+  <xacro:arg name="readonly" default="false" />
   <xacro:include filename="$(find ada_description)/urdf/ada.xacro"/>
   <xacro:include filename="$(find ada_hardware)/urdf/ada_hardware.ros2_control.xacro"/>
   <xacro:ada_hardware_interface
     name="Jaco2"
-    sim="$(arg sim)" />
+    sim="$(arg sim)"
+    readonly="$(arg readonly)" />
 </robot>

Commit message: Add hardware interface for Dynamixels

File: ada_hardware/urdf/ada_hardware.ros2_control.xacro (robot description, xacro)
@@ -101,3 +101,41 @@
     </ros2_control>
   </xacro:macro>
+  <xacro:macro name="dynamixel_hardware_interface" params="name sim readonly:=false">
+    <ros2_control name="${name}" type="system">
+      <hardware>
+        <xacro:if value="${sim == 'mock'}">
+          <plugin>mock_components/GenericSystem</plugin>
+          <param name="mock_sensor_commands">false</param>
+          <param name="state_following_offset">0.0</param>
+        </xacro:if>
+        <xacro:if value="${sim == 'none'}">
+          <plugin>ada_hardware/Dynamixel</plugin>
+          <param name="port" value="/dev/ttyUSB0" />
+          <param name="baud_rate" value="1000000" />
+        </xacro:if>
+      </hardware>
+      <joint name="AFMotor1_to_AFBase">
+        <param name="id">1</param>
+        <xacro:unless value="${readonly}">
+          <command_interface name="position" />
+          <command_interface name="velocity" />
+          <!-- <command_interface name="effort" /> -->
+        </xacro:unless>
+        <state_interface name="position" />
+        <state_interface name="velocity" />
+        <state_interface name="effort" />
+      </joint>
+      <joint name="AFFTAdapter_to_AFMotor2">
+        <param name="id">2</param>
+        <xacro:unless value="${readonly}">
+          <command_interface name="position" />
+          <command_interface name="velocity" />
+          <!-- <command_interface name="effort" /> -->
+        </xacro:unless>
+        <state_interface name="position" />
+        <state_interface name="velocity" />
+        <state_interface name="effort" />
+      </joint>
+    </ros2_control>
+  </xacro:macro>
 </robot>

File: ada_hardware/urdf/ada_hardware.xacro (robot description, xacro)
@@ -5,4 +5,5 @@
   <xacro:arg name="sim" default="none" />
   <xacro:arg name="readonly" default="false" />
+  <xacro:arg name="use_forque" default="true" />
   <xacro:include filename="$(find ada_description)/urdf/ada.xacro"/>
   <xacro:include filename="$(find ada_hardware)/urdf/ada_hardware.ros2_control.xacro"/>
@@ -11,3 +12,7 @@
     sim="$(arg sim)"
     readonly="$(arg readonly)" />
+  <xacro:dynamixel_hardware_interface
+    name="Dynamixel"
+    sim="$(arg sim)"
+    readonly="$(arg readonly)" />
 </robot>

Commit message: Fix parameter definitions for usb_port and baud_rate, rename joints

File: ada_hardware/urdf/ada_hardware.ros2_control.xacro (robot description, xacro)
@@ -111,9 +111,9 @@
         <xacro:if value="${sim == 'none'}">
           <plugin>ada_hardware/DynamixelHardware</plugin>
-          <param name="usb_port" value="/dev/ttyUSB0" />
-          <param name="baud_rate" value="1000000" />
+          <param name="usb_port">/dev/ttyUSB0</param>
+          <param name="baud_rate">1000000</param>
         </xacro:if>
       </hardware>
-      <joint name="AFMotor1_to_AFBase">
+      <joint name="af_joint_1">
         <param name="id">1</param>
         <xacro:unless value="${readonly}">
@@ -125,5 +125,5 @@
         <state_interface name="effort" />
       </joint>
-      <joint name="AFFTAdapter_to_AFMotor2">
+      <joint name="af_joint_2">
         <param name="id">2</param>
         <xacro:unless value="${readonly}">
