Commit message: Properly handle hand and arm controller switching in hardware interface.

File: ada_hardware/urdf/ada_hardware.xacro (robot description, xacro)
@@ -3,5 +3,5 @@
 <robot xmlns:xi="http://www.w3.org/2001/XInclude"
 	xmlns:xacro="http://www.ros.org/wiki/xacro" name="ada_hardware">
-  <xacro:arg name="use_mock_hardware" default="none" />
+  <xacro:arg name="sim" default="none" />
   <xacro:include filename="$(find ada_description)/urdf/ada.xacro"/>
   <xacro:include filename="$(find ada_hardware)/urdf/ada_hardware.ros2_control.xacro"/>

File: ada_moveit/config/ada.ros2_control.xacro (robot description, xacro)
@@ -1,11 +1,21 @@
 <?xml version="1.0"?>
 <robot xmlns:xacro="http://www.ros.org/wiki/xacro">
-    <xacro:macro name="ada_ros2_control" params="name initial_positions_file">
+    <xacro:macro name="ada_ros2_control" params="name initial_positions_file sim">
         <xacro:property name="initial_positions" value="${load_yaml(initial_positions_file)['initial_positions']}"/>
         <ros2_control name="${name}" type="system">
             <hardware>
-                <!-- By default, set up controllers for simulation. This won't work on real hardware -->
-                <plugin>ada_hardware/Jaco2</plugin>
-            </hardware>
+                <xacro:if value="${sim == 'mock'}">
+                  <plugin>mock_components/GenericSystem</plugin>
+                  <param name="mock_sensor_commands">false</param>
+                  <param name="state_following_offset">0.0</param>
+                </xacro:if>
+                <xacro:if value="${sim == 'isaac'}">
+                  <plugin>ada_hardware/JacoIsaac</plugin>
+                  <param name="namespace">/simulation</param>
+                </xacro:if>
+                <xacro:if value="${sim == 'none'}">
+                  <plugin>ada_hardware/Jaco2</plugin>
+                </xacro:if>
+              </hardware>
             <joint name="j2n6s200_joint_1">
                 <command_interface name="position"/>

File: ada_moveit/config/ada.urdf.xacro (robot description, xacro)
@@ -2,8 +2,11 @@
 <robot xmlns:xacro="http://www.ros.org/wiki/xacro" name="ada">
     <xacro:arg name="initial_positions_file" default="initial_positions.yaml" />
+    <xacro:arg name="sim" default="none" />
     <!-- Import ada urdf file -->
     <xacro:include filename="$(find ada_description)/urdf/ada.xacro" />
     <!-- Import control_xacro -->
     <xacro:include filename="ada.ros2_control.xacro" />
-    <xacro:ada_ros2_control name="ADAHardware" initial_positions_file="$(arg initial_positions_file)"/>
+    <xacro:ada_ros2_control name="ADAHardware"
+        initial_positions_file="$(arg initial_positions_file)"
+        sim="$(arg sim)" />
 </robot>

Commit message: Use updated ada macro

File: ada_hardware/urdf/ada_hardware.xacro (robot description, xacro)
@@ -5,7 +5,11 @@
   <xacro:arg name="sim" default="none" />
   <xacro:arg name="readonly" default="false" />
-  <xacro:arg name="end_effector_tool" default="articulable_fork" />
+  <xacro:arg name="end_effector_tool" default="fork" />
   <xacro:include filename="$(find ada_description)/urdf/ada.xacro"/>
   <xacro:include filename="$(find ada_hardware)/urdf/ada_hardware.ros2_control.xacro"/>
+  <link name="root"/>
+  <xacro:property name="root" value="root" />
+  <xacro:property name="end_effector_tool" value="$(arg end_effector_tool)" />
+  <xacro:ada base_parent="${root}" end_effector_tool="${end_effector_tool}" />
   <xacro:ada_hardware_interface
     name="Jaco2"

Commit message: Only load Dynamixel hardware interface if end_effector_tool is set to articulable_fork

File: ada_hardware/urdf/ada_hardware.xacro (robot description, xacro)
@@ -6,4 +6,5 @@
   <xacro:arg name="readonly" default="false" />
   <xacro:arg name="end_effector_tool" default="fork" />
+  <xacro:property name="end_effector_tool" value="$(arg end_effector_tool)" />
   <xacro:include filename="$(find ada_description)/urdf/ada.xacro"/>
   <xacro:include filename="$(find ada_hardware)/urdf/ada_hardware.ros2_control.xacro"/>
@@ -16,7 +17,9 @@
     sim="$(arg sim)"
     readonly="$(arg readonly)" />
-  <xacro:dynamixel_hardware_interface
-    name="DynamixelHardware"
-    sim="$(arg sim)"
-    readonly="$(arg readonly)" />
+  <xacro:if value="${end_effector_tool == 'articulable_fork'}">
+    <xacro:dynamixel_hardware_interface
+      name="DynamixelHardware"
+      sim="$(arg sim)"
+      readonly="$(arg readonly)" />
+  </xacro:if>
 </robot>

Commit message: Revert "Only load Dynamixel hardware interface if end_effector_tool is set to articulable_fork"
This reverts commit 669aa7d5a4f4f702bc6465c5465a9ef7680a808b.

File: ada_hardware/urdf/ada_hardware.xacro (robot description, xacro)
@@ -6,5 +6,4 @@
   <xacro:arg name="readonly" default="false" />
   <xacro:arg name="end_effector_tool" default="fork" />
-  <xacro:property name="end_effector_tool" value="$(arg end_effector_tool)" />
   <xacro:include filename="$(find ada_description)/urdf/ada.xacro"/>
   <xacro:include filename="$(find ada_hardware)/urdf/ada_hardware.ros2_control.xacro"/>
@@ -17,9 +16,7 @@
     sim="$(arg sim)"
     readonly="$(arg readonly)" />
-  <xacro:if value="${end_effector_tool == 'articulable_fork'}">
-    <xacro:dynamixel_hardware_interface
-      name="DynamixelHardware"
-      sim="$(arg sim)"
-      readonly="$(arg readonly)" />
-  </xacro:if>
+  <xacro:dynamixel_hardware_interface
+    name="DynamixelHardware"
+    sim="$(arg sim)"
+    readonly="$(arg readonly)" />
 </robot>

Commit message: Remove base_parent argument when instantiating ada macro

File: ada_hardware/urdf/ada_hardware.xacro (robot description, xacro)
@@ -8,8 +8,6 @@
   <xacro:include filename="$(find ada_description)/urdf/ada.xacro"/>
   <xacro:include filename="$(find ada_hardware)/urdf/ada_hardware.ros2_control.xacro"/>
-  <link name="root"/>
-  <xacro:property name="root" value="root" />
   <xacro:property name="end_effector_tool" value="$(arg end_effector_tool)" />
-  <xacro:ada base_parent="${root}" end_effector_tool="${end_effector_tool}" />
+  <xacro:ada end_effector_tool="${end_effector_tool}" />
   <xacro:ada_hardware_interface
     name="Jaco2"
