Commit message: Working MoveIt (running demo.launch.py) in both IsaacSim and Real

File: ada_moveit/config/ada.ros2_control.xacro (robot description, xacro)
@@ -2,5 +2,5 @@
 <robot xmlns:xacro="http://www.ros.org/wiki/xacro">
     <xacro:macro name="ada_ros2_control" params="name initial_positions_file sim">
-        <xacro:property name="initial_positions" value="${load_yaml(initial_positions_file)['initial_positions']}"/>
+        <xacro:property name="initial_positions" value="${xacro.load_yaml(initial_positions_file)['initial_positions']}"/>
         <ros2_control name="${name}" type="system">
             <hardware>
@@ -14,5 +14,5 @@
                   <param name="namespace">/simulation</param>
                 </xacro:if>
-                <xacro:if value="${sim == 'none'}">
+                <xacro:if value="${sim == 'real'}">
                   <plugin>ada_hardware/Jaco2</plugin>
                 </xacro:if>

File: ada_moveit/config/ada.urdf.xacro (robot description, xacro)
@@ -2,5 +2,5 @@
 <robot xmlns:xacro="http://www.ros.org/wiki/xacro" name="ada">
     <xacro:arg name="initial_positions_file" default="initial_positions.yaml" />
-    <xacro:arg name="sim" default="none" />
+    <xacro:arg name="sim" default="real" />
     <!-- Import ada urdf file -->
     <xacro:include filename="$(find ada_description)/urdf/ada.xacro" />

Commit message: Add ros2_control block for Articulable Fork, and initial positions

File: ada_moveit/config/ada.ros2_control.xacro (robot description, xacro)
@@ -132,3 +132,52 @@
         </ros2_control>
     </xacro:macro>
+    <xacro:macro name="af_ros2_control" params="name initial_positions_file sim">
+      <xacro:property name="initial_positions" value="${xacro.load_yaml(initial_positions_file)['initial_positions']}"/>
+      <ros2_control name="${name}" type="system">
+        <hardware>
+          <xacro:if value="${sim == 'mock'}">
+            <plugin>mock_components/GenericSystem</plugin>
+            <param name="mock_sensor_commands">false</param>
+            <param name="state_following_offset">0.0</param>
+          </xacro:if>
+          <xacro:if value="${sim == 'none'}">
+            <plugin>ada_hardware/DynamixelHardware</plugin>
+            <param name="usb_port">/dev/ttyUSB0</param>
+            <param name="baud_rate">1000000</param>
+          </xacro:if>
+        </hardware>
+        <joint name="af_joint_1">
+          <param name="id">1</param>
+          <xacro:unless value="${readonly}">
+            <command_interface name="position" />
+            <command_interface name="velocity" />
+          </xacro:unless>
+          <state_interface name="position">
+            <param name="initial_value">${initial_positions['af_joint_1']}</param>
+          </state_interface>
+          <state_interface name="velocity">
+              <param name="initial_value">0.0</param>
+          </state_interface>
+          <state_interface name="effort">
+              <param name="initial_value">0.0</param>
+          </state_interface>
+        </joint>
+        <joint name="af_joint_2">
+          <param name="id">2</param>
+          <xacro:unless value="${readonly}">
+            <command_interface name="position" />
+            <command_interface name="velocity" />
+          </xacro:unless>
+          <state_interface name="position">
+            <param name="initial_value">${initial_positions['af_joint_2']}</param>
+          </state_interface>
+          <state_interface name="velocity">
+              <param name="initial_value">0.0</param>
+          </state_interface>
+          <state_interface name="effort">
+              <param name="initial_value">0.0</param>
+          </state_interface>
+        </joint>
+      </ros2_control>
+    </xacro:macro>
 </robot>
