Commit message: Add configuration for end_effector_tool

File: ada_moveit/config/ada.urdf.xacro (robot description, xacro)
@@ -3,4 +3,7 @@
     <xacro:arg name="initial_positions_file" default="initial_positions.yaml" />
     <xacro:arg name="sim" default="real" />
+    <!-- TODO: figure out how to have ada.xacro inherit from this argument -->
+    <xacro:arg name="end_effector_tool" default="fork" />
+    <xacro:property name="cmp_end_effector_tool" value="$(arg end_effector_tool)"/>
     <!-- Import ada urdf file -->
     <xacro:include filename="$(find ada_description)/urdf/ada.xacro" />
@@ -10,6 +13,8 @@
         initial_positions_file="$(arg initial_positions_file)"
         sim="$(arg sim)" />
-    <xacro:af_ros2_control name="AFHardware"
-        initial_positions_file="$(arg initial_positions_file)"
-        sim="$(arg sim)" />
+    <xacro:if value="${cmp_end_effector_tool == 'articulable_fork'}">
+      <xacro:af_ros2_control name="AFHardware"
+          initial_positions_file="$(arg initial_positions_file)"
+          sim="$(arg sim)" />
+    </xacro:if>
 </robot>

Commit message: Use updated ada macro

File: ada_moveit/config/ada.urdf.xacro (robot description, xacro)
@@ -3,9 +3,11 @@
     <xacro:arg name="initial_positions_file" default="initial_positions.yaml" />
     <xacro:arg name="sim" default="real" />
-    <!-- TODO: figure out how to have ada.xacro inherit from this argument -->
     <xacro:arg name="end_effector_tool" default="fork" />
-    <xacro:property name="cmp_end_effector_tool" value="$(arg end_effector_tool)"/>
     <!-- Import ada urdf file -->
     <xacro:include filename="$(find ada_description)/urdf/ada.xacro" />
+    <link name="root"/>
+    <xacro:property name="root" value="root" />
+    <xacro:property name="end_effector_tool" value="$(arg end_effector_tool)" />
+    <xacro:ada base_parent="${root}" end_effector_tool="${end_effector_tool}" />
     <!-- Import control_xacro -->
     <xacro:include filename="ada.ros2_control.xacro" />
@@ -13,5 +15,5 @@
         initial_positions_file="$(arg initial_positions_file)"
         sim="$(arg sim)" />
-    <xacro:if value="${cmp_end_effector_tool == 'articulable_fork'}">
+    <xacro:if value="${end_effector_tool == 'articulable_fork'}">
       <xacro:af_ros2_control name="AFHardware"
           initial_positions_file="$(arg initial_positions_file)"

Commit message: Remove base_parent argument when instantiating ada macro

File: ada_moveit/config/ada.urdf.xacro (robot description, xacro)
@@ -6,8 +6,6 @@
     <!-- Import ada urdf file -->
     <xacro:include filename="$(find ada_description)/urdf/ada.xacro" />
-    <link name="root"/>
-    <xacro:property name="root" value="root" />
     <xacro:property name="end_effector_tool" value="$(arg end_effector_tool)" />
-    <xacro:ada base_parent="${root}" end_effector_tool="${end_effector_tool}" />
+    <xacro:ada end_effector_tool="${end_effector_tool}" />
     <!-- Import control_xacro -->
     <xacro:include filename="ada.ros2_control.xacro" />

Commit message: Add configurations for end_effector_tool argument

File: ada_moveit/config/ada.urdf.xacro (robot description, xacro)
@@ -16,9 +16,17 @@
     default="false"
   />
+  <xacro:arg
+    name="end_effector_tool"
+    default="fork"
+  />
   <!-- Import ada urdf file -->
   <xacro:include filename="$(find ada_description)/urdf/ada.xacro"/>
   <xacro:include filename="$(find articutool_description)/urdf/articutool.xacro"/>
+  <xacro:property
+    name="end_effector_tool"
+    value="$(arg end_effector_tool)"
+  />
   <xacro:ada use_forque="$(arg use_forque)"/>
-  <xacro:articutool base_parent="j2n6s200_end_effector" end_effector_tool="fork" joint_origin_rpy="0 0 ${J_PI/2}" joint_origin_xyz="0 -2.25 -1" dummy="false"/>
+  <xacro:articutool base_parent="j2n6s200_end_effector" end_effector_tool="${end_effector_tool}" joint_origin_rpy="0 0 ${J_PI/2}" joint_origin_xyz="0 -2.25 -1" dummy="false"/>
   <!-- Import control_xacro -->
   <xacro:include filename="ada.ros2_control.xacro"/>
