Commit message: Added fork tip frame

File: ada_description/urdf/forque/forque.xacro (robot description, xacro)
@@ -57,4 +57,10 @@
 	  	<xacro:forque_assembly_link link_name="forkTine" link_mesh="fork_tine"/>
 	  	<xacro:forque_assembly_joint joint_name="forkTine_to_forque" parent="forque" child="forkTine" joint_origin_xyz="-0.0054 0.008 0.093" joint_origin_rpy="0 ${J_PI} ${240*J_PI/180}"/>
+	  	<link name="forkTip" />
+	  	<joint name="forkTip_to_forkTine" type="fixed">
+		    <child link="forkTip"/>
+		    <parent link="forkTine"/>
+		    <origin rpy="${J_PI} 0 0" xyz="0.0135 0.007 0"/>
+		</joint>
 	</xacro:macro>
 </root>

Commit message: Fixed formatting

File: ada_description/urdf/forque/forque.xacro (robot description, xacro)
@@ -52,6 +52,4 @@
 		</joint>
 	</xacro:macro>
-	<!-- <inertia ixx="" iyy="" iyz="" izz="" ixy="" ixz=""/>
-	-->
 	<xacro:macro name="forque_assembly" params="base_parent use_antenna:=false">
 		<xacro:forque_assembly_link link_name="FTMount" link_mesh="2024_01_18_FTMount" mass="0.103" cog="0.010934 -0.138522 -0.05066">

Commit message: Added apriltag links

File: ada_description/urdf/forque/forque.xacro (robot description, xacro)
@@ -72,4 +72,10 @@
 		<!-- The slight rotation was manually added due to empirical deformations in the robot gripped, such that the fingers and fork handle were slightly pitched up relative to the wrist. -->
 		<xacro:forque_assembly_joint joint_name="forkHandle_to_FTMount" parent="FTMount" child="forkHandle" joint_origin_xyz="0 0 0.005" joint_origin_rpy="-0.025 0 0"/>
+		<!-- demo block to add the fork handle cover
+		<xacro:forque_assembly_link link_name="forkHandleCover" link_mesh="" mass="0" cog="0 0 0">
+			<xacro:insert_block name="default_inertial"/>
+		</xacro:forque_assembly_link>
+		<xacro:forque_assembly_joint joint_name="forkHandleCover_to_forkHandle" parent="forkHandle" child="forkHandleCover" joint_origin_xyz="0 0 0" joint_origin_rpy="0 0 0"/>
+		-->
 	  	<xacro:forque_assembly_link link_name="forque" link_mesh="ATI-9105-TW-NANO25-E" mass="0.0634" cog="0.0124692 0.0137169 0.010558">
 	  		<inertia ixx="0.000005235822" iyy="0.000006264852" iyz="-0.00000004033694" izz="0.00000640797" ixy="-0.0000003129932" ixz="0.000000013798"/>
@@ -86,4 +92,22 @@
 		    <origin rpy="${J_PI} 0 0" xyz="0.0135 0.007 0"/>
 		</joint>
+		<link name="apriltag_center" />
+	    <joint name="centerTag_to_handle" type="fixed">
+	        <child link="apriltag_center"/>
+	        <parent link="forkHandle"/>
+	        <origin rpy="${J_PI/6} ${J_PI} 0" xyz="0.01117 -0.196884 0.012848"/>
+	    </joint>
+	    <link name="apriltag_left" />
+	    <joint name="leftTag_to_handle" type="fixed">
+	        <child link="apriltag_left"/>
+	        <parent link="forkHandle"/>
+	        <origin rpy="0 ${J_PI} 0" xyz="0.022148 -0.170481 0.005781"/>
+	    </joint>
+	    <link name="apriltag_right" />
+	    <joint name="rightTag_to_handle" type="fixed">
+	        <child link="apriltag_right"/>
+	        <parent link="forkHandle"/>
+	        <origin rpy="0 ${J_PI} 0" xyz="0.000148 -0.170511 0.005781"/>
+	    </joint>
 	</xacro:macro>
 </root>

Commit message: [WIP] added joints, but that messes up MoveIt's chain

File: ada_description/urdf/forque/forque.xacro (robot description, xacro)
@@ -18,7 +18,8 @@
 		<inertia ixx="0.000005" iyy="0.000005" iyz="0" izz="0.000005" ixy="0" ixz="0"/>
 	</xacro:property>
-	<xacro:macro name="forque_assembly_link" params="link_name link_mesh mass:=0 cog:='0 0 0' *inertia">
+	<xacro:macro name="forque_assembly_link" params="link_name link_mesh mass:=0 cog:='0 0 0' origin_xyz:='0 0 0' *inertia">
 		<link name="${link_name}">
 			<visual>
+				<origin xyz="${origin_xyz}" rpy="0 0 0"/>
 				<geometry>
 					<mesh
@@ -31,4 +32,5 @@
 			</visual>
 			<collision>
+				<origin xyz="${origin_xyz}" rpy="0 0 0"/>
                 <geometry>
                     <mesh
@@ -66,10 +68,34 @@
 	  	  </xacro:forque_assembly_link>
 	  	  <xacro:forque_assembly_joint joint_name="FTAntenna_to_FT" parent="FT" child="FTAntenna" joint_origin_xyz="0 0 0" joint_origin_rpy="0 0 0"/>
-		  </xacro:if>
-	  	<xacro:forque_assembly_link link_name="forkHandle" link_mesh="2023_03_09_forkHandle" mass="0.0506" cog="0.0110024 -0.151715 -0.00934664">
+		</xacro:if>
+		<!-- TODO: The below 3 values were visually tuned, not precisely measured in a modeling software -->
+		<xacro:property name="forkHandle_offset_x" value="0.01105" />
+		<xacro:property name="forkHandle_offset_y" value="-0.0985" />
+		<xacro:property name="forkHandle_offset_z" value="-0.0095" />
+	  	<xacro:forque_assembly_link link_name="forkHandle" link_mesh="2023_03_09_forkHandle" mass="0.0506" cog="0.0110024 0.501715 -0.00934664" origin_xyz="${-forkHandle_offset_x} ${-forkHandle_offset_y} ${-forkHandle_offset_z}">
 	  		<inertia ixx="0.0000418078" iyy="0.0000177249" iyz="-0.000000210639" izz="0.00005200336" ixy="-0.000000396292" ixz="0.00000002424697"/>
 	  	</xacro:forque_assembly_link>
-		<!-- The slight rotation was manually added due to empirical deformations in the robot gripped, such that the fingers and fork handle were slightly pitched up relative to the wrist. -->
-		<xacro:forque_assembly_joint joint_name="forkHandle_to_FTMount" parent="FTMount" child="forkHandle" joint_origin_xyz="0 0 0.005" joint_origin_rpy="-0.025 0 0"/>
+		<!-- TODO: Before we delete the below two lines, does anyone know what the 0.005 z translation was for, and whether we should account for that in the new joints? -->
+		<!-- The slight rotation was manually added due to empirical deformations in the robot gripper, such that the fingers and fork handle were slightly pitched up relative to the wrist. -->
+		<!-- <xacro:forque_assembly_joint joint_name="forkHandle_to_FTMount" parent="FTMount" child="forkHandle" joint_origin_xyz="0 0 0.005" joint_origin_rpy="-0.025 0 0"/> -->
+		<link name="forkHandle_yaw"/>
+		<joint name="forkHandle_to_FTMount_yaw" type="revolute">
+			<parent link="FTMount" />
+			<child link="forkHandle_yaw" />
+			<axis xyz="0 0 1"/>
+			<origin xyz="${forkHandle_offset_x} ${forkHandle_offset_y} ${forkHandle_offset_z}" rpy="0 0 0" />
+			<!-- TODO: the below are arbitrary limits/dynamics and need to be tuned -->
+			<limit effort="80" velocity="0.15" lower="${-J_PI}" upper="${J_PI}"/>
+			<dynamics damping="0.0" friction="0.0"/>
+		</joint>
+		<joint name="forkHandle_to_FTMount_pitch" type="revolute">
+			<parent link="forkHandle_yaw" />
+			<child link="forkHandle" />
+			<axis xyz="1 0 0"/>
+			<origin xyz="0 0 0" rpy="0 0 0" />
+			<!-- TODO: the below are arbitrary limits/dynamics and need to be tuned -->
+			<limit effort="80" velocity="0.15" lower="${-J_PI}" upper="${J_PI}"/>
+			<dynamics damping="0.0" friction="0.0"/>
+		</joint>
 		<!-- demo block to add the fork handle cover
 		<xacro:forque_assembly_link link_name="forkHandleCover" link_mesh="" mass="0" cog="0 0 0">
@@ -81,5 +107,5 @@
 	  		<inertia ixx="0.000005235822" iyy="0.000006264852" iyz="-0.00000004033694" izz="0.00000640797" ixy="-0.0000003129932" ixz="0.000000013798"/>
 	  	</xacro:forque_assembly_link>
-	  	<xacro:forque_assembly_joint joint_name="forque_to_forkHandle" parent="forkHandle" child="forque" joint_origin_xyz="-0.00634 -0.222553 -0.004286" joint_origin_rpy="${J_PI/2} ${J_PI/3} 0"/>
+	  	<xacro:forque_assembly_joint joint_name="forque_to_forkHandle" parent="forkHandle" child="forque" joint_origin_xyz="${-0.00634 - forkHandle_offset_x} ${-0.222553 - forkHandle_offset_y} ${-0.004286 - forkHandle_offset_z}" joint_origin_rpy="${J_PI/2} ${J_PI/3} 0"/>
 	  	<xacro:forque_assembly_link link_name="forkTine" link_mesh="fork_tine" mass="0.024" cog="0.013090 0.0180789 0.0445231">
 	  		<inertia ixx="0.0000098769" iyy="0.000009848103" iyz="0.00000057639" izz="0.0000015674" ixy="0.000000000806182" ixz="-0.00000000296036"/>

Commit message: Positioned fork handle components and added cog, mass, and inertia for each

File: ada_description/urdf/forque/forque.xacro (robot description, xacro)
@@ -67,8 +67,12 @@
 	  	  <xacro:forque_assembly_joint joint_name="FTAntenna_to_FT" parent="FT" child="FTAntenna" joint_origin_xyz="0 0 0" joint_origin_rpy="0 0 0"/>
 		  </xacro:if>
-	  	<xacro:forque_assembly_link link_name="forkHandle" link_mesh="2024_06_24_forkHandleHollow" mass="0.0506" cog="0.0110024 -0.151715 -0.00934664">
-	  		<inertia ixx="0.0000418078" iyy="0.0000177249" iyz="-0.000000210639" izz="0.00005200336" ixy="-0.000000396292" ixz="0.00000002424697"/>
+	  	<xacro:forque_assembly_link link_name="forkHandle" link_mesh="2024_06_24_forkHandleHollow" mass="0.028" cog="0.011097 -0.162629 -0.011948">
+	  		<inertia ixx="0.00003114" iyy="0.000011867" iyz="0.00000054005" izz="0.000038478" ixy="-0.00000050626" ixz="0.000000082271"/>
 	  	</xacro:forque_assembly_link>
-		<xacro:forque_assembly_joint joint_name="forkHandle_to_FTMount" parent="FTMount" child="forkHandle" joint_origin_xyz="0 0 0" joint_origin_rpy="-0.025 0 0"/>
+		<xacro:forque_assembly_joint joint_name="forkHandle_to_FTMount" parent="FTMount" child="forkHandle" joint_origin_xyz="0 0.005 0.0013" joint_origin_rpy="-0.025 0 0"/>
+		<xacro:forque_assembly_link link_name="forkHandleCover" link_mesh="2024_06_24_forkHandleCover" mass="0.004" cog="0.011157 -0.168451 0.006404">
+	  		<inertia ixx="0.0000027878" iyy="0.00000064518" iyz="0.00000016201" izz="0.000003363634" ixy="0.00000000012805" ixz="0.00000000006585"/>
+	  	</xacro:forque_assembly_link>
+		<xacro:forque_assembly_joint joint_name="forkHandleCover_to_forkHandle" parent="forkHandle" child="forkHandleCover" joint_origin_xyz="0 0 0" joint_origin_rpy="0 0 0"/>
 	  	<xacro:forque_assembly_link link_name="forque" link_mesh="ATI-9105-TW-NANO25-E" mass="0.0634" cog="0.0124692 0.0137169 0.010558">
 	  		<inertia ixx="0.000005235822" iyy="0.000006264852" iyz="-0.00000004033694" izz="0.00000640797" ixy="-0.0000003129932" ixz="0.000000013798"/>

Commit message: Add hollow fork handle design to urdf (#47)
* [WIP] Added hollow fork and cover STLs to mesh folder

* Positioned fork handle components and added cog, mass, and inertia for each

File: ada_description/urdf/forque/forque.xacro (robot description, xacro)
@@ -67,8 +67,12 @@
 	  	  <xacro:forque_assembly_joint joint_name="FTAntenna_to_FT" parent="FT" child="FTAntenna" joint_origin_xyz="0 0 0" joint_origin_rpy="0 0 0"/>
 		  </xacro:if>
-	  	<xacro:forque_assembly_link link_name="forkHandle" link_mesh="2023_03_09_forkHandle" mass="0.0506" cog="0.0110024 -0.151715 -0.00934664">
-	  		<inertia ixx="0.0000418078" iyy="0.0000177249" iyz="-0.000000210639" izz="0.00005200336" ixy="-0.000000396292" ixz="0.00000002424697"/>
+	  	<xacro:forque_assembly_link link_name="forkHandle" link_mesh="2024_06_24_forkHandleHollow" mass="0.028" cog="0.011097 -0.162629 -0.011948">
+	  		<inertia ixx="0.00003114" iyy="0.000011867" iyz="0.00000054005" izz="0.000038478" ixy="-0.00000050626" ixz="0.000000082271"/>
 	  	</xacro:forque_assembly_link>
-		<xacro:forque_assembly_joint joint_name="forkHandle_to_FTMount" parent="FTMount" child="forkHandle" joint_origin_xyz="0 0 0" joint_origin_rpy="-0.025 0 0"/>
+		<xacro:forque_assembly_joint joint_name="forkHandle_to_FTMount" parent="FTMount" child="forkHandle" joint_origin_xyz="0 0.005 0.0013" joint_origin_rpy="-0.025 0 0"/>
+		<xacro:forque_assembly_link link_name="forkHandleCover" link_mesh="2024_06_24_forkHandleCover" mass="0.004" cog="0.011157 -0.168451 0.006404">
+	  		<inertia ixx="0.0000027878" iyy="0.00000064518" iyz="0.00000016201" izz="0.000003363634" ixy="0.00000000012805" ixz="0.00000000006585"/>
+	  	</xacro:forque_assembly_link>
+		<xacro:forque_assembly_joint joint_name="forkHandleCover_to_forkHandle" parent="forkHandle" child="forkHandleCover" joint_origin_xyz="0 0 0" joint_origin_rpy="0 0 0"/>
 	  	<xacro:forque_assembly_link link_name="forque" link_mesh="ATI-9105-TW-NANO25-E" mass="0.0634" cog="0.0124692 0.0137169 0.010558">
 	  		<inertia ixx="0.000005235822" iyy="0.000006264852" iyz="-0.00000004033694" izz="0.00000640797" ixy="-0.0000003129932" ixz="0.000000013798"/>

Commit message: Add Articulable Fork XACRO and STL

File: ada_description/urdf/forque/forque.xacro (robot description, xacro)
@@ -201,4 +201,104 @@
             joint_origin_rpy="-0.025 0 0"
             fixed="true"/>
+        <xacro:forque_assembly_link
+            link_name="AFBase"
+            link_mesh="fr12-h103"
+            mass="0.0907185"
+            cog="0.0 0.0 0.0">
+            <xacro:insert_block name="default_inertial"/>
+        </xacro:forque_assembly_link>
+        <xacro:forque_assembly_joint
+            joint_name="AFBase_to_forkHandle"
+            type="fixed"
+            parent="forkHandle"
+            child="AFBase"
+            joint_axis_xyz="0 0 1"
+            joint_origin_xyz="0.010929196 -0.278553 -0.011"
+            joint_origin_rpy="0 0 0"
+            fixed="true"/>
+        <xacro:forque_assembly_link
+            link_name="AFMotor1"
+            link_mesh="XC-430_idle"
+            mass="0.065"
+            cog="0.21641853 -14.751192 -16.796092">
+            <inertia
+                ixx="18680.931"
+                iyy="9585.9138"
+                iyz="-845.46678"
+                izz="17346.641"
+                ixy="1.3348619"
+                ixz="-45.354028"/>
+        </xacro:forque_assembly_link>
+        <xacro:forque_assembly_joint
+            joint_name="AFMotor1_to_AFBase"
+            type="revolute"
+            parent="AFBase"
+            child="AFMotor1"
+            joint_axis_xyz="0 0 1"
+            joint_origin_xyz="0 0 0"
+            joint_origin_rpy="${J_PI/2} 0 ${J_PI/2}"
+            joint_lower_limit="${-J_PI/2}"
+            joint_upper_limit="${J_PI/2}"
+            joint_velocity_limit="1"
+            joint_torque_limit="1.4"
+            fixed="false"/>
+        <xacro:forque_assembly_link
+            link_name="AFMotorFixture1"
+            link_mesh="fr12-s101"
+            mass="0.0453592"
+            cog="0 0 0">
+            <xacro:insert_block name="default_inertial"/>
+        </xacro:forque_assembly_link>
+        <xacro:forque_assembly_joint
+            joint_name="AFMotorFixture1_to_AFMotor1"
+            type="fixed"
+            parent="AFMotor1"
+            child="AFMotorFixture1"
+            joint_axis_xyz="0 0 1"
+            joint_origin_xyz="0 0 0"
+            joint_origin_rpy="0 ${-J_PI/2} 0"
+            fixed="true"/>
+        <xacro:forque_assembly_link
+            link_name="AFMotor2"
+            link_mesh="XC-430_idle"
+            mass="0.065"
+            cog="0.21641853 -14.751192 -16.796092">
+            <inertia
+                ixx="18680.931"
+                iyy="9585.9138"
+                iyz="-845.46678"
+                izz="17346.641"
+                ixy="1.3348619"
+                ixz="-45.354028"/>
+        </xacro:forque_assembly_link>
+        <xacro:forque_assembly_joint
+            joint_name="AFMotor2_to_AFMotorFixture1"
+            type="fixed"
+            parent="AFMotor1"
+            child="AFMotor2"
+            joint_axis_xyz="0 0 1"
+            joint_origin_xyz="-0.03825 0 0"
+            joint_origin_rpy="0 ${-J_PI/2} 0"
+            fixed="true"/>
+        <xacro:forque_assembly_link
+            link_name="AFFTAdapter"
+            link_mesh="roll_to_ft_adapter"
+            mass="0.001"
+            cog="0 0 0">
+            <xacro:insert_block name="default_inertial"/>
+        </xacro:forque_assembly_link>
+        <xacro:forque_assembly_joint
+            joint_name="AFFTAdapter_to_AFMotor2"
+            type="revolute"
+            parent="AFMotor2"
+            child="AFFTAdapter"
+            joint_axis_xyz="0 1 0"
+            joint_origin_xyz="0 0 0.019"
+            joint_origin_rpy="${-J_PI/2} 0 0"
+            joint_lower_limit="${-J_PI}"
+            joint_upper_limit="${J_PI}"
+            joint_velocity_limit="1"
+            joint_torque_limit="1.4"
+            fixed="false"/>
 	  	<xacro:forque_assembly_link
             link_name="forque"
@@ -215,10 +315,10 @@
 	  	</xacro:forque_assembly_link>
 	  	<xacro:forque_assembly_joint
-            joint_name="forque_to_forkHandle"
-            type="fixed"
-            parent="forkHandle"
+            joint_name="forque_to_AFFTAdapter"
+            type="fixed"
+            parent="AFFTAdapter"
             child="forque"
             joint_axis_xyz="0 0 1"
-            joint_origin_xyz="-0.00634 -0.222553 -0.004286"
+            joint_origin_xyz="-0.0175 -0.011 0.004"
             joint_origin_rpy="${J_PI/2} ${J_PI/3} 0"
             fixed="true"/>
