Commit message: Fix indentation

File: ada_description/urdf/forque/forque.xacro (robot description, xacro)
@@ -46,40 +46,40 @@
 	</xacro:macro>
 	<xacro:macro name="forque_assembly_joint" params="joint_name type parent child joint_axis_xyz joint_origin_xyz joint_origin_rpy joint_lower_limit:=${forque_assembly_dummy_default_value} joint_upper_limit:=${forque_assembly_dummy_default_value} joint_velocity_limit:=${forque_assembly_dummy_default_value} joint_torque_limit:=${forque_assembly_dummy_default_value} fixed:=false">
-        <xacro:if value="${(type == 'fixed' and not fixed) or (type != 'fixed' and fixed)}">
-            <xacro:ERROR_inconsistent_joint_type_specification/>
-        </xacro:if>
-        <xacro:if value="${type == 'revolute'}">
-            <xacro:if value="${joint_lower_limit == forque_assembly_dummy_default_value}">
-                <xacro:ERROR_joint_lower_limit_needs_to_be_set_for_a_revolute_joint/>
-            </xacro:if>
-            <xacro:if value="${joint_upper_limit == forque_assembly_dummy_default_value}">
-                <xacro:ERROR_joint_upper_limit_needs_to_be_set_for_a_revolute_joint/>
-            </xacro:if>
-        </xacro:if>
-        <xacro:unless value="${type =='fixed'}">
-            <xacro:if value="${joint_velocity_limit == forque_assembly_dummy_default_value}">
-                <xacro:ERROR_joint_velocity_limit_needs_to_be_set_for_a_non_fixed_joint/>
-            </xacro:if>
-            <xacro:if value="${joint_torque_limit == forque_assembly_dummy_default_value}">
-                <xacro:ERROR_joint_torque_limit_needs_to_be_set_for_a_non_fixed_joint/>
-            </xacro:if>
-        </xacro:unless>
-        <joint name="${joint_name}" type="${type}">
-            <parent link="${parent}"/>
-            <child link="${child}"/>
-            <axis xyz="${joint_axis_xyz}"/>
-            <xacro:if value="${type == 'revolute'}">
-                <limit
-                    effort="${joint_torque_limit}"
-                    velocity="${joint_velocity_limit}"
-                    lower="${joint_lower_limit}"
-                    upper="${joint_upper_limit}"/>
-            </xacro:if>
-            <xacro:if value="${type == 'continuous'}">
-                <limit effort="${joint_torque_limit}" velocity="${joint_velocity_limit}"/>
-            </xacro:if>
-            <origin xyz="${joint_origin_xyz}" rpy="${joint_origin_rpy}"/>
-            <dynamics damping="0.0" friction="0.0"/>
-        </joint>
+    <xacro:if value="${(type == 'fixed' and not fixed) or (type != 'fixed' and fixed)}">
+      <xacro:ERROR_inconsistent_joint_type_specification/>
+    </xacro:if>
+    <xacro:if value="${type == 'revolute'}">
+      <xacro:if value="${joint_lower_limit == forque_assembly_dummy_default_value}">
+        <xacro:ERROR_joint_lower_limit_needs_to_be_set_for_a_revolute_joint/>
+      </xacro:if>
+      <xacro:if value="${joint_upper_limit == forque_assembly_dummy_default_value}">
+        <xacro:ERROR_joint_upper_limit_needs_to_be_set_for_a_revolute_joint/>
+      </xacro:if>
+    </xacro:if>
+    <xacro:unless value="${type =='fixed'}">
+      <xacro:if value="${joint_velocity_limit == forque_assembly_dummy_default_value}">
+        <xacro:ERROR_joint_velocity_limit_needs_to_be_set_for_a_non_fixed_joint/>
+      </xacro:if>
+      <xacro:if value="${joint_torque_limit == forque_assembly_dummy_default_value}">
+        <xacro:ERROR_joint_torque_limit_needs_to_be_set_for_a_non_fixed_joint/>
+      </xacro:if>
+    </xacro:unless>
+    <joint name="${joint_name}" type="${type}">
+      <parent link="${parent}"/>
+      <child link="${child}"/>
+      <axis xyz="${joint_axis_xyz}"/>
+      <xacro:if value="${type == 'revolute'}">
+        <limit
+          effort="${joint_torque_limit}"
+          velocity="${joint_velocity_limit}"
+          lower="${joint_lower_limit}"
+          upper="${joint_upper_limit}"/>
+      </xacro:if>
+      <xacro:if value="${type == 'continuous'}">
+        <limit effort="${joint_torque_limit}" velocity="${joint_velocity_limit}"/>
+      </xacro:if>
+      <origin xyz="${joint_origin_xyz}" rpy="${joint_origin_rpy}"/>
+      <dynamics damping="0.0" friction="0.0"/>
+    </joint>
 	</xacro:macro>
 	<xacro:macro name="forque_assembly" params="base_parent end_effector_tool use_antenna:=false">

Commit message: Update forque Xacro macro

File: ada_description/urdf/forque/forque.xacro (robot description, xacro)
@@ -33,4 +33,8 @@
     />
   </xacro:property>
+  <xacro:property
+    name="forque_assembly_dummy_default_value"
+    value="1234567890"
+  />
   <xacro:macro
     name="forque_assembly_link"
@@ -69,16 +73,34 @@
   <xacro:macro
     name="forque_assembly_joint"
-    params="joint_name parent child joint_origin_xyz joint_origin_rpy"
+    params="joint_name type parent child joint_axis_xyz joint_origin_xyz joint_origin_rpy joint_lower_limit:=${forque_assembly_dummy_default_value} joint_upper_limit:=${forque_assembly_dummy_default_value} joint_velocity_limit:=${forque_assembly_dummy_default_value} joint_torque_limit:=${forque_assembly_dummy_default_value}"
   >
     <joint
       name="${joint_name}"
-      type="fixed"
+      type="${type}"
     >
       <parent link="${parent}"/>
       <child link="${child}"/>
-      <axis xyz="0 0 1"/>
+      <axis xyz="${joint_axis_xyz}"/>
+      <xacro:if value="${type == 'revolute'}">
+        <limit
+          effort="${joint_torque_limit}"
+          velocity="${joint_velocity_limit}"
+          lower="${joint_lower_limit}"
+          upper="${joint_upper_limit}"
+        />
+      </xacro:if>
+      <xacro:if value="${type == 'continuous'}">
+        <limit
+          effort="${joint_torque_limit}"
+          velocity="${joint_velocity_limit}"
+        />
+      </xacro:if>
       <origin
         xyz="${joint_origin_xyz}"
         rpy="${joint_origin_rpy}"
+      />
+      <dynamics
+        damping="0.0"
+        friction="0.0"
       />
     </joint>
@@ -105,6 +127,8 @@
     <xacro:forque_assembly_joint
       joint_name="FTMount_to_world"
+      type="fixed"
       parent="${base_parent}"
       child="FTMount"
+      joint_axis_xyz="0 0 1"
       joint_origin_xyz="0 0 -0.005"
       joint_origin_rpy="0 0 0"
@@ -127,6 +151,8 @@
     <xacro:forque_assembly_joint
       joint_name="FT_to_FTMount"
+      type="fixed"
       parent="FTMount"
       child="FT"
+      joint_axis_xyz="0 0 1"
       joint_origin_xyz="0 0 0"
       joint_origin_rpy="0 0 0"
@@ -143,6 +169,8 @@
       <xacro:forque_assembly_joint
         joint_name="FTAntenna_to_FT"
+        type="fixed"
         parent="FT"
         child="FTAntenna"
+        joint_axis_xyz="0 0 1"
         joint_origin_xyz="0 0 0"
         joint_origin_rpy="0 0 0"
@@ -167,6 +195,8 @@
     <xacro:forque_assembly_joint
       joint_name="forkHandle_to_FTMount"
+      type="fixed"
       parent="FTMount"
       child="forkHandle"
+      joint_axis_xyz="0 0 1"
       joint_origin_xyz="0 0.005 0.0013"
       joint_origin_rpy="-0.025 0 -0.0065"
@@ -189,6 +219,8 @@
     <xacro:forque_assembly_joint
       joint_name="forkHandleCover_to_forkHandle"
+      type="fixed"
       parent="forkHandle"
       child="forkHandleCover"
+      joint_axis_xyz="0 0 1"
       joint_origin_xyz="0 0 0"
       joint_origin_rpy="0 0 0"
@@ -211,6 +243,8 @@
     <xacro:forque_assembly_joint
       joint_name="forque_to_forkHandle"
+      type="fixed"
       parent="forkHandle"
       child="forque"
+      joint_axis_xyz="0 0 1"
       joint_origin_xyz="-0.00634 -0.222553 -0.004286"
       joint_origin_rpy="${J_PI/2} ${J_PI/3} 0"
@@ -233,6 +267,8 @@
     <xacro:forque_assembly_joint
       joint_name="forkTine_to_forque"
+      type="fixed"
       parent="forque"
       child="forkTine"
+      joint_axis_xyz="0 0 1"
       joint_origin_xyz="-0.0054 0.008 0.093"
       joint_origin_rpy="0 ${J_PI} ${240*J_PI/180}"

Commit message: Revert "Update forque Xacro macro"
This reverts commit 130922fe86c3708d6046c8b2f4715c25edc6f9d4.

File: ada_description/urdf/forque/forque.xacro (robot description, xacro)
@@ -33,8 +33,4 @@
     />
   </xacro:property>
-  <xacro:property
-    name="forque_assembly_dummy_default_value"
-    value="1234567890"
-  />
   <xacro:macro
     name="forque_assembly_link"
@@ -73,34 +69,16 @@
   <xacro:macro
     name="forque_assembly_joint"
-    params="joint_name type parent child joint_axis_xyz joint_origin_xyz joint_origin_rpy joint_lower_limit:=${forque_assembly_dummy_default_value} joint_upper_limit:=${forque_assembly_dummy_default_value} joint_velocity_limit:=${forque_assembly_dummy_default_value} joint_torque_limit:=${forque_assembly_dummy_default_value}"
+    params="joint_name parent child joint_origin_xyz joint_origin_rpy"
   >
     <joint
       name="${joint_name}"
-      type="${type}"
+      type="fixed"
     >
       <parent link="${parent}"/>
       <child link="${child}"/>
-      <axis xyz="${joint_axis_xyz}"/>
-      <xacro:if value="${type == 'revolute'}">
-        <limit
-          effort="${joint_torque_limit}"
-          velocity="${joint_velocity_limit}"
-          lower="${joint_lower_limit}"
-          upper="${joint_upper_limit}"
-        />
-      </xacro:if>
-      <xacro:if value="${type == 'continuous'}">
-        <limit
-          effort="${joint_torque_limit}"
-          velocity="${joint_velocity_limit}"
-        />
-      </xacro:if>
+      <axis xyz="0 0 1"/>
       <origin
         xyz="${joint_origin_xyz}"
         rpy="${joint_origin_rpy}"
-      />
-      <dynamics
-        damping="0.0"
-        friction="0.0"
       />
     </joint>
@@ -127,8 +105,6 @@
     <xacro:forque_assembly_joint
       joint_name="FTMount_to_world"
-      type="fixed"
       parent="${base_parent}"
       child="FTMount"
-      joint_axis_xyz="0 0 1"
       joint_origin_xyz="0 0 -0.005"
       joint_origin_rpy="0 0 0"
@@ -151,8 +127,6 @@
     <xacro:forque_assembly_joint
       joint_name="FT_to_FTMount"
-      type="fixed"
       parent="FTMount"
       child="FT"
-      joint_axis_xyz="0 0 1"
       joint_origin_xyz="0 0 0"
       joint_origin_rpy="0 0 0"
@@ -169,8 +143,6 @@
       <xacro:forque_assembly_joint
         joint_name="FTAntenna_to_FT"
-        type="fixed"
         parent="FT"
         child="FTAntenna"
-        joint_axis_xyz="0 0 1"
         joint_origin_xyz="0 0 0"
         joint_origin_rpy="0 0 0"
@@ -195,8 +167,6 @@
     <xacro:forque_assembly_joint
       joint_name="forkHandle_to_FTMount"
-      type="fixed"
       parent="FTMount"
       child="forkHandle"
-      joint_axis_xyz="0 0 1"
       joint_origin_xyz="0 0.005 0.0013"
       joint_origin_rpy="-0.025 0 -0.0065"
@@ -219,8 +189,6 @@
     <xacro:forque_assembly_joint
       joint_name="forkHandleCover_to_forkHandle"
-      type="fixed"
       parent="forkHandle"
       child="forkHandleCover"
-      joint_axis_xyz="0 0 1"
       joint_origin_xyz="0 0 0"
       joint_origin_rpy="0 0 0"
@@ -243,8 +211,6 @@
     <xacro:forque_assembly_joint
       joint_name="forque_to_forkHandle"
-      type="fixed"
       parent="forkHandle"
       child="forque"
-      joint_axis_xyz="0 0 1"
       joint_origin_xyz="-0.00634 -0.222553 -0.004286"
       joint_origin_rpy="${J_PI/2} ${J_PI/3} 0"
@@ -267,8 +233,6 @@
     <xacro:forque_assembly_joint
       joint_name="forkTine_to_forque"
-      type="fixed"
       parent="forque"
       child="forkTine"
-      joint_axis_xyz="0 0 1"
       joint_origin_xyz="-0.0054 0.008 0.093"
       joint_origin_rpy="0 ${J_PI} ${240*J_PI/180}"
